File: injector_drive6.sch (KiCad schematic (older format))
At the start: 17 parts, among them P36 CONN_1, P37 CONN_1, Q20 PIP-3104, Q21 HALL

Commit message: Removed LM1815 options. Now adaptive mode and square waves are the default,
Parts:
- C54: Field1 (none) -> newark,97M4148; Field2 (none) -> vendor1, smd w hem; Field3 (none) -> vendor2, thru w hem; Field4 (none) -> vendor2, smd w hem; Field5 (none) -> 200,V; Field6 (none) -> 10,%; Field7 (none) -> Multilayer Ceramic; Field8 (none) -> other,more,stuff
- D96, D99: Field1 (none) -> vendor1, thru w hem; Field2 (none) -> vendor1, smd w hem; Field3 (none) -> vendor2, thru w hem; Field4 (none) -> vendor2, smd w hem; Field5 (none) -> reverse,V; Field6 (none) -> current,A; Field7 (none) -> x; Field8 (none) -> other,more,stuff
- D97: Field1 (none) -> newark,18M3533; Field2 (none) -> vendor1, smd w hem; Field3 (none) -> vendor2, thru w hem; Field4 (none) -> vendor2, smd w hem; Field5 (none) -> 500,mW; Field6 (none) -> 20,mA; Field7 (none) -> X; Field8 (none) -> other,more,stuff
- D98: Field1 (none) -> newark,58K2469; Field2 (none) -> vendor1, smd w hem; Field3 (none) -> vendor2, thru w hem; Field4 (none) -> vendor2, smd w hem; Field5 (none) -> x,x; Field6 (none) -> x,x; Field7 (none) -> construct; Field8 (none) -> other,more,stuff
- L6: Field1 (none) -> vendor1, thru w hem; Field2 (none) -> vendor1, smd w hem; Field3 (none) -> vendor2, thru w hem; Field4 (none) -> vendor2, smd w hem; Field5 (none) -> x,x; Field6 (none) -> x,x; Field7 (none) -> x; Field8 (none) -> other,more,stuff
- Q20: Field1 (none) -> digi,PIP3104-ND; Field2 (none) -> vendor1, smd w hem; Field3 (none) -> vendor2, thru w hem; Field4 (none) -> vendor2, smd w hem; Field5 (none) -> 8,A; Field6 (none) -> x,x; Field7 (none) -> TOPFET; Field8 (none) -> other,more,stuff
- Q21: Field1 (none) -> digi,480-2002-ND; Field2 (none) -> vendor1, smd w hem; Field3 (none) -> vendor2, thru w hem; Field4 (none) -> vendor2, smd w hem; Field5 (none) -> x,x; Field6 (none) -> x,x; Field7 (none) -> x; Field8 (none) -> other,more,stuff
- R136: Field1 (none) -> newark,38k0327; Field2 (none) -> vendor1, smd w hem; Field3 (none) -> vendor2, thru w hem; Field4 (none) -> vendor2, smd w hem; Field5 (none) -> 250,mW; Field6 (none) -> 5,%; Field7 (none) -> carbon film; Field8 (none) -> other,more,stuff
- R137: Field1 (none) -> newark,38K0329; Field2 (none) -> vendor1, smd w hem; Field3 (none) -> vendor2, thru w hem; Field4 (none) -> vendor2, smd w hem; Field5 (none) -> 250,mW; Field6 (none) -> 5,%; Field7 (none) -> carbon film; Field8 (none) -> other,more,stuff
- R138: Field1 (none) -> newark,38k0352; Field2 (none) -> vendor1, smd w hem; Field3 (none) -> vendor2, thru w hem; Field4 (none) -> vendor2, smd w hem; Field5 (none) -> 250,mW; Field6 (none) -> 5,%; Field7 (none) -> carbon film; Field8 (none) -> other,more,stuff
- R139: Field1 (none) -> vendor1, thru w hem; Field2 (none) -> vendor1, smd w hem; Field3 (none) -> vendor2, thru w hem; Field4 (none) -> vendor2, smd w hem; Field5 (none) -> power,W; Field6 (none) -> tol,%; Field7 (none) -> construct; Field8 (none) -> other,more,stuff
- R140: Field1 (none) -> newark,38K0352; Field2 (none) -> vendor1, smd w hem; Field3 (none) -> vendor2, thru w hem; Field4 (none) -> vendor2, smd w hem; Field5 (none) -> 250,mW; Field6 (none) -> 5,%; Field7 (none) -> carbon film; Field8 (none) -> other,more,stuff
- R141: Field1 (none) -> newark,59K8561; Field2 (none) -> vendor1, smd w hem; Field3 (none) -> vendor2, thru w hem; Field4 (none) -> vendor2, smd w hem; Field5 (none) -> 1,W; Field6 (none) -> 5,%; Field7 (none) -> construct; Field8 (none) -> other,more,stuff
- R142: Field1 (none) -> newark,38K0340; Field2 (none) -> vendor1, smd w hem; Field3 (none) -> vendor2, thru w hem; Field4 (none) -> vendor2, smd w hem; Field5 (none) -> 1/4,W; Field6 (none) -> 5,%; Field7 (none) -> carbon film; Field8 (none) -> other,more,stuff
