File: thermistor_resistor_input1.sch (KiCad schematic (older format))
At the start: 4 parts, among them P53 CONN_1, P54 CONN_1, Q23 MOS_N

Commit message: Removed LM1815 options. Now adaptive mode and square waves are the default,
Parts:
- Q23: Field1 (none) -> digi,PIP3104-ND; Field2 (none) -> vendor1, smd w hem; Field3 (none) -> vendor2, thru w hem; Field4 (none) -> vendor2, smd w hem; Field5 (none) -> 8,A; Field6 (none) -> x,x; Field7 (none) -> TOPFET; Field8 (none) -> other,more,stuff
- R178: Field1 (none) -> newark,41K8850; Field2 (none) -> vendor1, smd w hem; Field3 (none) -> vendor2, thru w hem; Field4 (none) -> vendor2, smd w hem; Field5 (none) -> .125,W; Field6 (none) -> 1,%; Field7 (none) -> metal film; Field8 (none) -> other,more,stuff
Changed lines of the file:
@@
-EESchema Schematic File Version 1
-LIBS:power,./freeEMS_lib,device,conn,linear,regul,74xx,cmos4000,adc-dac,memory,xilinx,special,microcontrollers,dsp,microchip,analog_switches,motorola,texas,intel,audio,interface,digital-audio,philips,display,cypress,siliconi,contrib,valves,./freeEMS_1.cache
+EESchema Schematic File Version 2  date Fri 02 Jul 2010 02:24:35 PM ART
+LIBS:power
+LIBS:freeEMS_lib
+LIBS:device
+LIBS:conn
+LIBS:linear
+LIBS:regul
+LIBS:74xx
+LIBS:cmos4000
+LIBS:adc-dac
+LIBS:memory
+LIBS:xilinx
+LIBS:special
+LIBS:microcontrollers
+LIBS:dsp
+LIBS:microchip
+LIBS:analog_switches
+LIBS:motorola
+LIBS:texas
+LIBS:intel
+LIBS:audio
+LIBS:interface
+LIBS:digital-audio
+LIBS:philips
+LIBS:display
+LIBS:cypress
+LIBS:siliconi
+LIBS:contrib
+LIBS:valves
+LIBS:freeEMS_1-cache
 EELAYER 23  0
 EELAYER END
@@
 Sheet 40 41
 Title "freeEMS 1.0"
-Date "15 nov 2008"
+Date "2 jul 2010"
 Rev "A.20"
 Comp "diyefi.org"
@@
 U 1 1 48B16ED5
 P 3200 2150
-F 0 "Q23" H 3210 2320 60  0000 R C
-F 1 "MOS_N" H 3210 2000 60  0000 R C
-F 2 "TO92" V 3130 2900 60  0001 C C
-F 4 "digi,PIP3104-ND" V 1330 3900 60  0001 C C
-F 5 "vendor1, smd w hem" V 1330 3900 60  0001 C C
-F 6 "vendor2, thru w hem" V 1330 3900 60  0001 C C
-F 7 "vendor2, smd w hem" V 1330 3900 60  0001 C C
-F 8 "8,A" V 1330 3900 60  0001 C C
-F 9 "x,x" V 1330 3900 60  0001 C C
-F 10 "TOPFET" V 1330 3900 60  0001 C C
-F 11 "other,more,stuff" V 1330 3900 60  0001 C C
+F 0 "Q23" H 3210 2320 60  0000 R CNN
+F 1 "MOS_N" H 3210 2000 60  0000 R CNN
+F 2 "TO92" V 3130 2900 60  0001 C CNN
+F 4 "digi,PIP3104-ND" V 1330 3900 60  0001 C CNN "Field1"
+F 5 "vendor1, smd w hem" V 1330 3900 60  0001 C CNN "Field2"
+F 6 "vendor2, thru w hem" V 1330 3900 60  0001 C CNN "Field3"
+F 7 "vendor2, smd w hem" V 1330 3900 60  0001 C CNN "Field4"
+F 8 "8,A" V 1330 3900 60  0001 C CNN "Field5"
+F 9 "x,x" V 1330 3900 60  0001 C CNN "Field6"
+F 10 "TOPFET" V 1330 3900 60  0001 C CNN "Field7"
+F 11 "other,more,stuff" V 1330 3900 60  0001 C CNN "Field8"
 	1    3200 2150
 	1    0    0    -1
@@
 U 1 1 48AA1AB3
 P 3450 1950
-F 0 "P54" H 3530 1950 40  0000 L C
-F 1 "CONN_1" H 3450 2005 30  0001 C C
-F 2 "1PIN" V 1130 2600 60  0001 C C
+F 0 "P54" H 3530 1950 40  0000 L CNN
+F 1 "CONN_1" H 3450 2005 30  0001 C CNN
+F 2 "1PIN" V 1130 2600 60  0001 C CNN
 	1    3450 1950
 	1    0    0    -1
@@
 U 1 1 48AA1AB0
 P 3450 1750
-F 0 "P53" H 3530 1750 40  0000 L C
-F 1 "CONN_1" H 3450 1805 30  0001 C C
-F 2 "1PIN" V 1130 2600 60  0001 C C
+F 0 "P53" H 3530 1750 40  0000 L CNN
+F 1 "CONN_1" H 3450 1805 30  0001 C CNN
+F 2 "1PIN" V 1130 2600 60  0001 C CNN
 	1    3450 1750
 	1    0    0    -1
 $EndComp
-Text GLabel 2700 950  0    60   Output
+Text HLabel 2700 950  0    60   Output ~ 0
 5v_reg
 $Comp
@@
 U 1 1 488E4A25
 P 3300 1200
-F 0 "R178" V 3380 1200 50  0000 C C
-F 1 "2.7k" V 3300 1200 50  0000 C C
-F 2 "R4-SM0805" V 3480 1300 60  0001 C C
-F 4 "newark,41K8850" V 1130 2600 60  0001 C C
-F 5 "vendor1, smd w hem" V 1130 2600 60  0001 C C
-F 6 "vendor2, thru w hem" V 1130 2600 60  0001 C C
-F 7 "vendor2, smd w hem" V 1130 2600 60  0001 C C
-F 8 ".125,W" V 1130 2600 60  0001 C C
-F 9 "1,%" V 1130 2600 60  0001 C C
-F 10 "metal film" V 1130 2600 60  0001 C C
-F 11 "other,more,stuff" V 1130 2600 60  0001 C C
+F 0 "R178" V 3380 1200 50  0000 C CNN
+F 1 "2.7k" V 3300 1200 50  0000 C CNN
+F 2 "R4-SM0805" V 3480 1300 60  0001 C CNN
+F 4 "newark,41K8850" V 1130 2600 60  0001 C CNN "Field1"
+F 5 "vendor1, smd w hem" V 1130 2600 60  0001 C CNN "Field2"
+F 6 "vendor2, thru w hem" V 1130 2600 60  0001 C CNN "Field3"
+F 7 "vendor2, smd w hem" V 1130 2600 60  0001 C CNN "Field4"
+F 8 ".125,W" V 1130 2600 60  0001 C CNN "Field5"
+F 9 "1,%" V 1130 2600 60  0001 C CNN "Field6"
+F 10 "metal film" V 1130 2600 60  0001 C CNN "Field7"
+F 11 "other,more,stuff" V 1130 2600 60  0001 C CNN "Field8"
 	1    3300 1200
 	1    0    0    -1
 $EndComp
-Text GLabel 2650 2150 0    60   Input
+Text HLabel 2650 2150 0    60   Input ~ 0
 Measure_temp
-Text GLabel 2650 2350 0    60   BiDi
+Text HLabel 2650 2350 0    60   BiDi ~ 0
 analog_sensor_gnd
-Text GLabel 2700 1450 0    60   Output
+Text HLabel 2700 1450 0    60   Output ~ 0
 analog_sensor_TEMP
 $EndSCHEMATC

Commit message: Implemented P&H, removed current sense circuitry, removed all unnecessary files from the repo
Parts:
- R?: renamed from R178; Field5 .125,W -> .5,W
- renumbered P53 to P?, P54 to P?, Q23 to Q?
Connections:
- net analog_sensor_gnd: no longer P?.1, Q?.2 (D)
- new net: P?.1, Q?.2 (D)
Changed lines of the file:
@@
-EESchema Schematic File Version 2  date Fri 02 Jul 2010 05:44:26 PM ART
+EESchema Schematic File Version 2  date Sat 03 Jul 2010 10:49:02 AM ART
 LIBS:power
 LIBS:freeEMS_lib
@@
 EELAYER END
 $Descr A 11000 8500
-Sheet 40 41
+Sheet 1 41
 Title "freeEMS 1.0"
-Date "2 jul 2010"
-Rev "A.20"
+Date "3 jul 2010"
+Rev "A.07"
 Comp "diyefi.org"
 Comment1 "thermistor_resistor_input.sch"
@@
 Comment4 ""
 $EndDescr
-Connection ~ 3300 2350
-Wire Wire Line
-	2650 2350 3350 2350
-Wire Wire Line
-	3350 2350 3350 1950
-Wire Wire Line
-	3350 1950 3300 1950
-Wire Wire Line
-	2700 1450 3300 1450
-Wire Wire Line
-	2700 950  3300 950
-Wire Wire Line
-	2650 2150 3000 2150
-Wire Wire Line
-	3300 1450 3300 1750
 $Comp
-L PIP-3104 Q23
+L PIP-3104 Q?
 U 1 1 48B16ED5
 P 3200 2150
-F 0 "Q23" H 3210 2320 60  0000 R CNN
+F 0 "Q?" H 3210 2320 60  0000 R CNN
 F 1 "MOS_N" H 3210 2000 60  0000 R CNN
 F 2 "TO92" V 3130 2900 60  0001 C CNN
@@
 $EndComp
 $Comp
-L CONN_1 P54
+L CONN_1 P?
 U 1 1 48AA1AB3
 P 3450 1950
-F 0 "P54" H 3530 1950 40  0000 L CNN
+F 0 "P?" H 3530 1950 40  0000 L CNN
 F 1 "CONN_1" H 3450 2005 30  0001 C CNN
 F 2 "1PIN" V 1130 2600 60  0001 C CNN
@@
 $EndComp
 $Comp
-L CONN_1 P53
+L CONN_1 P?
 U 1 1 48AA1AB0
 P 3450 1750
-F 0 "P53" H 3530 1750 40  0000 L CNN
+F 0 "P?" H 3530 1750 40  0000 L CNN
 F 1 "CONN_1" H 3450 1805 30  0001 C CNN
 F 2 "1PIN" V 1130 2600 60  0001 C CNN
@@
 	1    0    0    -1
 $EndComp
+Wire Wire Line
+	3300 1750 3300 1450
+Wire Wire Line
+	2650 2150 3000 2150
+Wire Wire Line
+	2700 950  3300 950
+Wire Wire Line
+	3300 1450 2700 1450
+Wire Wire Line
+	2650 2350 3300 2350
 Text HLabel 2700 950  0    60   Output ~ 0
 5v_reg
 $Comp
-L R R178
+L R R?
 U 1 1 488E4A25
 P 3300 1200
-F 0 "R178" V 3380 1200 50  0000 C CNN
+F 0 "R?" V 3380 1200 50  0000 C CNN
 F 1 "2.7k" V 3300 1200 50  0000 C CNN
 F 2 "R4-SM0805" V 3480 1300 60  0001 C CNN
@@
 F 6 "vendor2, thru w hem" V 1130 2600 60  0001 C CNN "Field3"
 F 7 "vendor2, smd w hem" V 1130 2600 60  0001 C CNN "Field4"
-F 8 ".125,W" V 1130 2600 60  0001 C CNN "Field5"
+F 8 ".5,W" V 1130 2600 60  0001 C CNN "Field5"
 F 9 "1,%" V 1130 2600 60  0001 C CNN "Field6"
 F 10 "metal film" V 1130 2600 60  0001 C CNN "Field7"
