File: an_protect2.sch (KiCad schematic (older format))
At the start: 15 parts

Commit message: Removed LM1815 options. Now adaptive mode and square waves are the default,
Parts:
- C34, C35, C36: Field1 (none) -> newark,39K8137; Field2 (none) -> vendor1, smd w hem; Field3 (none) -> vendor2, thru w hem; Field4 (none) -> vendor2, smd w hem; Field5 (none) -> 50,V; Field6 (none) -> 10,%; Field7 (none) -> Multilayer Ceramic; Field8 (none) -> other,more,stuff
- D49, D50, D51, D52, D53, D54: Field1 (none) -> newark,10M2940; Field2 (none) -> vendor1, smd w hem; Field3 (none) -> vendor2, thru w hem; Field4 (none) -> vendor2, smd w hem; Field5 (none) -> 1000,V; Field6 (none) -> 1,A; Field7 (none) -> x; Field8 (none) -> other,more,stuff
- R64, R65, R66, R68, R70: Field1 (none) -> newark,38K0327; Field2 (none) -> vendor1, smd w hem; Field3 (none) -> vendor2, thru w hem; Field4 (none) -> vendor2, smd w hem; Field5 (none) -> 1/4,W; Field6 (none) -> 5,%; Field7 (none) -> Carbon film; Field8 (none) -> other,more,stuff
- R69: Field1 (none) -> newark,38K0327; Field2 (none) -> vendor1, smd w hem; Field3 (none) -> vendor2, thru w hem; Field4 (none) -> vendor2, smd w hem; Field5 (none) -> 1/4,W; Field6 (none) -> 5,%; Field7 (none) -> carbon film; Field8 (none) -> other,more,stuff

Commit message: Implemented P&H, removed current sense circuitry, removed all unnecessary files from the repo
Parts:
- renumbered C36 to C?, C35 to C?, C34 to C?, D53 to D?, D54 to D?, D51 to D?, D52 to D?, D49 to D?, D50 to D?, R66 to R?, R70 to R?, R65 to R?, R69 to R?, R64 to R?, R68 to R?
Changed lines of the file:
@@
-EESchema Schematic File Version 2  date Fri 02 Jul 2010 05:44:26 PM ART
+EESchema Schematic File Version 2  date Sat 03 Jul 2010 10:49:02 AM ART
 LIBS:power
 LIBS:freeEMS_lib
@@
 EELAYER END
 $Descr A 11000 8500
-Sheet 22 41
+Sheet 1 41
 Title "freeEMS 1.0"
-Date "2 jul 2010"
-Rev "A.20"
+Date "3 jul 2010"
+Rev "A.07"
 Comp "diyefi.org"
 Comment1 "an_protect.sch"
@@
 Connection ~ 2750 800
 Wire Wire Line
-	6500 800  2650 800
-Wire Wire Line
-	6500 3450 2650 3450
+	2650 800  6500 800
+Wire Wire Line
+	2650 3450 6500 3450
 Wire Wire Line
 	4200 4050 4550 4050
@@
 Connection ~ 6500 2150
 $Comp
-L R R68
+L R R?
 U 1 1 489597BF
 P 3950 4050
-F 0 "R68" V 4030 4050 50  0000 C CNN
+F 0 "R?" V 4030 4050 50  0000 C CNN
 F 1 "1k" V 3950 4050 50  0000 C CNN
 F 2 "R4-SM0805" V 4130 4150 60  0001 C CNN
@@
 $EndComp
 $Comp
-L GND #PWR035
+L GND #PWR?
 U 1 1 489597BE
 P 2000 4500
-F 0 "#PWR035" H 2000 4500 30  0001 C CNN
+F 0 "#PWR?" H 2000 4500 30  0001 C CNN
 F 1 "GND" H 2000 4430 30  0001 C CNN
 	1    2000 4500
@@
 $EndComp
 $Comp
-L DIODE D50
+L DIODE D?
 U 1 1 489597BD
 P 2650 4250
-F 0 "D50" H 2650 4350 40  0000 C CNN
+F 0 "D?" H 2650 4350 40  0000 C CNN
 F 1 "1N4148" H 2650 4150 40  0000 C CNN
 F 2 "D4-SMB" V 1130 2600 60  0001 C CNN
@@
 $EndComp
 $Comp
-L C C34
+L C C?
 U 1 1 489597BC
 P 3200 4250
-F 0 "C34" H 3250 4350 50  0000 L CNN
+F 0 "C?" H 3250 4350 50  0000 L CNN
 F 1 "100nf" H 3250 4150 50  0000 L CNN
 F 2 "C1V7" V 1130 2600 60  0001 C CNN
@@
 $EndComp
 $Comp
-L R R64
+L R R?
 U 1 1 489597BB
 P 2250 4050
-F 0 "R64" V 2330 4050 50  0000 C CNN
+F 0 "R?" V 2330 4050 50  0000 C CNN
 F 1 "1k" V 2250 4050 50  0000 C CNN
 F 2 "R4-SM0805" V 2430 4150 60  0001 C CNN
@@
 $EndComp
 $Comp
-L DIODE D49
+L DIODE D?
 U 1 1 489597BA
 P 2650 3650
-F 0 "D49" H 2650 3750 40  0000 C CNN
+F 0 "D?" H 2650 3750 40  0000 C CNN
 F 1 "1N4148" H 2650 3550 40  0000 C CNN
 F 2 "D4-SMB" V 1130 2600 60  0001 C CNN
@@
 analog_sensor_out_3
 $Comp
-L R R69
+L R R?
 U 1 1 489597B9
 P 4000 2750
-F 0 "R69" V 4080 2750 50  0000 C CNN
+F 0 "R?" V 4080 2750 50  0000 C CNN
 F 1 "1k" V 4000 2750 50  0000 C CNN
 F 2 "R4-SM0805" V 4180 2850 60  0001 C CNN
@@
 $EndComp
 $Comp
-L GND #PWR036
+L GND #PWR?
 U 1 1 489597B8
 P 2050 3200
-F 0 "#PWR036" H 2050 3200 30  0001 C CNN
+F 0 "#PWR?" H 2050 3200 30  0001 C CNN
 F 1 "GND" H 2050 3130 30  0001 C CNN
 	1    2050 3200
@@
 $EndComp
 $Comp
-L DIODE D52
+L DIODE D?
 U 1 1 489597B7
 P 2700 2950
-F 0 "D52" H 2700 3050 40  0000 C CNN
+F 0 "D?" H 2700 3050 40  0000 C CNN
 F 1 "1N4148" H 2700 2850 40  0000 C CNN
 F 2 "D4-SMB" V 1130 2600 60  0001 C CNN
@@
 $EndComp
 $Comp
-L C C35
+L C C?
 U 1 1 489597B6
 P 3250 2950
-F 0 "C35" H 3300 3050 50  0000 L CNN
+F 0 "C?" H 3300 3050 50  0000 L CNN
 F 1 "100nf" H 3300 2850 50  0000 L CNN
 F 2 "C1V7" V 1130 2600 60  0001 C CNN
@@
 $EndComp
 $Comp
-L R R65
+L R R?
 U 1 1 489597B5
 P 2300 2750
-F 0 "R65" V 2380 2750 50  0000 C CNN
+F 0 "R?" V 2380 2750 50  0000 C CNN
 F 1 "1k" V 2300 2750 50  0000 C CNN
 F 2 "R4-SM0805" V 2480 2850 60  0001 C CNN
@@
 $EndComp
 $Comp
-L DIODE D51
+L DIODE D?
 U 1 1 489597B4
 P 2700 2350
-F 0 "D51" H 2700 2450 40  0000 C CNN
+F 0 "D?" H 2700 2450 40  0000 C CNN
 F 1 "1N4148" H 2700 2250 40  0000 C CNN
 F 2 "D4-SMB" V 1130 2600 60  0001 C CNN
@@
 analog_sensor_out_2
 $Comp
-L R R70
+L R R?
 U 1 1 488CCA4A
 P 4050 1400
-F 0 "R70" V 4130 1400 50  0000 C CNN
+F 0 "R?" V 4130 1400 50  0000 C CNN
 F 1 "1k" V 4050 1400 50  0000 C CNN
 F 2 "R4-SM0805" V 4230 1500 60  0001 C CNN
@@
 $EndComp
 $Comp
-L GND #PWR037
+L GND #PWR?
 U 1 1 486F8C14
 P 2100 1850
-F 0 "#PWR037" H 2100 1850 30  0001 C CNN
+F 0 "#PWR?" H 2100 1850 30  0001 C CNN
 F 1 "GND" H 2100 1780 30  0001 C CNN
 	1    2100 1850
@@
 $EndComp
 $Comp
-L DIODE D54
+L DIODE D?
 U 1 1 486F8B98
 P 2750 1600
-F 0 "D54" H 2750 1700 40  0000 C CNN
+F 0 "D?" H 2750 1700 40  0000 C CNN
 F 1 "1N4148" H 2750 1500 40  0000 C CNN
 F 2 "D4-SMB" V 1130 2600 60  0001 C CNN
@@
 $EndComp
 $Comp
-L C C36
+L C C?
 U 1 1 486F8B93
 P 3300 1600
-F 0 "C36" H 3350 1700 50  0000 L CNN
+F 0 "C?" H 3350 1700 50  0000 L CNN
 F 1 "100nf" H 3350 1500 50  0000 L CNN
 F 2 "C1V7" V 1130 2600 60  0001 C CNN
@@
 $EndComp
 $Comp
-L R R66
+L R R?
 U 1 1 486F8B82
 P 2350 1400
-F 0 "R66" V 2430 1400 50  0000 C CNN
+F 0 "R?" V 2430 1400 50  0000 C CNN
 F 1 "1k" V 2350 1400 50  0000 C CNN
 F 2 "R4-SM0805" V 2530 1500 60  0001 C CNN
@@
 $EndComp
 $Comp
-L DIODE D53
+L DIODE D?
 U 1 1 486F8B5C
 P 2750 1000
-F 0 "D53" H 2750 1100 40  0000 C CNN
+F 0 "D?" H 2750 1100 40  0000 C CNN
 F 1 "1N4148" H 2750 900 40  0000 C CNN
 F 2 "D4-SMB" V 1130 2600 60  0001 C CNN

Commit message: Corrected ERC errors by fixing the custom FreeEMS components pinouts
Parts:
- removed C?: 100nf, C1V7, symbol C
- removed D? (x2): 1N4148, D4-SMB, symbol DIODE
- removed R? (x3): 1k, R4-SM0805, symbol R
- added C31: 100nf, C1V7, symbol C
- added D31, D36: 1N4148, D4-SMB, symbol DIODE
- added R49, R50, R51: 1k, R4-SM0805, symbol R
- gave numbers to parts that had none: 9
Connections:
- net GND: now also C31.2, D36.1 (A)
- net analog_sensor_in_1: now also R49.2
- net analog_sensor_out_2: now also R51.1
- net analog_sensor_out_3: now also R50.1
- net analog_sensor_vcc: now also D31.2 (K)
- net at D35.1 (A), R52.2: now also C31.1, D36.2 (K), R49.1
- net at C30.1, D33.1 (A), D34.2 (K)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: now also R51.2
- net at C29.1, D32.2 (K), R47.1: now also D31.1 (A), R50.2
Changed lines of the file:
@@
-EESchema Schematic File Version 2  date Sat 03 Jul 2010 10:49:02 AM ART
+EESchema Schematic File Version 2  date Sat 03 Jul 2010 12:32:24 PM ART
 LIBS:power
 LIBS:freeEMS_lib
@@
 Connection ~ 2750 800
 Wire Wire Line
-	2650 800  6500 800
-Wire Wire Line
-	2650 3450 6500 3450
+	6500 800  2650 800
+Wire Wire Line
+	6500 3450 2650 3450
 Wire Wire Line
 	4200 4050 4550 4050
@@
 Connection ~ 6500 2150
 $Comp
-L R R?
-U 1 1 489597BF
+L R R50
+U 1 1 4C2F52F7
 P 3950 4050
-F 0 "R?" V 4030 4050 50  0000 C CNN
+F 0 "R50" V 4030 4050 50  0000 C CNN
 F 1 "1k" V 3950 4050 50  0000 C CNN
 F 2 "R4-SM0805" V 4130 4150 60  0001 C CNN
@@
 $EndComp
 $Comp
-L GND #PWR?
-U 1 1 489597BE
+L GND #PWR056
+U 1 1 4C2F52F6
 P 2000 4500
-F 0 "#PWR?" H 2000 4500 30  0001 C CNN
+F 0 "#PWR056" H 2000 4500 30  0001 C CNN
 F 1 "GND" H 2000 4430 30  0001 C CNN
 	1    2000 4500
@@
 $EndComp
 $Comp
-L DIODE D?
+L DIODE D32
 U 1 1 489597BD
 P 2650 4250
-F 0 "D?" H 2650 4350 40  0000 C CNN
+F 0 "D32" H 2650 4350 40  0000 C CNN
 F 1 "1N4148" H 2650 4150 40  0000 C CNN
 F 2 "D4-SMB" V 1130 2600 60  0001 C CNN
@@
 $EndComp
 $Comp
-L C C?
+L C C29
 U 1 1 489597BC
 P 3200 4250
-F 0 "C?" H 3250 4350 50  0000 L CNN
+F 0 "C29" H 3250 4350 50  0000 L CNN
 F 1 "100nf" H 3250 4150 50  0000 L CNN
 F 2 "C1V7" V 1130 2600 60  0001 C CNN
@@
 $EndComp
 $Comp
-L R R?
+L R R47
 U 1 1 489597BB
 P 2250 4050
-F 0 "R?" V 2330 4050 50  0000 C CNN
+F 0 "R47" V 2330 4050 50  0000 C CNN
 F 1 "1k" V 2250 4050 50  0000 C CNN
 F 2 "R4-SM0805" V 2430 4150 60  0001 C CNN
@@
 $EndComp
 $Comp
-L DIODE D?
-U 1 1 489597BA
+L DIODE D31
+U 1 1 4C2F52F2
 P 2650 3650
-F 0 "D?" H 2650 3750 40  0000 C CNN
+F 0 "D31" H 2650 3750 40  0000 C CNN
 F 1 "1N4148" H 2650 3550 40  0000 C CNN
 F 2 "D4-SMB" V 1130 2600 60  0001 C CNN
@@
 analog_sensor_out_3
 $Comp
-L R R?
-U 1 1 489597B9
+L R R51
+U 1 1 4C2F52F1
 P 4000 2750
-F 0 "R?" V 4080 2750 50  0000 C CNN
+F 0 "R51" V 4080 2750 50  0000 C CNN
 F 1 "1k" V 4000 2750 50  0000 C CNN
 F 2 "R4-SM0805" V 4180 2850 60  0001 C CNN
@@
 $EndComp
 $Comp
-L GND #PWR?
+L GND #PWR057
 U 1 1 489597B8
 P 2050 3200
-F 0 "#PWR?" H 2050 3200 30  0001 C CNN
+F 0 "#PWR057" H 2050 3200 30  0001 C CNN
 F 1 "GND" H 2050 3130 30  0001 C CNN
 	1    2050 3200
@@
 $EndComp
 $Comp
-L DIODE D?
+L DIODE D34
 U 1 1 489597B7
 P 2700 2950
-F 0 "D?" H 2700 3050 40  0000 C CNN
+F 0 "D34" H 2700 3050 40  0000 C CNN
 F 1 "1N4148" H 2700 2850 40  0000 C CNN
 F 2 "D4-SMB" V 1130 2600 60  0001 C CNN
@@
 $EndComp
 $Comp
-L C C?
+L C C30
 U 1 1 489597B6
 P 3250 2950
-F 0 "C?" H 3300 3050 50  0000 L CNN
+F 0 "C30" H 3300 3050 50  0000 L CNN
 F 1 "100nf" H 3300 2850 50  0000 L CNN
 F 2 "C1V7" V 1130 2600 60  0001 C CNN
@@
 $EndComp
 $Comp
-L R R?
+L R R48
 U 1 1 489597B5
 P 2300 2750
-F 0 "R?" V 2380 2750 50  0000 C CNN
+F 0 "R48" V 2380 2750 50  0000 C CNN
 F 1 "1k" V 2300 2750 50  0000 C CNN
 F 2 "R4-SM0805" V 2480 2850 60  0001 C CNN
@@
 $EndComp
 $Comp
-L DIODE D?
+L DIODE D33
 U 1 1 489597B4
 P 2700 2350
-F 0 "D?" H 2700 2450 40  0000 C CNN
+F 0 "D33" H 2700 2450 40  0000 C CNN
 F 1 "1N4148" H 2700 2250 40  0000 C CNN
 F 2 "D4-SMB" V 1130 2600 60  0001 C CNN
@@
 analog_sensor_out_2
 $Comp
-L R R?
+L R R52
 U 1 1 488CCA4A
 P 4050 1400
-F 0 "R?" V 4130 1400 50  0000 C CNN
+F 0 "R52" V 4130 1400 50  0000 C CNN
 F 1 "1k" V 4050 1400 50  0000 C CNN
 F 2 "R4-SM0805" V 4230 1500 60  0001 C CNN
@@
 $EndComp
 $Comp
-L GND #PWR?
-U 1 1 486F8C14
+L GND #PWR058
+U 1 1 4C2F52A8
 P 2100 1850
-F 0 "#PWR?" H 2100 1850 30  0001 C CNN
+F 0 "#PWR058" H 2100 1850 30  0001 C CNN
 F 1 "GND" H 2100 1780 30  0001 C CNN
 	1    2100 1850
@@
 $EndComp
 $Comp
-L DIODE D?
-U 1 1 486F8B98
+L DIODE D36
+U 1 1 4C2F52A7
 P 2750 1600
-F 0 "D?" H 2750 1700 40  0000 C CNN
+F 0 "D36" H 2750 1700 40  0000 C CNN
 F 1 "1N4148" H 2750 1500 40  0000 C CNN
 F 2 "D4-SMB" V 1130 2600 60  0001 C CNN
@@
 $EndComp
 $Comp
-L C C?
-U 1 1 486F8B93
+L C C31
+U 1 1 4C2F52A6
 P 3300 1600
-F 0 "C?" H 3350 1700 50  0000 L CNN
+F 0 "C31" H 3350 1700 50  0000 L CNN
 F 1 "100nf" H 3350 1500 50  0000 L CNN
 F 2 "C1V7" V 1130 2600 60  0001 C CNN
@@
 $EndComp
 $Comp
-L R R?
-U 1 1 486F8B82
+L R R49
+U 1 1 4C2F52A5
 P 2350 1400
-F 0 "R?" V 2430 1400 50  0000 C CNN
+F 0 "R49" V 2430 1400 50  0000 C CNN
 F 1 "1k" V 2350 1400 50  0000 C CNN
 F 2 "R4-SM0805" V 2530 1500 60  0001 C CNN
@@
 $EndComp
 $Comp
-L DIODE D?
+L DIODE D35
 U 1 1 486F8B5C
 P 2750 1000
-F 0 "D?" H 2750 1100 40  0000 C CNN
+F 0 "D35" H 2750 1100 40  0000 C CNN
 F 1 "1N4148" H 2750 900 40  0000 C CNN
 F 2 "D4-SMB" V 1130 2600 60  0001 C CNN

Commit message: MAP circuit compatible with external sensors. Baro is left untouched
Parts:
- removed D32, D34, D36: 1N4148, D4-SMB, symbol DIODE
- added D32, D34, D36: SCHOTTKY, SOD-123, symbol DIODESCH
Connections:
- net GND: now also D32.1 (A), D34.1 (A), D36.1 (A)
- net at C31.1, D35.1 (A), R49.1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: now also D36.2 (K)
- net at C30.1, D33.1 (A), R48.1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: now also D34.2 (K)
- net at C29.1, D31.1 (A), R47.1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: now also D32.2 (K)
Changed lines of the file:
@@
-EESchema Schematic File Version 2  date Thu 22 Jul 2010 10:06:33 AM ART
+EESchema Schematic File Version 2  date Sat 24 Jul 2010 11:01:40 AM ART
 LIBS:power
 LIBS:freeEMS_lib
@@
 Sheet 28 41
 Title "freeEMS 1.0"
-Date "22 jul 2010"
+Date "24 jul 2010"
 Rev "A.07"
 Comp "diyefi.org"
@@
 Comment4 ""
 $EndDescr
+$Comp
+L DIODESCH D36
+U 1 1 4C4972F9
+P 2750 1600
+F 0 "D36" H 2750 1700 40  0000 C CNN
+F 1 "SCHOTTKY" H 2750 1500 40  0000 C CNN
+F 2 "SOD-123" H 2750 1600 60  0001 C CNN
+	1    2750 1600
+	0    -1   -1   0
+$EndComp
+$Comp
+L DIODESCH D34
+U 1 1 4C4972F8
+P 2700 2950
+F 0 "D34" H 2700 3050 40  0000 C CNN
+F 1 "SCHOTTKY" H 2700 2850 40  0000 C CNN
+F 2 "SOD-123" H 2700 2950 60  0001 C CNN
+	1    2700 2950
+	0    -1   -1   0
+$EndComp
+$Comp
+L DIODESCH D32
+U 1 1 4C4972F7
+P 2650 4250
+F 0 "D32" H 2650 4350 40  0000 C CNN
+F 1 "SCHOTTKY" H 2650 4150 40  0000 C CNN
+F 2 "SOD-123" H 2650 4250 60  0001 C CNN
+	1    2650 4250
+	0    -1   -1   0
+$EndComp
 Wire Wire Line
 	6500 800  6500 3450
@@
 	1    2000 4500
 	1    0    0    -1
-$EndComp
-$Comp
-L DIODE D32
-U 1 1 489597BD
-P 2650 4250
-F 0 "D32" H 2650 4350 40  0000 C CNN
-F 1 "1N4148" H 2650 4150 40  0000 C CNN
-F 2 "D4-SMB" V 1130 2600 60  0001 C CNN
-F 4 "newark,10M2940" V 1130 2600 60  0001 C CNN "Field1"
-F 5 "vendor1, smd w hem" V 1130 2600 60  0001 C CNN "Field2"
-F 6 "vendor2, thru w hem" V 1130 2600 60  0001 C CNN "Field3"
-F 7 "vendor2, smd w hem" V 1130 2600 60  0001 C CNN "Field4"
-F 8 "1000,V" V 1130 2600 60  0001 C CNN "Field5"
-F 9 "1,A" V 1130 2600 60  0001 C CNN "Field6"
-F 10 "x" V 1130 2600 60  0001 C CNN "Field7"
-F 11 "other,more,stuff" V 1130 2600 60  0001 C CNN "Field8"
-	1    2650 4250
-	0    -1   -1   0
 $EndComp
 $Comp
@@
 $EndComp
 $Comp
-L DIODE D34
-U 1 1 489597B7
-P 2700 2950
-F 0 "D34" H 2700 3050 40  0000 C CNN
-F 1 "1N4148" H 2700 2850 40  0000 C CNN
-F 2 "D4-SMB" V 1130 2600 60  0001 C CNN
-F 4 "newark,10M2940" V 1130 2600 60  0001 C CNN "Field1"
-F 5 "vendor1, smd w hem" V 1130 2600 60  0001 C CNN "Field2"
-F 6 "vendor2, thru w hem" V 1130 2600 60  0001 C CNN "Field3"
-F 7 "vendor2, smd w hem" V 1130 2600 60  0001 C CNN "Field4"
-F 8 "1000,V" V 1130 2600 60  0001 C CNN "Field5"
-F 9 "1,A" V 1130 2600 60  0001 C CNN "Field6"
-F 10 "x" V 1130 2600 60  0001 C CNN "Field7"
-F 11 "other,more,stuff" V 1130 2600 60  0001 C CNN "Field8"
-	1    2700 2950
-	0    -1   -1   0
-$EndComp
-$Comp
 L C C30
 U 1 1 489597B6
@@
 $EndComp
 $Comp
-L DIODE D36
-U 1 1 4C2F52A7
-P 2750 1600
-F 0 "D36" H 2750 1700 40  0000 C CNN
-F 1 "1N4148" H 2750 1500 40  0000 C CNN
-F 2 "D4-SMB" V 1130 2600 60  0001 C CNN
-F 4 "newark,10M2940" V 1130 2600 60  0001 C CNN "Field1"
-F 5 "vendor1, smd w hem" V 1130 2600 60  0001 C CNN "Field2"
-F 6 "vendor2, thru w hem" V 1130 2600 60  0001 C CNN "Field3"
-F 7 "vendor2, smd w hem" V 1130 2600 60  0001 C CNN "Field4"
-F 8 "1000,V" V 1130 2600 60  0001 C CNN "Field5"
-F 9 "1,A" V 1130 2600 60  0001 C CNN "Field6"
-F 10 "x" V 1130 2600 60  0001 C CNN "Field7"
-F 11 "other,more,stuff" V 1130 2600 60  0001 C CNN "Field8"
-	1    2750 1600
-	0    -1   -1   0
-$EndComp
-$Comp
