File: an_protect4.sch (KiCad schematic (older format))
At the start: 20 parts

Commit message: Removed LM1815 options. Now adaptive mode and square waves are the default,
Parts:
- C41, C42, C43, C44: Field1 (none) -> newark,39K8137; Field2 (none) -> vendor1, smd w hem; Field3 (none) -> vendor2, thru w hem; Field4 (none) -> vendor2, smd w hem; Field5 (none) -> 50,V; Field6 (none) -> 10,%; Field7 (none) -> Multilayer Ceramic; Field8 (none) -> other,more,stuff
- D63, D64, D65, D66, D67, D68, D69, D70: Field1 (none) -> newark,10M2940; Field2 (none) -> vendor1, smd w hem; Field3 (none) -> vendor2, thru w hem; Field4 (none) -> vendor2, smd w hem; Field5 (none) -> 1000,V; Field6 (none) -> 1,A; Field7 (none) -> x; Field8 (none) -> other,more,stuff
- R79: Field1 (none) -> newark38K0327,; Field2 (none) -> vendor1, smd w hem; Field3 (none) -> vendor2, thru w hem; Field4 (none) -> vendor2, smd w hem; Field5 (none) -> 1/4,W; Field6 (none) -> 5,%; Field7 (none) -> Carbon film; Field8 (none) -> other,more,stuff
- R80, R81, R82, R83, R84, R86: Field1 (none) -> newark,38K0327; Field2 (none) -> vendor1, smd w hem; Field3 (none) -> vendor2, thru w hem; Field4 (none) -> vendor2, smd w hem; Field5 (none) -> 1/4,W; Field6 (none) -> 5,%; Field7 (none) -> Carbon film; Field8 (none) -> other,more,stuff
- R85: Field1 (none) -> newark,38K0327; Field2 (none) -> vendor1, smd w hem; Field3 (none) -> vendor2, thru w hem; Field4 (none) -> vendor2, smd w hem; Field5 (none) -> 1/4,W; Field6 (none) -> 5,%; Field7 (none) -> carbon film; Field8 (none) -> other,more,stuff

Commit message: Implemented P&H, removed current sense circuitry, removed all unnecessary files from the repo
Parts:
- R?: renamed from R83; Field1 newark,38K0327 -> newark,72K6178; Field7 Carbon film -> Carbon Composition
- renumbered C44 to C?, C43 to C?, C42 to C?, C41 to C?, D69 to D?, D70 to D?, D67 to D?, D68 to D?, D65 to D?, D66 to D?, D63 to D?, D64 to D?, R82 to R?, R86 to R?, R81 to R?, R85 to R?, R80 to R?, R84 to R?, R79 to R?
Changed lines of the file:
@@
-EESchema Schematic File Version 2  date Fri 02 Jul 2010 05:44:26 PM ART
+EESchema Schematic File Version 2  date Sat 03 Jul 2010 10:49:02 AM ART
 LIBS:power
 LIBS:freeEMS_lib
@@
 EELAYER END
 $Descr A 11000 8500
-Sheet 23 41
+Sheet 1 41
 Title "freeEMS 1.0"
-Date "2 jul 2010"
-Rev "A.20"
+Date "3 jul 2010"
+Rev "A.07"
 Comp "diyefi.org"
 Comment1 "an_protect.sch"
@@
 Connection ~ 6500 2150
 $Comp
-L R R83
+L R R?
 U 1 1 489597C5
 P 3900 5450
-F 0 "R83" V 3980 5450 50  0000 C CNN
+F 0 "R?" V 3980 5450 50  0000 C CNN
 F 1 "1k" V 3900 5450 50  0000 C CNN
 F 2 "R4-SM0805" V 4080 5550 60  0001 C CNN
-F 4 "newark,38K0327" V 1130 2600 60  0001 C CNN "Field1"
-F 5 "vendor1, smd w hem" V 1130 2600 60  0001 C CNN "Field2"
-F 6 "vendor2, thru w hem" V 1130 2600 60  0001 C CNN "Field3"
-F 7 "vendor2, smd w hem" V 1130 2600 60  0001 C CNN "Field4"
-F 8 "1/4,W" V 1130 2600 60  0001 C CNN "Field5"
-F 9 "5,%" V 1130 2600 60  0001 C CNN "Field6"
-F 10 "Carbon film" V 1130 2600 60  0001 C CNN "Field7"
+F 4 "newark,72K6178" V 1130 2600 60  0001 C CNN "Field1"
+F 5 "vendor1, smd w hem" V 1130 2600 60  0001 C CNN "Field2"
+F 6 "vendor2, thru w hem" V 1130 2600 60  0001 C CNN "Field3"
+F 7 "vendor2, smd w hem" V 1130 2600 60  0001 C CNN "Field4"
+F 8 "1/4,W" V 1130 2600 60  0001 C CNN "Field5"
+F 9 "5,%" V 1130 2600 60  0001 C CNN "Field6"
+F 10 "Carbon Composition" V 1130 2600 60  0001 C CNN "Field7"
 F 11 "other,more,stuff" V 1130 2600 60  0001 C CNN "Field8"
 	1    3900 5450
@@
 $EndComp
 $Comp
-L GND #PWR038
+L GND #PWR?
 U 1 1 489597C4
 P 1950 5900
-F 0 "#PWR038" H 1950 5900 30  0001 C CNN
+F 0 "#PWR?" H 1950 5900 30  0001 C CNN
 F 1 "GND" H 1950 5830 30  0001 C CNN
 	1    1950 5900
@@
 $EndComp
 $Comp
-L DIODE D64
+L DIODE D?
 U 1 1 489597C3
 P 2600 5650
-F 0 "D64" H 2600 5750 40  0000 C CNN
+F 0 "D?" H 2600 5750 40  0000 C CNN
 F 1 "1N4148" H 2600 5550 40  0000 C CNN
 F 2 "D4-SMB" V 1130 2600 60  0001 C CNN
@@
 $EndComp
 $Comp
-L C C41
+L C C?
 U 1 1 489597C2
 P 3150 5650
-F 0 "C41" H 3200 5750 50  0000 L CNN
+F 0 "C?" H 3200 5750 50  0000 L CNN
 F 1 "100nf" H 3200 5550 50  0000 L CNN
 F 2 "C1V7" V 1130 2600 60  0001 C CNN
@@
 $EndComp
 $Comp
-L R R79
+L R R?
 U 1 1 489597C1
 P 2200 5450
-F 0 "R79" V 2280 5450 50  0000 C CNN
+F 0 "R?" V 2280 5450 50  0000 C CNN
 F 1 "1k" V 2200 5450 50  0000 C CNN
 F 2 "R4-SM0805" V 2380 5550 60  0001 C CNN
@@
 $EndComp
 $Comp
-L DIODE D63
+L DIODE D?
 U 1 1 489597C0
 P 2600 5050
-F 0 "D63" H 2600 5150 40  0000 C CNN
+F 0 "D?" H 2600 5150 40  0000 C CNN
 F 1 "1N4148" H 2600 4950 40  0000 C CNN
 F 2 "D4-SMB" V 1130 2600 60  0001 C CNN
@@
 analog_sensor_out_4
 $Comp
-L R R84
+L R R?
 U 1 1 489597BF
 P 3950 4050
-F 0 "R84" V 4030 4050 50  0000 C CNN
+F 0 "R?" V 4030 4050 50  0000 C CNN
 F 1 "1k" V 3950 4050 50  0000 C CNN
 F 2 "R4-SM0805" V 4130 4150 60  0001 C CNN
@@
 $EndComp
 $Comp
-L GND #PWR039
+L GND #PWR?
 U 1 1 489597BE
 P 2000 4500
-F 0 "#PWR039" H 2000 4500 30  0001 C CNN
+F 0 "#PWR?" H 2000 4500 30  0001 C CNN
 F 1 "GND" H 2000 4430 30  0001 C CNN
 	1    2000 4500
@@
 $EndComp
 $Comp
-L DIODE D66
+L DIODE D?
 U 1 1 489597BD
 P 2650 4250
-F 0 "D66" H 2650 4350 40  0000 C CNN
+F 0 "D?" H 2650 4350 40  0000 C CNN
 F 1 "1N4148" H 2650 4150 40  0000 C CNN
 F 2 "D4-SMB" V 1130 2600 60  0001 C CNN
@@
 $EndComp
 $Comp
-L C C42
+L C C?
 U 1 1 489597BC
 P 3200 4250
-F 0 "C42" H 3250 4350 50  0000 L CNN
+F 0 "C?" H 3250 4350 50  0000 L CNN
 F 1 "100nf" H 3250 4150 50  0000 L CNN
 F 2 "C1V7" V 1130 2600 60  0001 C CNN
@@
 $EndComp
 $Comp
-L R R80
+L R R?
 U 1 1 489597BB
 P 2250 4050
-F 0 "R80" V 2330 4050 50  0000 C CNN
+F 0 "R?" V 2330 4050 50  0000 C CNN
 F 1 "1k" V 2250 4050 50  0000 C CNN
 F 2 "R4-SM0805" V 2430 4150 60  0001 C CNN
@@
 $EndComp
 $Comp
-L DIODE D65
+L DIODE D?
 U 1 1 489597BA
 P 2650 3650
-F 0 "D65" H 2650 3750 40  0000 C CNN
+F 0 "D?" H 2650 3750 40  0000 C CNN
 F 1 "1N4148" H 2650 3550 40  0000 C CNN
 F 2 "D4-SMB" V 1130 2600 60  0001 C CNN
@@
 analog_sensor_out_3
 $Comp
-L R R85
+L R R?
 U 1 1 489597B9
 P 4000 2750
-F 0 "R85" V 4080 2750 50  0000 C CNN
+F 0 "R?" V 4080 2750 50  0000 C CNN
 F 1 "1k" V 4000 2750 50  0000 C CNN
 F 2 "R4-SM0805" V 4180 2850 60  0001 C CNN
@@
 $EndComp
 $Comp
-L GND #PWR040
+L GND #PWR?
 U 1 1 489597B8
 P 2050 3200
-F 0 "#PWR040" H 2050 3200 30  0001 C CNN
+F 0 "#PWR?" H 2050 3200 30  0001 C CNN
 F 1 "GND" H 2050 3130 30  0001 C CNN
 	1    2050 3200
@@
 $EndComp
 $Comp
-L DIODE D68
+L DIODE D?
 U 1 1 489597B7
 P 2700 2950
-F 0 "D68" H 2700 3050 40  0000 C CNN
+F 0 "D?" H 2700 3050 40  0000 C CNN
 F 1 "1N4148" H 2700 2850 40  0000 C CNN
 F 2 "D4-SMB" V 1130 2600 60  0001 C CNN
@@
 $EndComp
 $Comp
-L C C43
+L C C?
 U 1 1 489597B6
 P 3250 2950
-F 0 "C43" H 3300 3050 50  0000 L CNN
+F 0 "C?" H 3300 3050 50  0000 L CNN
 F 1 "100nf" H 3300 2850 50  0000 L CNN
 F 2 "C1V7" V 1130 2600 60  0001 C CNN
@@
 $EndComp
 $Comp
-L R R81
+L R R?
 U 1 1 489597B5
 P 2300 2750
-F 0 "R81" V 2380 2750 50  0000 C CNN
+F 0 "R?" V 2380 2750 50  0000 C CNN
 F 1 "1k" V 2300 2750 50  0000 C CNN
 F 2 "R4-SM0805" V 2480 2850 60  0001 C CNN
@@
 $EndComp
 $Comp
-L DIODE D67
+L DIODE D?
 U 1 1 489597B4
 P 2700 2350
-F 0 "D67" H 2700 2450 40  0000 C CNN
+F 0 "D?" H 2700 2450 40  0000 C CNN
 F 1 "1N4148" H 2700 2250 40  0000 C CNN
 F 2 "D4-SMB" V 1130 2600 60  0001 C CNN
@@
 analog_sensor_out_2
 $Comp
-L R R86
+L R R?
 U 1 1 488CCA4A
 P 4050 1400
-F 0 "R86" V 4130 1400 50  0000 C CNN
+F 0 "R?" V 4130 1400 50  0000 C CNN
 F 1 "1k" V 4050 1400 50  0000 C CNN
 F 2 "R4-SM0805" V 4230 1500 60  0001 C CNN
@@
 $EndComp
 $Comp
-L GND #PWR041
+L GND #PWR?
 U 1 1 486F8C14
 P 2100 1850
-F 0 "#PWR041" H 2100 1850 30  0001 C CNN
+F 0 "#PWR?" H 2100 1850 30  0001 C CNN
 F 1 "GND" H 2100 1780 30  0001 C CNN
 	1    2100 1850
@@
 $EndComp
 $Comp
-L DIODE D70
+L DIODE D?
 U 1 1 486F8B98
 P 2750 1600
-F 0 "D70" H 2750 1700 40  0000 C CNN
+F 0 "D?" H 2750 1700 40  0000 C CNN
 F 1 "1N4148" H 2750 1500 40  0000 C CNN
 F 2 "D4-SMB" V 1130 2600 60  0001 C CNN
@@
 $EndComp
 $Comp
-L C C44
+L C C?
 U 1 1 486F8B93
 P 3300 1600
-F 0 "C44" H 3350 1700 50  0000 L CNN
+F 0 "C?" H 3350 1700 50  0000 L CNN
 F 1 "100nf" H 3350 1500 50  0000 L CNN
 F 2 "C1V7" V 1130 2600 60  0001 C CNN
@@
 $EndComp
 $Comp
-L R R82
+L R R?
 U 1 1 486F8B82
 P 2350 1400
-F 0 "R82" V 2430 1400 50  0000 C CNN
+F 0 "R?" V 2430 1400 50  0000 C CNN
 F 1 "1k" V 2350 1400 50  0000 C CNN
 F 2 "R4-SM0805" V 2530 1500 60  0001 C CNN
@@
 $EndComp
 $Comp
-L DIODE D69
+L DIODE D?
 U 1 1 486F8B5C
 P 2750 1000
-F 0 "D69" H 2750 1100 40  0000 C CNN
+F 0 "D?" H 2750 1100 40  0000 C CNN
 F 1 "1N4148" H 2750 900 40  0000 C CNN
 F 2 "D4-SMB" V 1130 2600 60  0001 C CNN

Commit message: Corrected ERC errors by fixing the custom FreeEMS components pinouts
Parts:
- removed C? (x2): 100nf, C1V7, symbol C
- removed D? (x4): 1N4148, D4-SMB, symbol DIODE
- removed R? (x3): 1k, R4-SM0805, symbol R
- added C33, C34: 100nf, C1V7, symbol C
- added D40, D41, D42, D43: 1N4148, D4-SMB, symbol DIODE
- added R54, R55, R60: 1k, R4-SM0805, symbol R
- gave numbers to parts that had none: 11
Connections:
- net GND: now also C33.2, C34.2, D40.1 (A), D42.1 (A)
- net analog_sensor_in_2: now also R55.2
- net analog_sensor_in_3: now also R54.2
- net analog_sensor_out_1: now also R60.1
- net analog_sensor_vcc: now also D41.2 (K), D43.2 (K)
- net at C35.1, D44.2 (K), R56.1: now also D43.1 (A), R60.2
- net at R59.2: now also C34.1, D41.1 (A), D42.2 (K), R55.1
- net at D39.1 (A), R58.2: now also C33.1, D40.2 (K), R54.1
Changed lines of the file:
@@
-EESchema Schematic File Version 2  date Sat 03 Jul 2010 10:49:02 AM ART
+EESchema Schematic File Version 2  date Sat 03 Jul 2010 12:32:24 PM ART
 LIBS:power
 LIBS:freeEMS_lib
@@
 Connection ~ 6500 2150
 $Comp
-L R R?
+L R R57
 U 1 1 489597C5
 P 3900 5450
-F 0 "R?" V 3980 5450 50  0000 C CNN
+F 0 "R57" V 3980 5450 50  0000 C CNN
 F 1 "1k" V 3900 5450 50  0000 C CNN
 F 2 "R4-SM0805" V 4080 5550 60  0001 C CNN
@@
 $EndComp
 $Comp
-L GND #PWR?
+L GND #PWR059
 U 1 1 489597C4
 P 1950 5900
-F 0 "#PWR?" H 1950 5900 30  0001 C CNN
+F 0 "#PWR059" H 1950 5900 30  0001 C CNN
 F 1 "GND" H 1950 5830 30  0001 C CNN
 	1    1950 5900
@@
 $EndComp
 $Comp
-L DIODE D?
+L DIODE D38
 U 1 1 489597C3
 P 2600 5650
-F 0 "D?" H 2600 5750 40  0000 C CNN
+F 0 "D38" H 2600 5750 40  0000 C CNN
 F 1 "1N4148" H 2600 5550 40  0000 C CNN
 F 2 "D4-SMB" V 1130 2600 60  0001 C CNN
@@
 $EndComp
 $Comp
-L C C?
+L C C32
 U 1 1 489597C2
 P 3150 5650
-F 0 "C?" H 3200 5750 50  0000 L CNN
+F 0 "C32" H 3200 5750 50  0000 L CNN
 F 1 "100nf" H 3200 5550 50  0000 L CNN
 F 2 "C1V7" V 1130 2600 60  0001 C CNN
@@
 $EndComp
 $Comp
-L R R?
+L R R53
 U 1 1 489597C1
 P 2200 5450
-F 0 "R?" V 2280 5450 50  0000 C CNN
+F 0 "R53" V 2280 5450 50  0000 C CNN
 F 1 "1k" V 2200 5450 50  0000 C CNN
 F 2 "R4-SM0805" V 2380 5550 60  0001 C CNN
@@
 $EndComp
 $Comp
-L DIODE D?
+L DIODE D37
 U 1 1 489597C0
 P 2600 5050
-F 0 "D?" H 2600 5150 40  0000 C CNN
+F 0 "D37" H 2600 5150 40  0000 C CNN
 F 1 "1N4148" H 2600 4950 40  0000 C CNN
 F 2 "D4-SMB" V 1130 2600 60  0001 C CNN
@@
 analog_sensor_out_4
 $Comp
-L R R?
+L R R58
 U 1 1 489597BF
 P 3950 4050
-F 0 "R?" V 4030 4050 50  0000 C CNN
+F 0 "R58" V 4030 4050 50  0000 C CNN
 F 1 "1k" V 3950 4050 50  0000 C CNN
 F 2 "R4-SM0805" V 4130 4150 60  0001 C CNN
@@
 $EndComp
 $Comp
-L GND #PWR?
+L GND #PWR060
 U 1 1 489597BE
 P 2000 4500
-F 0 "#PWR?" H 2000 4500 30  0001 C CNN
+F 0 "#PWR060" H 2000 4500 30  0001 C CNN
 F 1 "GND" H 2000 4430 30  0001 C CNN
 	1    2000 4500
@@
 $EndComp
 $Comp
-L DIODE D?
-U 1 1 489597BD
+L DIODE D40
+U 1 1 4C2F52F5
 P 2650 4250
-F 0 "D?" H 2650 4350 40  0000 C CNN
+F 0 "D40" H 2650 4350 40  0000 C CNN
 F 1 "1N4148" H 2650 4150 40  0000 C CNN
 F 2 "D4-SMB" V 1130 2600 60  0001 C CNN
@@
 $EndComp
 $Comp
-L C C?
-U 1 1 489597BC
+L C C33
+U 1 1 4C2F52F4
 P 3200 4250
-F 0 "C?" H 3250 4350 50  0000 L CNN
+F 0 "C33" H 3250 4350 50  0000 L CNN
 F 1 "100nf" H 3250 4150 50  0000 L CNN
 F 2 "C1V7" V 1130 2600 60  0001 C CNN
@@
 $EndComp
 $Comp
-L R R?
-U 1 1 489597BB
+L R R54
+U 1 1 4C2F52F3
 P 2250 4050
-F 0 "R?" V 2330 4050 50  0000 C CNN
+F 0 "R54" V 2330 4050 50  0000 C CNN
 F 1 "1k" V 2250 4050 50  0000 C CNN
 F 2 "R4-SM0805" V 2430 4150 60  0001 C CNN
@@
 $EndComp
 $Comp
-L DIODE D?
+L DIODE D39
 U 1 1 489597BA
 P 2650 3650
-F 0 "D?" H 2650 3750 40  0000 C CNN
+F 0 "D39" H 2650 3750 40  0000 C CNN
 F 1 "1N4148" H 2650 3550 40  0000 C CNN
 F 2 "D4-SMB" V 1130 2600 60  0001 C CNN
@@
 analog_sensor_out_3
 $Comp
-L R R?
+L R R59
 U 1 1 489597B9
 P 4000 2750
-F 0 "R?" V 4080 2750 50  0000 C CNN
+F 0 "R59" V 4080 2750 50  0000 C CNN
 F 1 "1k" V 4000 2750 50  0000 C CNN
 F 2 "R4-SM0805" V 4180 2850 60  0001 C CNN
@@
 $EndComp
 $Comp
-L GND #PWR?
-U 1 1 489597B8
+L GND #PWR061
+U 1 1 4C2F52F0
 P 2050 3200
-F 0 "#PWR?" H 2050 3200 30  0001 C CNN
+F 0 "#PWR061" H 2050 3200 30  0001 C CNN
 F 1 "GND" H 2050 3130 30  0001 C CNN
 	1    2050 3200
@@
 $EndComp
 $Comp
-L DIODE D?
-U 1 1 489597B7
+L DIODE D42
+U 1 1 4C2F52EF
 P 2700 2950
-F 0 "D?" H 2700 3050 40  0000 C CNN
+F 0 "D42" H 2700 3050 40  0000 C CNN
 F 1 "1N4148" H 2700 2850 40  0000 C CNN
 F 2 "D4-SMB" V 1130 2600 60  0001 C CNN
@@
 $EndComp
 $Comp
-L C C?
-U 1 1 489597B6
+L C C34
+U 1 1 4C2F52EE
 P 3250 2950
-F 0 "C?" H 3300 3050 50  0000 L CNN
+F 0 "C34" H 3300 3050 50  0000 L CNN
 F 1 "100nf" H 3300 2850 50  0000 L CNN
 F 2 "C1V7" V 1130 2600 60  0001 C CNN
@@
 $EndComp
 $Comp
-L R R?
-U 1 1 489597B5
+L R R55
+U 1 1 4C2F52ED
 P 2300 2750
-F 0 "R?" V 2380 2750 50  0000 C CNN
+F 0 "R55" V 2380 2750 50  0000 C CNN
 F 1 "1k" V 2300 2750 50  0000 C CNN
 F 2 "R4-SM0805" V 2480 2850 60  0001 C CNN
@@
 $EndComp
 $Comp
-L DIODE D?
-U 1 1 489597B4
+L DIODE D41
+U 1 1 4C2F52EC
 P 2700 2350
-F 0 "D?" H 2700 2450 40  0000 C CNN
+F 0 "D41" H 2700 2450 40  0000 C CNN
 F 1 "1N4148" H 2700 2250 40  0000 C CNN
 F 2 "D4-SMB" V 1130 2600 60  0001 C CNN
@@
 analog_sensor_out_2
 $Comp
-L R R?
-U 1 1 488CCA4A
+L R R60
+U 1 1 4C2F52DC
 P 4050 1400
-F 0 "R?" V 4130 1400 50  0000 C CNN
+F 0 "R60" V 4130 1400 50  0000 C CNN
 F 1 "1k" V 4050 1400 50  0000 C CNN
 F 2 "R4-SM0805" V 4230 1500 60  0001 C CNN
@@
 $EndComp
 $Comp
-L GND #PWR?
+L GND #PWR062
 U 1 1 486F8C14
 P 2100 1850
-F 0 "#PWR?" H 2100 1850 30  0001 C CNN
+F 0 "#PWR062" H 2100 1850 30  0001 C CNN
 F 1 "GND" H 2100 1780 30  0001 C CNN
 	1    2100 1850
@@
 $EndComp
 $Comp
-L DIODE D?
+L DIODE D44
 U 1 1 486F8B98
 P 2750 1600
-F 0 "D?" H 2750 1700 40  0000 C CNN
+F 0 "D44" H 2750 1700 40  0000 C CNN
 F 1 "1N4148" H 2750 1500 40  0000 C CNN
 F 2 "D4-SMB" V 1130 2600 60  0001 C CNN
@@
 $EndComp
 $Comp
-L C C?
+L C C35
 U 1 1 486F8B93
 P 3300 1600
-F 0 "C?" H 3350 1700 50  0000 L CNN
+F 0 "C35" H 3350 1700 50  0000 L CNN
 F 1 "100nf" H 3350 1500 50  0000 L CNN
 F 2 "C1V7" V 1130 2600 60  0001 C CNN
@@
 $EndComp
 $Comp
-L R R?
+L R R56
 U 1 1 486F8B82
 P 2350 1400
-F 0 "R?" V 2430 1400 50  0000 C CNN
+F 0 "R56" V 2430 1400 50  0000 C CNN
 F 1 "1k" V 2350 1400 50  0000 C CNN
 F 2 "R4-SM0805" V 2530 1500 60  0001 C CNN
@@
 $EndComp
 $Comp
-L DIODE D?
-U 1 1 486F8B5C
+L DIODE D43
+U 1 1 4C2F52A4
 P 2750 1000
-F 0 "D?" H 2750 1100 40  0000 C CNN
+F 0 "D43" H 2750 1100 40  0000 C CNN
 F 1 "1N4148" H 2750 900 40  0000 C CNN
 F 2 "D4-SMB" V 1130 2600 60  0001 C CNN

Commit message: MAP circuit compatible with external sensors. Baro is left untouched
Parts:
- removed D38, D40, D42, D44: 1N4148, D4-SMB, symbol DIODE
- added D38, D40, D42, D44: SCHOTTKY, SOD-123, symbol DIODESCH
Connections:
- net GND: now also D38.1 (A), D40.1 (A), D42.1 (A), D44.1 (A)
- net at C35.1, D43.1 (A), R56.1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: now also D44.2 (K)
- net at C34.1, D41.1 (A), R55.1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: now also D42.2 (K)
- net at C33.1, D39.1 (A), R54.1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: now also D40.2 (K)
- net at C32.1, D37.1 (A), R53.1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: now also D38.2 (K)
Changed lines of the file:
@@
-EESchema Schematic File Version 2  date Thu 22 Jul 2010 10:06:33 AM ART
+EESchema Schematic File Version 2  date Sat 24 Jul 2010 11:01:40 AM ART
 LIBS:power
 LIBS:freeEMS_lib
@@
 EELAYER END
 $Descr A 11000 8500
-Sheet 1 41
+Sheet 29 41
 Title "freeEMS 1.0"
-Date "22 jul 2010"
+Date "24 jul 2010"
 Rev "A.07"
 Comp "diyefi.org"
@@
 Comment4 ""
 $EndDescr
+$Comp
+L DIODESCH D38
+U 1 1 4C4973C4
+P 2600 5650
+F 0 "D38" H 2600 5750 40  0000 C CNN
+F 1 "SCHOTTKY" H 2600 5550 40  0000 C CNN
+F 2 "SOD-123" H 2600 5650 60  0001 C CNN
+	1    2600 5650
+	0    -1   -1   0
+$EndComp
+$Comp
+L DIODESCH D40
+U 1 1 4C4973C0
+P 2650 4250
+F 0 "D40" H 2650 4350 40  0000 C CNN
+F 1 "SCHOTTKY" H 2650 4150 40  0000 C CNN
+F 2 "SOD-123" H 2650 4250 60  0001 C CNN
+	1    2650 4250
+	0    -1   -1   0
+$EndComp
+$Comp
+L DIODESCH D42
+U 1 1 4C4973B6
+P 2700 2950
+F 0 "D42" H 2700 3050 40  0000 C CNN
+F 1 "SCHOTTKY" H 2700 2850 40  0000 C CNN
+F 2 "SOD-123" H 2700 2950 60  0001 C CNN
+	1    2700 2950
+	0    -1   -1   0
+$EndComp
+$Comp
+L DIODESCH D44
+U 1 1 4C4973B0
+P 2750 1600
+F 0 "D44" H 2750 1700 40  0000 C CNN
+F 1 "SCHOTTKY" H 2750 1500 40  0000 C CNN
+F 2 "SOD-123" H 2750 1600 60  0001 C CNN
+	1    2750 1600
+	0    -1   -1   0
+$EndComp
 Connection ~ 2750 800
 Wire Wire Line
@@
 $EndComp
 $Comp
-L DIODE D38
-U 1 1 489597C3
-P 2600 5650
-F 0 "D38" H 2600 5750 40  0000 C CNN
-F 1 "1N4148" H 2600 5550 40  0000 C CNN
-F 2 "D4-SMB" V 1130 2600 60  0001 C CNN
-F 4 "newark,10M2940" V 1130 2600 60  0001 C CNN "Field1"
-F 5 "vendor1, smd w hem" V 1130 2600 60  0001 C CNN "Field2"
-F 6 "vendor2, thru w hem" V 1130 2600 60  0001 C CNN "Field3"
-F 7 "vendor2, smd w hem" V 1130 2600 60  0001 C CNN "Field4"
-F 8 "1000,V" V 1130 2600 60  0001 C CNN "Field5"
-F 9 "1,A" V 1130 2600 60  0001 C CNN "Field6"
-F 10 "x" V 1130 2600 60  0001 C CNN "Field7"
-F 11 "other,more,stuff" V 1130 2600 60  0001 C CNN "Field8"
-	1    2600 5650
-	0    -1   -1   0
-$EndComp
-$Comp
 L C C32
 U 1 1 489597C2
@@
 $EndComp
 $Comp
-L DIODE D40
-U 1 1 4C2F52F5
-P 2650 4250
-F 0 "D40" H 2650 4350 40  0000 C CNN
-F 1 "1N4148" H 2650 4150 40  0000 C CNN
-F 2 "D4-SMB" V 1130 2600 60  0001 C CNN
-F 4 "newark,10M2940" V 1130 2600 60  0001 C CNN "Field1"
-F 5 "vendor1, smd w hem" V 1130 2600 60  0001 C CNN "Field2"
-F 6 "vendor2, thru w hem" V 1130 2600 60  0001 C CNN "Field3"
-F 7 "vendor2, smd w hem" V 1130 2600 60  0001 C CNN "Field4"
-F 8 "1000,V" V 1130 2600 60  0001 C CNN "Field5"
-F 9 "1,A" V 1130 2600 60  0001 C CNN "Field6"
-F 10 "x" V 1130 2600 60  0001 C CNN "Field7"
-F 11 "other,more,stuff" V 1130 2600 60  0001 C CNN "Field8"
-	1    2650 4250
-	0    -1   -1   0
-$EndComp
-$Comp
 L C C33
 U 1 1 4C2F52F4
@@
 $EndComp
 $Comp
-L DIODE D42
-U 1 1 4C2F52EF
-P 2700 2950
-F 0 "D42" H 2700 3050 40  0000 C CNN
-F 1 "1N4148" H 2700 2850 40  0000 C CNN
-F 2 "D4-SMB" V 1130 2600 60  0001 C CNN
-F 4 "newark,10M2940" V 1130 2600 60  0001 C CNN "Field1"
-F 5 "vendor1, smd w hem" V 1130 2600 60  0001 C CNN "Field2"
-F 6 "vendor2, thru w hem" V 1130 2600 60  0001 C CNN "Field3"
-F 7 "vendor2, smd w hem" V 1130 2600 60  0001 C CNN "Field4"
-F 8 "1000,V" V 1130 2600 60  0001 C CNN "Field5"
-F 9 "1,A" V 1130 2600 60  0001 C CNN "Field6"
-F 10 "x" V 1130 2600 60  0001 C CNN "Field7"
-F 11 "other,more,stuff" V 1130 2600 60  0001 C CNN "Field8"
-	1    2700 2950
-	0    -1   -1   0
-$EndComp
-$Comp
 L C C34
 U 1 1 4C2F52EE
@@
 $EndComp
 $Comp
-L DIODE D44
-U 1 1 486F8B98
-P 2750 1600
-F 0 "D44" H 2750 1700 40  0000 C CNN
-F 1 "1N4148" H 2750 1500 40  0000 C CNN
-F 2 "D4-SMB" V 1130 2600 60  0001 C CNN
-F 4 "newark,10M2940" V 1130 2600 60  0001 C CNN "Field1"
-F 5 "vendor1, smd w hem" V 1130 2600 60  0001 C CNN "Field2"
-F 6 "vendor2, thru w hem" V 1130 2600 60  0001 C CNN "Field3"
-F 7 "vendor2, smd w hem" V 1130 2600 60  0001 C CNN "Field4"
-F 8 "1000,V" V 1130 2600 60  0001 C CNN "Field5"
-F 9 "1,A" V 1130 2600 60  0001 C CNN "Field6"
-F 10 "x" V 1130 2600 60  0001 C CNN "Field7"
-F 11 "other,more,stuff" V 1130 2600 60  0001 C CNN "Field8"
-	1    2750 1600
-	0    -1   -1   0
-$EndComp
-$Comp
