File: an_protect4.sch (KiCad schematic (older format))
At the start: 20 parts

Commit message: 4 temperature inputs and 2 extra aux analog inputs.
Parts:
- removed C34, C35: 100nf, C1V7, symbol C
- removed D39: 1N4148, D4-SMB, symbol DIODE
- removed R56, R57, R58: 1k, R4-SM0805, symbol R
- added C91, C92: 100nf, C1V7, symbol C
- added D68: 1N4148, D4-SMB, symbol DIODE
- added R170, R171, R172: 1k, R4-SM0805, symbol R
- renumbered C32 to C89, C33 to C90, D37 to D66, D38 to D67, D40 to D69, D41 to D70, D42 to D71, D43 to D72, D44 to D73, R53 to R167, R54 to R168, R55 to R169, R59 to R173, R60 to R174
Connections:
- net GND: now also C91.2, C92.2
- net analog_sensor_in_1: now also R170.2
- net analog_sensor_out_3: now also R172.1
- net analog_sensor_out_4: now also R171.1
- net analog_sensor_vcc: now also D68.2 (K)
- net at D72.1 (A), D73.2 (K), R174.2: now also C92.1, R170.1
- net at D70.1 (A), D71.2 (K), R169.1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: now also C91.1
- net at C90.1, D69.2 (K), R168.1: now also D68.1 (A), R172.2
- net at C89.1, D66.1 (A), D67.2 (K)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: now also R171.2
Changed lines of the file:
@@
-EESchema Schematic File Version 2  date Sat 24 Jul 2010 11:01:40 AM ART
+EESchema Schematic File Version 2  date Sun 25 Jul 2010 03:39:31 PM ART
 LIBS:power
 LIBS:freeEMS_lib
@@
 EELAYER END
 $Descr A 11000 8500
-Sheet 29 41
+Sheet 5 46
 Title "freeEMS 1.0"
-Date "24 jul 2010"
+Date "25 jul 2010"
 Rev "A.07"
 Comp "diyefi.org"
@@
 $EndDescr
 $Comp
-L DIODESCH D38
+L DIODESCH D67
 U 1 1 4C4973C4
 P 2600 5650
-F 0 "D38" H 2600 5750 40  0000 C CNN
+AR Path="/4C4C6618/4C4973C4" Ref="D67"  Part="1"
+AR Path="/4C2E1E7D/4C4973C4" Ref="D59"  Part="1"
+F 0 "D67" H 2600 5750 40  0000 C CNN
 F 1 "SCHOTTKY" H 2600 5550 40  0000 C CNN
 F 2 "SOD-123" H 2600 5650 60  0001 C CNN
@@
 $EndComp
 $Comp
-L DIODESCH D40
+L DIODESCH D69
 U 1 1 4C4973C0
 P 2650 4250
-F 0 "D40" H 2650 4350 40  0000 C CNN
+AR Path="/4C4C6618/4C4973C0" Ref="D69"  Part="1"
+AR Path="/4C2E1E7D/4C4973C0" Ref="D61"  Part="1"
+F 0 "D69" H 2650 4350 40  0000 C CNN
 F 1 "SCHOTTKY" H 2650 4150 40  0000 C CNN
 F 2 "SOD-123" H 2650 4250 60  0001 C CNN
@@
 $EndComp
 $Comp
-L DIODESCH D42
+L DIODESCH D71
 U 1 1 4C4973B6
 P 2700 2950
-F 0 "D42" H 2700 3050 40  0000 C CNN
+AR Path="/4C4C6618/4C4973B6" Ref="D71"  Part="1"
+AR Path="/4C2E1E7D/4C4973B6" Ref="D63"  Part="1"
+F 0 "D71" H 2700 3050 40  0000 C CNN
 F 1 "SCHOTTKY" H 2700 2850 40  0000 C CNN
 F 2 "SOD-123" H 2700 2950 60  0001 C CNN
@@
 $EndComp
 $Comp
-L DIODESCH D44
+L DIODESCH D73
 U 1 1 4C4973B0
 P 2750 1600
-F 0 "D44" H 2750 1700 40  0000 C CNN
+AR Path="/4C4C6618/4C4973B0" Ref="D73"  Part="1"
+AR Path="/4C2E1E7D/4C4973B0" Ref="D65"  Part="1"
+F 0 "D73" H 2750 1700 40  0000 C CNN
 F 1 "SCHOTTKY" H 2750 1500 40  0000 C CNN
 F 2 "SOD-123" H 2750 1600 60  0001 C CNN
@@
 Connection ~ 6500 2150
 $Comp
-L R R57
-U 1 1 489597C5
+L R R171
+U 1 1 4C4C7B57
 P 3900 5450
-F 0 "R57" V 3980 5450 50  0000 C CNN
+AR Path="/4C4C6618/4C4C7B57" Ref="R171"  Part="1"
+AR Path="/4C2E1E7D/4C4C7B57" Ref="R163"  Part="1"
+F 0 "R171" V 3980 5450 50  0000 C CNN
 F 1 "1k" V 3900 5450 50  0000 C CNN
 F 2 "R4-SM0805" V 4080 5550 60  0001 C CNN
@@
 $EndComp
 $Comp
-L GND #PWR059
+L GND #PWR72
 U 1 1 489597C4
 P 1950 5900
-F 0 "#PWR059" H 1950 5900 30  0001 C CNN
+AR Path="/4C4C6618/489597C4" Ref="#PWR72"  Part="1"
+AR Path="/4C2E1E7D/489597C4" Ref="#PWR38"  Part="1"
+F 0 "#PWR72" H 1950 5900 30  0001 C CNN
 F 1 "GND" H 1950 5830 30  0001 C CNN
 	1    1950 5900
@@
 $EndComp
 $Comp
-L C C32
+L C C89
 U 1 1 489597C2
 P 3150 5650
-F 0 "C32" H 3200 5750 50  0000 L CNN
+AR Path="/4C4C6618/489597C2" Ref="C89"  Part="1"
+AR Path="/4C2E1E7D/489597C2" Ref="C85"  Part="1"
+F 0 "C89" H 3200 5750 50  0000 L CNN
 F 1 "100nf" H 3200 5550 50  0000 L CNN
 F 2 "C1V7" V 1130 2600 60  0001 C CNN
@@
 $EndComp
 $Comp
-L R R53
+L R R167
 U 1 1 489597C1
 P 2200 5450
-F 0 "R53" V 2280 5450 50  0000 C CNN
+AR Path="/4C4C6618/489597C1" Ref="R167"  Part="1"
+AR Path="/4C2E1E7D/489597C1" Ref="R159"  Part="1"
+F 0 "R167" V 2280 5450 50  0000 C CNN
 F 1 "1k" V 2200 5450 50  0000 C CNN
 F 2 "R4-SM0805" V 2380 5550 60  0001 C CNN
@@
 $EndComp
 $Comp
-L DIODE D37
+L DIODE D66
 U 1 1 489597C0
 P 2600 5050
-F 0 "D37" H 2600 5150 40  0000 C CNN
+AR Path="/4C4C6618/489597C0" Ref="D66"  Part="1"
+AR Path="/4C2E1E7D/489597C0" Ref="D58"  Part="1"
+F 0 "D66" H 2600 5150 40  0000 C CNN
 F 1 "1N4148" H 2600 4950 40  0000 C CNN
 F 2 "D4-SMB" V 1130 2600 60  0001 C CNN
@@
 analog_sensor_out_4
 $Comp
-L R R58
-U 1 1 489597BF
+L R R172
+U 1 1 4C4C7B52
 P 3950 4050
-F 0 "R58" V 4030 4050 50  0000 C CNN
+AR Path="/4C4C6618/4C4C7B52" Ref="R172"  Part="1"
+AR Path="/4C2E1E7D/4C4C7B52" Ref="R164"  Part="1"
+F 0 "R172" V 4030 4050 50  0000 C CNN
 F 1 "1k" V 3950 4050 50  0000 C CNN
 F 2 "R4-SM0805" V 4130 4150 60  0001 C CNN
@@
 $EndComp
 $Comp
-L GND #PWR060
-U 1 1 489597BE
+L GND #PWR73
+U 1 1 4C4C7B51
 P 2000 4500
-F 0 "#PWR060" H 2000 4500 30  0001 C CNN
+AR Path="/4C4C6618/4C4C7B51" Ref="#PWR73"  Part="1"
+AR Path="/4C2E1E7D/4C4C7B51" Ref="#PWR39"  Part="1"
+F 0 "#PWR73" H 2000 4500 30  0001 C CNN
 F 1 "GND" H 2000 4430 30  0001 C CNN
 	1    2000 4500
@@
 $EndComp
 $Comp
-L C C33
+L C C90
 U 1 1 4C2F52F4
 P 3200 4250
-F 0 "C33" H 3250 4350 50  0000 L CNN
+AR Path="/4C4C6618/4C2F52F4" Ref="C90"  Part="1"
+AR Path="/4C2E1E7D/4C2F52F4" Ref="C86"  Part="1"
+F 0 "C90" H 3250 4350 50  0000 L CNN
 F 1 "100nf" H 3250 4150 50  0000 L CNN
 F 2 "C1V7" V 1130 2600 60  0001 C CNN
@@
 $EndComp
 $Comp
-L R R54
+L R R168
 U 1 1 4C2F52F3
 P 2250 4050
-F 0 "R54" V 2330 4050 50  0000 C CNN
+AR Path="/4C4C6618/4C2F52F3" Ref="R168"  Part="1"
+AR Path="/4C2E1E7D/4C2F52F3" Ref="R160"  Part="1"
+F 0 "R168" V 2330 4050 50  0000 C CNN
 F 1 "1k" V 2250 4050 50  0000 C CNN
 F 2 "R4-SM0805" V 2430 4150 60  0001 C CNN
@@
 $EndComp
 $Comp
-L DIODE D39
-U 1 1 489597BA
+L DIODE D68
+U 1 1 4C4C7B50
 P 2650 3650
-F 0 "D39" H 2650 3750 40  0000 C CNN
+AR Path="/4C4C6618/4C4C7B50" Ref="D68"  Part="1"
+AR Path="/4C2E1E7D/4C4C7B50" Ref="D60"  Part="1"
+F 0 "D68" H 2650 3750 40  0000 C CNN
 F 1 "1N4148" H 2650 3550 40  0000 C CNN
 F 2 "D4-SMB" V 1130 2600 60  0001 C CNN
@@
 analog_sensor_out_3
 $Comp
-L R R59
+L R R173
 U 1 1 489597B9
 P 4000 2750
-F 0 "R59" V 4080 2750 50  0000 C CNN
+AR Path="/4C4C6618/489597B9" Ref="R173"  Part="1"
+AR Path="/4C2E1E7D/489597B9" Ref="R165"  Part="1"
+F 0 "R173" V 4080 2750 50  0000 C CNN
 F 1 "1k" V 4000 2750 50  0000 C CNN
 F 2 "R4-SM0805" V 4180 2850 60  0001 C CNN
@@
 $EndComp
 $Comp
-L GND #PWR061
+L GND #PWR74
 U 1 1 4C2F52F0
 P 2050 3200
-F 0 "#PWR061" H 2050 3200 30  0001 C CNN
+AR Path="/4C4C6618/4C2F52F0" Ref="#PWR74"  Part="1"
+AR Path="/4C2E1E7D/4C2F52F0" Ref="#PWR40"  Part="1"
+F 0 "#PWR74" H 2050 3200 30  0001 C CNN
 F 1 "GND" H 2050 3130 30  0001 C CNN
 	1    2050 3200
@@
 $EndComp
 $Comp
-L C C34
-U 1 1 4C2F52EE
+L C C91
+U 1 1 4C4C7B5C
 P 3250 2950
-F 0 "C34" H 3300 3050 50  0000 L CNN
+AR Path="/4C4C6618/4C4C7B5C" Ref="C91"  Part="1"
+AR Path="/4C2E1E7D/4C4C7B5C" Ref="C87"  Part="1"
+F 0 "C91" H 3300 3050 50  0000 L CNN
 F 1 "100nf" H 3300 2850 50  0000 L CNN
 F 2 "C1V7" V 1130 2600 60  0001 C CNN
@@
 $EndComp
 $Comp
-L R R55
+L R R169
 U 1 1 4C2F52ED
 P 2300 2750
-F 0 "R55" V 2380 2750 50  0000 C CNN
+AR Path="/4C4C6618/4C2F52ED" Ref="R169"  Part="1"
+AR Path="/4C2E1E7D/4C2F52ED" Ref="R161"  Part="1"
+F 0 "R169" V 2380 2750 50  0000 C CNN
 F 1 "1k" V 2300 2750 50  0000 C CNN
 F 2 "R4-SM0805" V 2480 2850 60  0001 C CNN
@@
 $EndComp
 $Comp
-L DIODE D41
+L DIODE D70
 U 1 1 4C2F52EC
 P 2700 2350
-F 0 "D41" H 2700 2450 40  0000 C CNN
+AR Path="/4C4C6618/4C2F52EC" Ref="D70"  Part="1"
+AR Path="/4C2E1E7D/4C2F52EC" Ref="D62"  Part="1"
+F 0 "D70" H 2700 2450 40  0000 C CNN
 F 1 "1N4148" H 2700 2250 40  0000 C CNN
 F 2 "D4-SMB" V 1130 2600 60  0001 C CNN
@@
 analog_sensor_out_2
 $Comp
-L R R60
+L R R174
 U 1 1 4C2F52DC
 P 4050 1400
-F 0 "R60" V 4130 1400 50  0000 C CNN
+AR Path="/4C4C6618/4C2F52DC" Ref="R174"  Part="1"
+AR Path="/4C2E1E7D/4C2F52DC" Ref="R166"  Part="1"
+F 0 "R174" V 4130 1400 50  0000 C CNN
 F 1 "1k" V 4050 1400 50  0000 C CNN
 F 2 "R4-SM0805" V 4230 1500 60  0001 C CNN
@@
 $EndComp
 $Comp
-L GND #PWR062
-U 1 1 486F8C14
+L GND #PWR75
+U 1 1 4C4C7B4E
 P 2100 1850
-F 0 "#PWR062" H 2100 1850 30  0001 C CNN
+AR Path="/4C4C6618/4C4C7B4E" Ref="#PWR75"  Part="1"
+AR Path="/4C2E1E7D/4C4C7B4E" Ref="#PWR41"  Part="1"
+F 0 "#PWR75" H 2100 1850 30  0001 C CNN
 F 1 "GND" H 2100 1780 30  0001 C CNN
 	1    2100 1850
@@
 $EndComp
 $Comp
-L C C35
-U 1 1 486F8B93
+L C C92
+U 1 1 4C4C7B4D
 P 3300 1600
-F 0 "C35" H 3350 1700 50  0000 L CNN
+AR Path="/4C4C6618/4C4C7B4D" Ref="C92"  Part="1"
+AR Path="/4C2E1E7D/4C4C7B4D" Ref="C88"  Part="1"
+F 0 "C92" H 3350 1700 50  0000 L CNN
 F 1 "100nf" H 3350 1500 50  0000 L CNN
 F 2 "C1V7" V 1130 2600 60  0001 C CNN
@@
 $EndComp
 $Comp
-L R R56
-U 1 1 486F8B82
+L R R170
+U 1 1 4C4C7B4C
 P 2350 1400
-F 0 "R56" V 2430 1400 50  0000 C CNN
+AR Path="/4C4C6618/4C4C7B4C" Ref="R170"  Part="1"
+AR Path="/4C2E1E7D/4C4C7B4C" Ref="R162"  Part="1"
+F 0 "R170" V 2430 1400 50  0000 C CNN
 F 1 "1k" V 2350 1400 50  0000 C CNN
 F 2 "R4-SM0805" V 2530 1500 60  0001 C CNN
@@
 $EndComp
 $Comp
-L DIODE D43
+L DIODE D72
 U 1 1 4C2F52A4
 P 2750 1000
-F 0 "D43" H 2750 1100 40  0000 C CNN
+AR Path="/4C4C6618/4C2F52A4" Ref="D72"  Part="1"
+AR Path="/4C2E1E7D/4C2F52A4" Ref="D64"  Part="1"
+F 0 "D72" H 2750 1100 40  0000 C CNN
 F 1 "1N4148" H 2750 900 40  0000 C CNN
 F 2 "D4-SMB" V 1130 2600 60  0001 C CNN
