File: digi_protect_I5.sch (KiCad schematic (older format))
At the start: 5 parts

Commit message: Removed LM1815 options. Now adaptive mode and square waves are the default,
Parts:
- C17: Field1 (none) -> newark,39K8137; Field2 (none) -> vendor1, smd w hem; Field3 (none) -> vendor2, thru w hem; Field4 (none) -> vendor2, smd w hem; Field5 (none) -> 50,V; Field6 (none) -> 10,%; Field7 (none) -> Multilayer Ceramic; Field8 (none) -> other,more,stuff
- D21: Field1 (none) -> newark,98K1092; Field2 (none) -> vendor1, smd w hem; Field3 (none) -> vendor2, thru w hem; Field4 (none) -> vendor2, smd w hem; Field5 (none) -> reverse,V; Field6 (none) -> current,A; Field7 (none) -> x; Field8 (none) -> other,more,stuff
- D22: Field1 (none) -> newark,18M3285; Field2 (none) -> vendor1, smd w hem; Field3 (none) -> vendor2, thru w hem; Field4 (none) -> vendor2, smd w hem; Field5 (none) -> 500,mW; Field6 (none) -> 20,mA; Field7 (none) -> X; Field8 (none) -> other,more,stuff
- R19, R20: Field1 (none) -> newark,38K0328; Field2 (none) -> vendor1, smd w hem; Field3 (none) -> vendor2, thru w hem; Field4 (none) -> vendor2, smd w hem; Field5 (none) -> 250,mW; Field6 (none) -> 5,%; Field7 (none) -> Carbon Film; Field8 (none) -> other,more,stuff
Changed lines of the file:
@@
-EESchema Schematic File Version 1
-LIBS:power,./freeEMS_lib,device,conn,linear,regul,74xx,cmos4000,adc-dac,memory,xilinx,special,microcontrollers,dsp,microchip,analog_switches,motorola,texas,intel,audio,interface,digital-audio,philips,display,cypress,siliconi,contrib,valves,./freeEMS_1.cache
+EESchema Schematic File Version 2  date Fri 02 Jul 2010 02:24:35 PM ART
+LIBS:power
+LIBS:freeEMS_lib
+LIBS:device
+LIBS:conn
+LIBS:linear
+LIBS:regul
+LIBS:74xx
+LIBS:cmos4000
+LIBS:adc-dac
+LIBS:memory
+LIBS:xilinx
+LIBS:special
+LIBS:microcontrollers
+LIBS:dsp
+LIBS:microchip
+LIBS:analog_switches
+LIBS:motorola
+LIBS:texas
+LIBS:intel
+LIBS:audio
+LIBS:interface
+LIBS:digital-audio
+LIBS:philips
+LIBS:display
+LIBS:cypress
+LIBS:siliconi
+LIBS:contrib
+LIBS:valves
+LIBS:freeEMS_1-cache
 EELAYER 23  0
 EELAYER END
@@
 Sheet 8 41
 Title "freeEMS 1.0"
-Date "15 nov 2008"
+Date "2 jul 2010"
 Rev "A.20"
 Comp "diyefi.org"
@@
 U 1 1 489B944C
 P 4100 1750
-F 0 "R20" V 4180 1750 50  0000 C C
-F 1 "10k" V 4100 1750 50  0000 C C
-F 2 "R4-SM0805" V 4280 1850 60  0001 C C
-F 4 "newark,38K0328" V 1130 2600 60  0001 C C
-F 5 "vendor1, smd w hem" V 1130 2600 60  0001 C C
-F 6 "vendor2, thru w hem" V 1130 2600 60  0001 C C
-F 7 "vendor2, smd w hem" V 1130 2600 60  0001 C C
-F 8 "250,mW" V 1130 2600 60  0001 C C
-F 9 "5,%" V 1130 2600 60  0001 C C
-F 10 "Carbon Film" V 1130 2600 60  0001 C C
-F 11 "other,more,stuff" V 1130 2600 60  0001 C C
+F 0 "R20" V 4180 1750 50  0000 C CNN
+F 1 "10k" V 4100 1750 50  0000 C CNN
+F 2 "R4-SM0805" V 4280 1850 60  0001 C CNN
+F 4 "newark,38K0328" V 1130 2600 60  0001 C CNN "Field1"
+F 5 "vendor1, smd w hem" V 1130 2600 60  0001 C CNN "Field2"
+F 6 "vendor2, thru w hem" V 1130 2600 60  0001 C CNN "Field3"
+F 7 "vendor2, smd w hem" V 1130 2600 60  0001 C CNN "Field4"
+F 8 "250,mW" V 1130 2600 60  0001 C CNN "Field5"
+F 9 "5,%" V 1130 2600 60  0001 C CNN "Field6"
+F 10 "Carbon Film" V 1130 2600 60  0001 C CNN "Field7"
+F 11 "other,more,stuff" V 1130 2600 60  0001 C CNN "Field8"
 	1    4100 1750
 	0    1    1    0
@@
 U 1 1 489B937D
 P 2800 1550
-F 0 "D21" H 2800 1650 40  0000 C C
-F 1 "DIODE" H 2800 1450 40  0000 C C
-F 2 "D4-SMB" V 1130 2600 60  0001 C C
-F 4 "newark,98K1092" V 1130 2600 60  0001 C C
-F 5 "vendor1, smd w hem" V 1130 2600 60  0001 C C
-F 6 "vendor2, thru w hem" V 1130 2600 60  0001 C C
-F 7 "vendor2, smd w hem" V 1130 2600 60  0001 C C
-F 8 "reverse,V" V 1130 2600 60  0001 C C
-F 9 "current,A" V 1130 2600 60  0001 C C
-F 10 "x" V 1130 2600 60  0001 C C
-F 11 "other,more,stuff" V 1130 2600 60  0001 C C
+F 0 "D21" H 2800 1650 40  0000 C CNN
+F 1 "DIODE" H 2800 1450 40  0000 C CNN
+F 2 "D4-SMB" V 1130 2600 60  0001 C CNN
+F 4 "newark,98K1092" V 1130 2600 60  0001 C CNN "Field1"
+F 5 "vendor1, smd w hem" V 1130 2600 60  0001 C CNN "Field2"
+F 6 "vendor2, thru w hem" V 1130 2600 60  0001 C CNN "Field3"
+F 7 "vendor2, smd w hem" V 1130 2600 60  0001 C CNN "Field4"
+F 8 "reverse,V" V 1130 2600 60  0001 C CNN "Field5"
+F 9 "current,A" V 1130 2600 60  0001 C CNN "Field6"
+F 10 "x" V 1130 2600 60  0001 C CNN "Field7"
+F 11 "other,more,stuff" V 1130 2600 60  0001 C CNN "Field8"
 	1    2800 1550
 	0    -1   -1   0
 $EndComp
-Text GLabel 1950 1350 0    60   Input
+Text HLabel 1950 1350 0    60   Input ~ 0
 digi_vcc
 $Comp
@@
 U 1 1 486F8DB9
 P 2800 1950
-F 0 "D22" H 2800 2050 50  0000 C C
-F 1 "5V1" H 2800 1850 40  0000 C C
-F 2 "D4-SMB" V 1130 2600 60  0001 C C
-F 4 "newark,18M3285" V 1130 2600 60  0001 C C
-F 5 "vendor1, smd w hem" V 1130 2600 60  0001 C C
-F 6 "vendor2, thru w hem" V 1130 2600 60  0001 C C
-F 7 "vendor2, smd w hem" V 1130 2600 60  0001 C C
-F 8 "500,mW" V 1130 2600 60  0001 C C
-F 9 "20,mA" V 1130 2600 60  0001 C C
-F 10 "X" V 1130 2600 60  0001 C C
-F 11 "other,more,stuff" V 1130 2600 60  0001 C C
+F 0 "D22" H 2800 2050 50  0000 C CNN
+F 1 "5V1" H 2800 1850 40  0000 C CNN
+F 2 "D4-SMB" V 1130 2600 60  0001 C CNN
+F 4 "newark,18M3285" V 1130 2600 60  0001 C CNN "Field1"
+F 5 "vendor1, smd w hem" V 1130 2600 60  0001 C CNN "Field2"
+F 6 "vendor2, thru w hem" V 1130 2600 60  0001 C CNN "Field3"
+F 7 "vendor2, smd w hem" V 1130 2600 60  0001 C CNN "Field4"
+F 8 "500,mW" V 1130 2600 60  0001 C CNN "Field5"
+F 9 "20,mA" V 1130 2600 60  0001 C CNN "Field6"
+F 10 "X" V 1130 2600 60  0001 C CNN "Field7"
+F 11 "other,more,stuff" V 1130 2600 60  0001 C CNN "Field8"
 	1    2800 1950
 	0    -1   -1   0
@@
 U 1 1 486F8D89
 P 2400 1750
-F 0 "R19" V 2480 1750 50  0000 C C
-F 1 "10k" V 2400 1750 50  0000 C C
-F 2 "R4-SM0805" V 2580 1850 60  0001 C C
-F 4 "newark,38K0328" V 1130 2600 60  0001 C C
-F 5 "vendor1, smd w hem" V 1130 2600 60  0001 C C
-F 6 "vendor2, thru w hem" V 1130 2600 60  0001 C C
-F 7 "vendor2, smd w hem" V 1130 2600 60  0001 C C
-F 8 "250,mW" V 1130 2600 60  0001 C C
-F 9 "5,%" V 1130 2600 60  0001 C C
-F 10 "Carbon Film" V 1130 2600 60  0001 C C
-F 11 "other,more,stuff" V 1130 2600 60  0001 C C
+F 0 "R19" V 2480 1750 50  0000 C CNN
+F 1 "10k" V 2400 1750 50  0000 C CNN
+F 2 "R4-SM0805" V 2580 1850 60  0001 C CNN
+F 4 "newark,38K0328" V 1130 2600 60  0001 C CNN "Field1"
+F 5 "vendor1, smd w hem" V 1130 2600 60  0001 C CNN "Field2"
+F 6 "vendor2, thru w hem" V 1130 2600 60  0001 C CNN "Field3"
+F 7 "vendor2, smd w hem" V 1130 2600 60  0001 C CNN "Field4"
+F 8 "250,mW" V 1130 2600 60  0001 C CNN "Field5"
+F 9 "5,%" V 1130 2600 60  0001 C CNN "Field6"
+F 10 "Carbon Film" V 1130 2600 60  0001 C CNN "Field7"
+F 11 "other,more,stuff" V 1130 2600 60  0001 C CNN "Field8"
 	1    2400 1750
 	0    1    1    0
@@
 U 1 1 486F8D85
 P 3250 1950
-F 0 "C17" H 3300 2050 50  0000 L C
-F 1 "100nF" H 3300 1850 50  0000 L C
-F 2 "C1V7" V 1130 2600 60  0001 C C
-F 4 "newark,39K8137" V 1130 2600 60  0001 C C
-F 5 "vendor1, smd w hem" V 1130 2600 60  0001 C C
-F 6 "vendor2, thru w hem" V 1130 2600 60  0001 C C
-F 7 "vendor2, smd w hem" V 1130 2600 60  0001 C C
-F 8 "50,V" V 1130 2600 60  0001 C C
-F 9 "10,%" V 1130 2600 60  0001 C C
-F 10 "Multilayer Ceramic" V 1130 2600 60  0001 C C
-F 11 "other,more,stuff" V 1130 2600 60  0001 C C
+F 0 "C17" H 3300 2050 50  0000 L CNN
+F 1 "100nF" H 3300 1850 50  0000 L CNN
+F 2 "C1V7" V 1130 2600 60  0001 C CNN
+F 4 "newark,39K8137" V 1130 2600 60  0001 C CNN "Field1"
+F 5 "vendor1, smd w hem" V 1130 2600 60  0001 C CNN "Field2"
+F 6 "vendor2, thru w hem" V 1130 2600 60  0001 C CNN "Field3"
+F 7 "vendor2, smd w hem" V 1130 2600 60  0001 C CNN "Field4"
+F 8 "50,V" V 1130 2600 60  0001 C CNN "Field5"
+F 9 "10,%" V 1130 2600 60  0001 C CNN "Field6"
+F 10 "Multilayer Ceramic" V 1130 2600 60  0001 C CNN "Field7"
+F 11 "other,more,stuff" V 1130 2600 60  0001 C CNN "Field8"
 	1    3250 1950
 	1    0    0    -1
@@
 U 1 1 486F8D7E
 P 2800 2250
-F 0 "#PWR029" H 2800 2250 30  0001 C C
-F 1 "GND" H 2800 2180 30  0001 C C
+F 0 "#PWR029" H 2800 2250 30  0001 C CNN
+F 1 "GND" H 2800 2180 30  0001 C CNN
 	1    2800 2250
 	1    0    0    -1
 $EndComp
-Text GLabel 1950 2150 0    60   BiDi
+Text HLabel 1950 2150 0    60   BiDi ~ 0
 digi_gnd
-Text GLabel 1950 1750 0    60   BiDi
+Text HLabel 1950 1750 0    60   BiDi ~ 0
 digi_CPU
-Text GLabel 4550 1750 2    60   BiDi
+Text HLabel 4550 1750 2    60   BiDi ~ 0
 digi_device
 $EndSCHEMATC

Commit message: Implemented P&H, removed current sense circuitry, removed all unnecessary files from the repo
Parts:
- renumbered C17 to C?, D22 to D?, D21 to D?, R19 to R?, R20 to R?
Changed lines of the file:
@@
-EESchema Schematic File Version 2  date Fri 02 Jul 2010 05:44:26 PM ART
+EESchema Schematic File Version 2  date Sat 03 Jul 2010 10:49:02 AM ART
 LIBS:power
 LIBS:freeEMS_lib
@@
 EELAYER END
 $Descr A4 11700 8267
-Sheet 8 41
+Sheet 1 41
 Title "freeEMS 1.0"
-Date "2 jul 2010"
-Rev "A.20"
+Date "3 jul 2010"
+Rev "A.08"
 Comp "diyefi.org"
 Comment1 "digi_protect.sch"
@@
 Connection ~ 2800 2150
 $Comp
-L R R20
+L R R?
 U 1 1 489B944C
 P 4100 1750
-F 0 "R20" V 4180 1750 50  0000 C CNN
+F 0 "R?" V 4180 1750 50  0000 C CNN
 F 1 "10k" V 4100 1750 50  0000 C CNN
 F 2 "R4-SM0805" V 4280 1850 60  0001 C CNN
@@
 $EndComp
 $Comp
-L DIODE D21
+L DIODE D?
 U 1 1 489B937D
 P 2800 1550
-F 0 "D21" H 2800 1650 40  0000 C CNN
+F 0 "D?" H 2800 1650 40  0000 C CNN
 F 1 "DIODE" H 2800 1450 40  0000 C CNN
 F 2 "D4-SMB" V 1130 2600 60  0001 C CNN
@@
 digi_vcc
 $Comp
-L ZENER D22
+L ZENER D?
 U 1 1 486F8DB9
 P 2800 1950
-F 0 "D22" H 2800 2050 50  0000 C CNN
+F 0 "D?" H 2800 2050 50  0000 C CNN
 F 1 "5V1" H 2800 1850 40  0000 C CNN
 F 2 "D4-SMB" V 1130 2600 60  0001 C CNN
@@
 $EndComp
 $Comp
-L R R19
+L R R?
 U 1 1 486F8D89
 P 2400 1750
-F 0 "R19" V 2480 1750 50  0000 C CNN
+F 0 "R?" V 2480 1750 50  0000 C CNN
 F 1 "10k" V 2400 1750 50  0000 C CNN
 F 2 "R4-SM0805" V 2580 1850 60  0001 C CNN
@@
 $EndComp
 $Comp
-L C C17
+L C C?
 U 1 1 486F8D85
 P 3250 1950
-F 0 "C17" H 3300 2050 50  0000 L CNN
+F 0 "C?" H 3300 2050 50  0000 L CNN
 F 1 "100nF" H 3300 1850 50  0000 L CNN
 F 2 "C1V7" V 1130 2600 60  0001 C CNN
@@
 $EndComp
 $Comp
-L GND #PWR029
+L GND #PWR?
 U 1 1 486F8D7E
 P 2800 2250
-F 0 "#PWR029" H 2800 2250 30  0001 C CNN
+F 0 "#PWR?" H 2800 2250 30  0001 C CNN
 F 1 "GND" H 2800 2180 30  0001 C CNN
 	1    2800 2250

Commit message: Corrected ERC errors by fixing the custom FreeEMS components pinouts
Parts:
- removed C?: 100nF, C1V7, symbol C
- removed D?: 5V1, D4-SMB, symbol ZENER
- removed D?: DIODE, D4-SMB, symbol DIODE
- removed R? (x2): 10k, R4-SM0805, symbol R
- added C17: 100nF, C1V7, symbol C
- added D13: DIODE, D4-SMB, symbol DIODE
- added D14: 5V1, D4-SMB, symbol ZENER
- added R11, R12: 10k, R4-SM0805, symbol R
Connections:
- net GND: now also C17.2, D14.1 (A)
- net digi_CPU: now also R11.2
- net digi_device: now also R12.1
- net digi_vcc: now also D13.2 (K)
- new net: C17.1, R11.1, R12.2
- new net: D13.1 (A), D14.2 (K)
Changed lines of the file:
@@
-EESchema Schematic File Version 2  date Sat 03 Jul 2010 10:49:02 AM ART
+EESchema Schematic File Version 2  date Sat 03 Jul 2010 12:32:24 PM ART
 LIBS:power
 LIBS:freeEMS_lib
@@
 Connection ~ 2800 2150
 $Comp
-L R R?
-U 1 1 489B944C
+L R R12
+U 1 1 4C2F5305
 P 4100 1750
-F 0 "R?" V 4180 1750 50  0000 C CNN
+F 0 "R12" V 4180 1750 50  0000 C CNN
 F 1 "10k" V 4100 1750 50  0000 C CNN
 F 2 "R4-SM0805" V 4280 1850 60  0001 C CNN
@@
 $EndComp
 $Comp
-L DIODE D?
-U 1 1 489B937D
+L DIODE D13
+U 1 1 4C2F52F9
 P 2800 1550
-F 0 "D?" H 2800 1650 40  0000 C CNN
+F 0 "D13" H 2800 1650 40  0000 C CNN
 F 1 "DIODE" H 2800 1450 40  0000 C CNN
 F 2 "D4-SMB" V 1130 2600 60  0001 C CNN
@@
 digi_vcc
 $Comp
-L ZENER D?
-U 1 1 486F8DB9
+L ZENER D14
+U 1 1 4C2F52C9
 P 2800 1950
-F 0 "D?" H 2800 2050 50  0000 C CNN
+F 0 "D14" H 2800 2050 50  0000 C CNN
 F 1 "5V1" H 2800 1850 40  0000 C CNN
 F 2 "D4-SMB" V 1130 2600 60  0001 C CNN
@@
 $EndComp
 $Comp
-L R R?
-U 1 1 486F8D89
+L R R11
+U 1 1 4C2F52BF
 P 2400 1750
-F 0 "R?" V 2480 1750 50  0000 C CNN
+F 0 "R11" V 2480 1750 50  0000 C CNN
 F 1 "10k" V 2400 1750 50  0000 C CNN
 F 2 "R4-SM0805" V 2580 1850 60  0001 C CNN
@@
 $EndComp
 $Comp
-L C C?
-U 1 1 486F8D85
+L C C17
+U 1 1 4C2F52B6
 P 3250 1950
-F 0 "C?" H 3300 2050 50  0000 L CNN
+F 0 "C17" H 3300 2050 50  0000 L CNN
 F 1 "100nF" H 3300 1850 50  0000 L CNN
 F 2 "C1V7" V 1130 2600 60  0001 C CNN
@@
 $EndComp
 $Comp
-L GND #PWR?
-U 1 1 486F8D7E
+L GND #PWR050
+U 1 1 4C2F52AA
 P 2800 2250
-F 0 "#PWR?" H 2800 2250 30  0001 C CNN
+F 0 "#PWR050" H 2800 2250 30  0001 C CNN
 F 1 "GND" H 2800 2180 30  0001 C CNN
 	1    2800 2250

Commit message: Exchanged current sensing with peak&hold, and a closer approach to a more integrated design.
Parts:
- removed D13: DIODE, D4-SMB, symbol DIODE
Connections:
- net at C17.1, R11.1, R12.2: now also D14.2 (K)
Changed lines of the file:
@@
-EESchema Schematic File Version 2  date Sat 03 Jul 2010 05:37:07 PM ART
+EESchema Schematic File Version 2  date Thu 22 Jul 2010 10:06:33 AM ART
 LIBS:power
 LIBS:freeEMS_lib
@@
 EELAYER END
 $Descr A4 11700 8267
-Sheet 1 41
+Sheet 14 41
 Title "freeEMS 1.0"
-Date "3 jul 2010"
+Date "22 jul 2010"
 Rev "A.08"
 Comp "diyefi.org"
@@
 Comment4 ""
 $EndDescr
+Connection ~ 2800 1750
+Connection ~ 2800 2150
 Wire Wire Line
-	4350 1750 4550 1750
+	3250 2150 1950 2150
 Wire Wire Line
-	2800 1350 1950 1350
+	2150 1750 1950 1750
+Connection ~ 3250 1750
+Wire Wire Line
+	3850 1750 2650 1750
 Wire Wire Line
 	2800 2250 2800 2150
 Wire Wire Line
-	3850 1750 2650 1750
-Connection ~ 3250 1750
-Wire Wire Line
-	2150 1750 1950 1750
-Wire Wire Line
-	3250 2150 1950 2150
-Connection ~ 2800 2150
+	4350 1750 4550 1750
 $Comp
 L R R12
@@
 $EndComp
 $Comp
-L DIODE D13
-U 1 1 4C2F52F9
-P 2800 1550
-F 0 "D13" H 2800 1650 40  0000 C CNN
-F 1 "DIODE" H 2800 1450 40  0000 C CNN
-F 2 "D4-SMB" V 1130 2600 60  0001 C CNN
-F 4 "newark,98K1092" V 1130 2600 60  0001 C CNN "Field1"
-F 5 "vendor1, smd w hem" V 1130 2600 60  0001 C CNN "Field2"
-F 6 "vendor2, thru w hem" V 1130 2600 60  0001 C CNN "Field3"
-F 7 "vendor2, smd w hem" V 1130 2600 60  0001 C CNN "Field4"
-F 8 "reverse,V" V 1130 2600 60  0001 C CNN "Field5"
-F 9 "current,A" V 1130 2600 60  0001 C CNN "Field6"
-F 10 "x" V 1130 2600 60  0001 C CNN "Field7"
-F 11 "other,more,stuff" V 1130 2600 60  0001 C CNN "Field8"
-	1    2800 1550
-	0    -1   -1   0
-$EndComp
-Text HLabel 1950 1350 0    60   Input ~ 0
-digi_vcc
-$Comp
 L ZENER D14
