File: digi_protect_misc1.sch (KiCad schematic (older format))
At the start: 5 parts

Commit message: Removed LM1815 options. Now adaptive mode and square waves are the default,
Parts:
- C28: Field1 (none) -> newark,39K8137; Field2 (none) -> vendor1, smd w hem; Field3 (none) -> vendor2, thru w hem; Field4 (none) -> vendor2, smd w hem; Field5 (none) -> 50,V; Field6 (none) -> 10,%; Field7 (none) -> Multilayer Ceramic; Field8 (none) -> other,more,stuff
- D37: Field1 (none) -> newark,98K1092; Field2 (none) -> vendor1, smd w hem; Field3 (none) -> vendor2, thru w hem; Field4 (none) -> vendor2, smd w hem; Field5 (none) -> reverse,V; Field6 (none) -> current,A; Field7 (none) -> x; Field8 (none) -> other,more,stuff
- D38: Field1 (none) -> newark,18M3285; Field2 (none) -> vendor1, smd w hem; Field3 (none) -> vendor2, thru w hem; Field4 (none) -> vendor2, smd w hem; Field5 (none) -> 500,mW; Field6 (none) -> 20,mA; Field7 (none) -> X; Field8 (none) -> other,more,stuff
- R53, R54: Field1 (none) -> newark,38K0328; Field2 (none) -> vendor1, smd w hem; Field3 (none) -> vendor2, thru w hem; Field4 (none) -> vendor2, smd w hem; Field5 (none) -> 250,mW; Field6 (none) -> 5,%; Field7 (none) -> Carbon Film; Field8 (none) -> other,more,stuff
Changed lines of the file:
@@
-EESchema Schematic File Version 1
-LIBS:power,./freeEMS_lib,device,conn,linear,regul,74xx,cmos4000,adc-dac,memory,xilinx,special,microcontrollers,dsp,microchip,analog_switches,motorola,texas,intel,audio,interface,digital-audio,philips,display,cypress,siliconi,contrib,valves,./freeEMS_1.cache
+EESchema Schematic File Version 2  date Fri 02 Jul 2010 02:24:35 PM ART
+LIBS:power
+LIBS:freeEMS_lib
+LIBS:device
+LIBS:conn
+LIBS:linear
+LIBS:regul
+LIBS:74xx
+LIBS:cmos4000
+LIBS:adc-dac
+LIBS:memory
+LIBS:xilinx
+LIBS:special
+LIBS:microcontrollers
+LIBS:dsp
+LIBS:microchip
+LIBS:analog_switches
+LIBS:motorola
+LIBS:texas
+LIBS:intel
+LIBS:audio
+LIBS:interface
+LIBS:digital-audio
+LIBS:philips
+LIBS:display
+LIBS:cypress
+LIBS:siliconi
+LIBS:contrib
+LIBS:valves
+LIBS:freeEMS_1-cache
 EELAYER 23  0
 EELAYER END
@@
 Sheet 21 41
 Title "freeEMS 1.0"
-Date "15 nov 2008"
+Date "2 jul 2010"
 Rev "A.20"
 Comp "diyefi.org"
@@
 U 1 1 489B944C
 P 4100 1750
-F 0 "R54" V 4180 1750 50  0000 C C
-F 1 "10k" V 4100 1750 50  0000 C C
-F 2 "R4-SM0805" V 4280 1850 60  0001 C C
-F 4 "newark,38K0328" V 1130 2600 60  0001 C C
-F 5 "vendor1, smd w hem" V 1130 2600 60  0001 C C
-F 6 "vendor2, thru w hem" V 1130 2600 60  0001 C C
-F 7 "vendor2, smd w hem" V 1130 2600 60  0001 C C
-F 8 "250,mW" V 1130 2600 60  0001 C C
-F 9 "5,%" V 1130 2600 60  0001 C C
-F 10 "Carbon Film" V 1130 2600 60  0001 C C
-F 11 "other,more,stuff" V 1130 2600 60  0001 C C
+F 0 "R54" V 4180 1750 50  0000 C CNN
+F 1 "10k" V 4100 1750 50  0000 C CNN
+F 2 "R4-SM0805" V 4280 1850 60  0001 C CNN
+F 4 "newark,38K0328" V 1130 2600 60  0001 C CNN "Field1"
+F 5 "vendor1, smd w hem" V 1130 2600 60  0001 C CNN "Field2"
+F 6 "vendor2, thru w hem" V 1130 2600 60  0001 C CNN "Field3"
+F 7 "vendor2, smd w hem" V 1130 2600 60  0001 C CNN "Field4"
+F 8 "250,mW" V 1130 2600 60  0001 C CNN "Field5"
+F 9 "5,%" V 1130 2600 60  0001 C CNN "Field6"
+F 10 "Carbon Film" V 1130 2600 60  0001 C CNN "Field7"
+F 11 "other,more,stuff" V 1130 2600 60  0001 C CNN "Field8"
 	1    4100 1750
 	0    1    1    0
@@
 U 1 1 489B937D
 P 2800 1550
-F 0 "D37" H 2800 1650 40  0000 C C
-F 1 "DIODE" H 2800 1450 40  0000 C C
-F 2 "D4-SMB" V 1130 2600 60  0001 C C
-F 4 "newark,98K1092" V 1130 2600 60  0001 C C
-F 5 "vendor1, smd w hem" V 1130 2600 60  0001 C C
-F 6 "vendor2, thru w hem" V 1130 2600 60  0001 C C
-F 7 "vendor2, smd w hem" V 1130 2600 60  0001 C C
-F 8 "reverse,V" V 1130 2600 60  0001 C C
-F 9 "current,A" V 1130 2600 60  0001 C C
-F 10 "x" V 1130 2600 60  0001 C C
-F 11 "other,more,stuff" V 1130 2600 60  0001 C C
+F 0 "D37" H 2800 1650 40  0000 C CNN
+F 1 "DIODE" H 2800 1450 40  0000 C CNN
+F 2 "D4-SMB" V 1130 2600 60  0001 C CNN
+F 4 "newark,98K1092" V 1130 2600 60  0001 C CNN "Field1"
+F 5 "vendor1, smd w hem" V 1130 2600 60  0001 C CNN "Field2"
+F 6 "vendor2, thru w hem" V 1130 2600 60  0001 C CNN "Field3"
+F 7 "vendor2, smd w hem" V 1130 2600 60  0001 C CNN "Field4"
+F 8 "reverse,V" V 1130 2600 60  0001 C CNN "Field5"
+F 9 "current,A" V 1130 2600 60  0001 C CNN "Field6"
+F 10 "x" V 1130 2600 60  0001 C CNN "Field7"
+F 11 "other,more,stuff" V 1130 2600 60  0001 C CNN "Field8"
 	1    2800 1550
 	0    -1   -1   0
 $EndComp
-Text GLabel 1950 1350 0    60   Input
+Text HLabel 1950 1350 0    60   Input ~ 0
 digi_vcc
 $Comp
@@
 U 1 1 486F8DB9
 P 2800 1950
-F 0 "D38" H 2800 2050 50  0000 C C
-F 1 "5V1" H 2800 1850 40  0000 C C
-F 2 "D4-SMB" V 1130 2600 60  0001 C C
-F 4 "newark,18M3285" V 1130 2600 60  0001 C C
-F 5 "vendor1, smd w hem" V 1130 2600 60  0001 C C
-F 6 "vendor2, thru w hem" V 1130 2600 60  0001 C C
-F 7 "vendor2, smd w hem" V 1130 2600 60  0001 C C
-F 8 "500,mW" V 1130 2600 60  0001 C C
-F 9 "20,mA" V 1130 2600 60  0001 C C
-F 10 "X" V 1130 2600 60  0001 C C
-F 11 "other,more,stuff" V 1130 2600 60  0001 C C
+F 0 "D38" H 2800 2050 50  0000 C CNN
+F 1 "5V1" H 2800 1850 40  0000 C CNN
+F 2 "D4-SMB" V 1130 2600 60  0001 C CNN
+F 4 "newark,18M3285" V 1130 2600 60  0001 C CNN "Field1"
+F 5 "vendor1, smd w hem" V 1130 2600 60  0001 C CNN "Field2"
+F 6 "vendor2, thru w hem" V 1130 2600 60  0001 C CNN "Field3"
+F 7 "vendor2, smd w hem" V 1130 2600 60  0001 C CNN "Field4"
+F 8 "500,mW" V 1130 2600 60  0001 C CNN "Field5"
+F 9 "20,mA" V 1130 2600 60  0001 C CNN "Field6"
+F 10 "X" V 1130 2600 60  0001 C CNN "Field7"
+F 11 "other,more,stuff" V 1130 2600 60  0001 C CNN "Field8"
 	1    2800 1950
 	0    -1   -1   0
@@
 U 1 1 486F8D89
 P 2400 1750
-F 0 "R53" V 2480 1750 50  0000 C C
-F 1 "10k" V 2400 1750 50  0000 C C
-F 2 "R4-SM0805" V 2580 1850 60  0001 C C
-F 4 "newark,38K0328" V 1130 2600 60  0001 C C
-F 5 "vendor1, smd w hem" V 1130 2600 60  0001 C C
-F 6 "vendor2, thru w hem" V 1130 2600 60  0001 C C
-F 7 "vendor2, smd w hem" V 1130 2600 60  0001 C C
-F 8 "250,mW" V 1130 2600 60  0001 C C
-F 9 "5,%" V 1130 2600 60  0001 C C
-F 10 "Carbon Film" V 1130 2600 60  0001 C C
-F 11 "other,more,stuff" V 1130 2600 60  0001 C C
+F 0 "R53" V 2480 1750 50  0000 C CNN
+F 1 "10k" V 2400 1750 50  0000 C CNN
+F 2 "R4-SM0805" V 2580 1850 60  0001 C CNN
+F 4 "newark,38K0328" V 1130 2600 60  0001 C CNN "Field1"
+F 5 "vendor1, smd w hem" V 1130 2600 60  0001 C CNN "Field2"
+F 6 "vendor2, thru w hem" V 1130 2600 60  0001 C CNN "Field3"
+F 7 "vendor2, smd w hem" V 1130 2600 60  0001 C CNN "Field4"
+F 8 "250,mW" V 1130 2600 60  0001 C CNN "Field5"
+F 9 "5,%" V 1130 2600 60  0001 C CNN "Field6"
+F 10 "Carbon Film" V 1130 2600 60  0001 C CNN "Field7"
+F 11 "other,more,stuff" V 1130 2600 60  0001 C CNN "Field8"
 	1    2400 1750
 	0    1    1    0
@@
 U 1 1 486F8D85
 P 3250 1950
-F 0 "C28" H 3300 2050 50  0000 L C
-F 1 "100nF" H 3300 1850 50  0000 L C
-F 2 "C1V7" V 1130 2600 60  0001 C C
-F 4 "newark,39K8137" V 1130 2600 60  0001 C C
-F 5 "vendor1, smd w hem" V 1130 2600 60  0001 C C
-F 6 "vendor2, thru w hem" V 1130 2600 60  0001 C C
-F 7 "vendor2, smd w hem" V 1130 2600 60  0001 C C
-F 8 "50,V" V 1130 2600 60  0001 C C
-F 9 "10,%" V 1130 2600 60  0001 C C
-F 10 "Multilayer Ceramic" V 1130 2600 60  0001 C C
-F 11 "other,more,stuff" V 1130 2600 60  0001 C C
+F 0 "C28" H 3300 2050 50  0000 L CNN
+F 1 "100nF" H 3300 1850 50  0000 L CNN
+F 2 "C1V7" V 1130 2600 60  0001 C CNN
+F 4 "newark,39K8137" V 1130 2600 60  0001 C CNN "Field1"
+F 5 "vendor1, smd w hem" V 1130 2600 60  0001 C CNN "Field2"
+F 6 "vendor2, thru w hem" V 1130 2600 60  0001 C CNN "Field3"
+F 7 "vendor2, smd w hem" V 1130 2600 60  0001 C CNN "Field4"
+F 8 "50,V" V 1130 2600 60  0001 C CNN "Field5"
+F 9 "10,%" V 1130 2600 60  0001 C CNN "Field6"
+F 10 "Multilayer Ceramic" V 1130 2600 60  0001 C CNN "Field7"
+F 11 "other,more,stuff" V 1130 2600 60  0001 C CNN "Field8"
 	1    3250 1950
 	1    0    0    -1
@@
 U 1 1 486F8D7E
 P 2800 2250
-F 0 "#PWR034" H 2800 2250 30  0001 C C
-F 1 "GND" H 2800 2180 30  0001 C C
+F 0 "#PWR034" H 2800 2250 30  0001 C CNN
+F 1 "GND" H 2800 2180 30  0001 C CNN
 	1    2800 2250
 	1    0    0    -1
 $EndComp
-Text GLabel 1950 2150 0    60   BiDi
+Text HLabel 1950 2150 0    60   BiDi ~ 0
 digi_gnd
-Text GLabel 1950 1750 0    60   BiDi
+Text HLabel 1950 1750 0    60   BiDi ~ 0
 digi_CPU
-Text GLabel 4550 1750 2    60   BiDi
+Text HLabel 4550 1750 2    60   BiDi ~ 0
 digi_device
 $EndSCHEMATC

Commit message: Implemented P&H, removed current sense circuitry, removed all unnecessary files from the repo
Parts:
- renumbered C28 to C?, D38 to D?, D37 to D?, R53 to R?, R54 to R?
Changed lines of the file:
@@
-EESchema Schematic File Version 2  date Fri 02 Jul 2010 05:44:26 PM ART
+EESchema Schematic File Version 2  date Sat 03 Jul 2010 10:49:02 AM ART
 LIBS:power
 LIBS:freeEMS_lib
@@
 EELAYER END
 $Descr A4 11700 8267
-Sheet 21 41
+Sheet 1 41
 Title "freeEMS 1.0"
-Date "2 jul 2010"
-Rev "A.20"
+Date "3 jul 2010"
+Rev "A.08"
 Comp "diyefi.org"
 Comment1 "digi_protect.sch"
@@
 Connection ~ 2800 2150
 $Comp
-L R R54
+L R R?
 U 1 1 489B944C
 P 4100 1750
-F 0 "R54" V 4180 1750 50  0000 C CNN
+F 0 "R?" V 4180 1750 50  0000 C CNN
 F 1 "10k" V 4100 1750 50  0000 C CNN
 F 2 "R4-SM0805" V 4280 1850 60  0001 C CNN
@@
 $EndComp
 $Comp
-L DIODE D37
+L DIODE D?
 U 1 1 489B937D
 P 2800 1550
-F 0 "D37" H 2800 1650 40  0000 C CNN
+F 0 "D?" H 2800 1650 40  0000 C CNN
 F 1 "DIODE" H 2800 1450 40  0000 C CNN
 F 2 "D4-SMB" V 1130 2600 60  0001 C CNN
@@
 digi_vcc
 $Comp
-L ZENER D38
+L ZENER D?
 U 1 1 486F8DB9
 P 2800 1950
-F 0 "D38" H 2800 2050 50  0000 C CNN
+F 0 "D?" H 2800 2050 50  0000 C CNN
 F 1 "5V1" H 2800 1850 40  0000 C CNN
 F 2 "D4-SMB" V 1130 2600 60  0001 C CNN
@@
 $EndComp
 $Comp
-L R R53
+L R R?
 U 1 1 486F8D89
 P 2400 1750
-F 0 "R53" V 2480 1750 50  0000 C CNN
+F 0 "R?" V 2480 1750 50  0000 C CNN
 F 1 "10k" V 2400 1750 50  0000 C CNN
 F 2 "R4-SM0805" V 2580 1850 60  0001 C CNN
@@
 $EndComp
 $Comp
-L C C28
+L C C?
 U 1 1 486F8D85
 P 3250 1950
-F 0 "C28" H 3300 2050 50  0000 L CNN
+F 0 "C?" H 3300 2050 50  0000 L CNN
 F 1 "100nF" H 3300 1850 50  0000 L CNN
 F 2 "C1V7" V 1130 2600 60  0001 C CNN
@@
 $EndComp
 $Comp
-L GND #PWR034
+L GND #PWR?
 U 1 1 486F8D7E
 P 2800 2250
-F 0 "#PWR034" H 2800 2250 30  0001 C CNN
+F 0 "#PWR?" H 2800 2250 30  0001 C CNN
 F 1 "GND" H 2800 2180 30  0001 C CNN
 	1    2800 2250

Commit message: Corrected ERC errors by fixing the custom FreeEMS components pinouts
Parts:
- removed C?: 100nF, C1V7, symbol C
- removed D?: 5V1, D4-SMB, symbol ZENER
- removed D?: DIODE, D4-SMB, symbol DIODE
- removed R? (x2): 10k, R4-SM0805, symbol R
- added C28: 100nF, C1V7, symbol C
- added D29: DIODE, D4-SMB, symbol DIODE
- added D30: 5V1, D4-SMB, symbol ZENER
- added R45, R46: 10k, R4-SM0805, symbol R
Connections:
- net GND: now also C28.2, D30.1 (A)
- net digi_CPU: now also R45.2
- net digi_device: now also R46.1
- net digi_vcc: now also D29.2 (K)
- new net: C28.1, R45.1, R46.2
- new net: D29.1 (A), D30.2 (K)
Changed lines of the file:
@@
-EESchema Schematic File Version 2  date Sat 03 Jul 2010 10:49:02 AM ART
+EESchema Schematic File Version 2  date Sat 03 Jul 2010 12:32:24 PM ART
 LIBS:power
 LIBS:freeEMS_lib
@@
 Connection ~ 2800 2150
 $Comp
-L R R?
-U 1 1 489B944C
+L R R46
+U 1 1 4C2F5309
 P 4100 1750
-F 0 "R?" V 4180 1750 50  0000 C CNN
+F 0 "R46" V 4180 1750 50  0000 C CNN
 F 1 "10k" V 4100 1750 50  0000 C CNN
 F 2 "R4-SM0805" V 4280 1850 60  0001 C CNN
@@
 $EndComp
 $Comp
-L DIODE D?
-U 1 1 489B937D
+L DIODE D29
+U 1 1 4C2F5301
 P 2800 1550
-F 0 "D?" H 2800 1650 40  0000 C CNN
+F 0 "D29" H 2800 1650 40  0000 C CNN
 F 1 "DIODE" H 2800 1450 40  0000 C CNN
 F 2 "D4-SMB" V 1130 2600 60  0001 C CNN
@@
 digi_vcc
 $Comp
-L ZENER D?
-U 1 1 486F8DB9
+L ZENER D30
+U 1 1 4C2F52C7
 P 2800 1950
-F 0 "D?" H 2800 2050 50  0000 C CNN
+F 0 "D30" H 2800 2050 50  0000 C CNN
 F 1 "5V1" H 2800 1850 40  0000 C CNN
 F 2 "D4-SMB" V 1130 2600 60  0001 C CNN
@@
 $EndComp
 $Comp
-L R R?
-U 1 1 486F8D89
+L R R45
+U 1 1 4C2F52BE
 P 2400 1750
-F 0 "R?" V 2480 1750 50  0000 C CNN
+F 0 "R45" V 2480 1750 50  0000 C CNN
 F 1 "10k" V 2400 1750 50  0000 C CNN
 F 2 "R4-SM0805" V 2580 1850 60  0001 C CNN
@@
 $EndComp
 $Comp
-L C C?
-U 1 1 486F8D85
+L C C28
+U 1 1 4C2F52BA
 P 3250 1950
-F 0 "C?" H 3300 2050 50  0000 L CNN
+F 0 "C28" H 3300 2050 50  0000 L CNN
 F 1 "100nF" H 3300 1850 50  0000 L CNN
 F 2 "C1V7" V 1130 2600 60  0001 C CNN
@@
 $EndComp
 $Comp
-L GND #PWR?
-U 1 1 486F8D7E
+L GND #PWR055
+U 1 1 4C2F52B1
 P 2800 2250
-F 0 "#PWR?" H 2800 2250 30  0001 C CNN
+F 0 "#PWR055" H 2800 2250 30  0001 C CNN
 F 1 "GND" H 2800 2180 30  0001 C CNN
 	1    2800 2250

Commit message: Exchanged current sensing with peak&hold, and a closer approach to a more integrated design.
Parts:
- removed D29: DIODE, D4-SMB, symbol DIODE
Connections:
- net at C28.1, R45.1, R46.2: now also D30.2 (K)
Changed lines of the file:
@@
-EESchema Schematic File Version 2  date Sat 03 Jul 2010 05:37:07 PM ART
+EESchema Schematic File Version 2  date Thu 22 Jul 2010 10:06:33 AM ART
 LIBS:power
 LIBS:freeEMS_lib
@@
 EELAYER END
 $Descr A4 11700 8267
-Sheet 1 41
+Sheet 27 41
 Title "freeEMS 1.0"
-Date "3 jul 2010"
+Date "22 jul 2010"
 Rev "A.08"
 Comp "diyefi.org"
@@
 Comment4 ""
 $EndDescr
+Connection ~ 2800 1750
+Connection ~ 2800 2150
 Wire Wire Line
-	4350 1750 4550 1750
+	3250 2150 1950 2150
 Wire Wire Line
-	2800 1350 1950 1350
+	2150 1750 1950 1750
+Connection ~ 3250 1750
+Wire Wire Line
+	3850 1750 2650 1750
 Wire Wire Line
 	2800 2250 2800 2150
 Wire Wire Line
-	3850 1750 2650 1750
-Connection ~ 3250 1750
-Wire Wire Line
-	2150 1750 1950 1750
-Wire Wire Line
-	3250 2150 1950 2150
-Connection ~ 2800 2150
+	4350 1750 4550 1750
 $Comp
 L R R46
@@
 $EndComp
 $Comp
-L DIODE D29
-U 1 1 4C2F5301
-P 2800 1550
-F 0 "D29" H 2800 1650 40  0000 C CNN
-F 1 "DIODE" H 2800 1450 40  0000 C CNN
-F 2 "D4-SMB" V 1130 2600 60  0001 C CNN
-F 4 "newark,98K1092" V 1130 2600 60  0001 C CNN "Field1"
-F 5 "vendor1, smd w hem" V 1130 2600 60  0001 C CNN "Field2"
-F 6 "vendor2, thru w hem" V 1130 2600 60  0001 C CNN "Field3"
-F 7 "vendor2, smd w hem" V 1130 2600 60  0001 C CNN "Field4"
-F 8 "reverse,V" V 1130 2600 60  0001 C CNN "Field5"
-F 9 "current,A" V 1130 2600 60  0001 C CNN "Field6"
-F 10 "x" V 1130 2600 60  0001 C CNN "Field7"
-F 11 "other,more,stuff" V 1130 2600 60  0001 C CNN "Field8"
-	1    2800 1550
-	0    -1   -1   0
-$EndComp
-Text HLabel 1950 1350 0    60   Input ~ 0
-digi_vcc
-$Comp
 L ZENER D30
