File: ignition2.sch (KiCad schematic (older format))
At the start: 9 parts, among them P14 CONN_1, P15 CONN_1, Q5 MOSFET_N, SW5 SWITCH_INV

Commit message: Removed LM1815 options. Now adaptive mode and square waves are the default,
Parts:
- D29: Field1 (none) -> newark,58k2469; Field2 (none) -> vendor1, smd w hem; Field3 (none) -> vendor2, thru w hem; Field4 (none) -> vendor2, smd w hem; Field5 (none) -> x,x; Field6 (none) -> x,x; Field7 (none) -> green; Field8 (none) -> other,more,stuff
- Q5: Field1 (none) -> digi,PIP3104-ND; Field2 (none) -> vendor1, smd w hem; Field3 (none) -> vendor2, thru w hem; Field4 (none) -> vendor2, smd w hem; Field5 (none) -> 8,A; Field6 (none) -> x,x; Field7 (none) -> TOPFET; Field8 (none) -> other,more,stuff
- R39, R40: Field1 (none) -> newark,38k0327; Field2 (none) -> vendor1, smd w hem; Field3 (none) -> vendor2, thru w hem; Field4 (none) -> vendor2, smd w hem; Field5 (none) -> 250,mW; Field6 (none) -> 5,%; Field7 (none) -> carbon film; Field8 (none) -> other,more,stuff
- R41: Field1 (none) -> newark,38k0340; Field2 (none) -> vendor1, smd w hem; Field3 (none) -> vendor2, thru w hem; Field4 (none) -> vendor2, smd w hem; Field5 (none) -> 1/4,W; Field6 (none) -> 5,%; Field7 (none) -> carbon film; Field8 (none) -> other,more,stuff
- R42: Field1 (none) -> newark,38K0328; Field2 (none) -> vendor1, smd w hem; Field3 (none) -> vendor2, thru w hem; Field4 (none) -> vendor2, smd w hem; Field5 (none) -> 250,mW; Field6 (none) -> 5,%; Field7 (none) -> carbon film; Field8 (none) -> other,more,stuff
Changed lines of the file:
@@
-EESchema Schematic File Version 1
-LIBS:power,./freeEMS_lib,device,conn,linear,regul,74xx,cmos4000,adc-dac,memory,xilinx,special,microcontrollers,dsp,microchip,analog_switches,motorola,texas,intel,audio,interface,digital-audio,philips,display,cypress,siliconi,contrib,valves,./freeEMS_1.cache
+EESchema Schematic File Version 2  date Fri 02 Jul 2010 02:24:35 PM ART
+LIBS:power
+LIBS:freeEMS_lib
+LIBS:device
+LIBS:conn
+LIBS:linear
+LIBS:regul
+LIBS:74xx
+LIBS:cmos4000
+LIBS:adc-dac
+LIBS:memory
+LIBS:xilinx
+LIBS:special
+LIBS:microcontrollers
+LIBS:dsp
+LIBS:microchip
+LIBS:analog_switches
+LIBS:motorola
+LIBS:texas
+LIBS:intel
+LIBS:audio
+LIBS:interface
+LIBS:digital-audio
+LIBS:philips
+LIBS:display
+LIBS:cypress
+LIBS:siliconi
+LIBS:contrib
+LIBS:valves
+LIBS:freeEMS_1-cache
 EELAYER 23  0
 EELAYER END
@@
 Sheet 14 41
 Title "freeEMS 1.0"
-Date "15 nov 2008"
+Date "2 jul 2010"
 Rev "A.20"
 Comp "diyefi.org"
@@
 U 1 1 48B16ED5
 P 4000 2050
-F 0 "Q5" H 4010 2220 60  0000 R C
-F 1 "MOSFET_N" H 4010 1900 60  0000 R C
-F 2 "TO220_sm" V 3930 2800 60  0001 C C
-F 4 "digi,PIP3104-ND" V 2130 3800 60  0001 C C
-F 5 "vendor1, smd w hem" V 2130 3800 60  0001 C C
-F 6 "vendor2, thru w hem" V 2130 3800 60  0001 C C
-F 7 "vendor2, smd w hem" V 2130 3800 60  0001 C C
-F 8 "8,A" V 2130 3800 60  0001 C C
-F 9 "x,x" V 2130 3800 60  0001 C C
-F 10 "TOPFET" V 2130 3800 60  0001 C C
-F 11 "other,more,stuff" V 2130 3800 60  0001 C C
+F 0 "Q5" H 4010 2220 60  0000 R CNN
+F 1 "MOSFET_N" H 4010 1900 60  0000 R CNN
+F 2 "TO220_sm" V 3930 2800 60  0001 C CNN
+F 4 "digi,PIP3104-ND" V 2130 3800 60  0001 C CNN "Field1"
+F 5 "vendor1, smd w hem" V 2130 3800 60  0001 C CNN "Field2"
+F 6 "vendor2, thru w hem" V 2130 3800 60  0001 C CNN "Field3"
+F 7 "vendor2, smd w hem" V 2130 3800 60  0001 C CNN "Field4"
+F 8 "8,A" V 2130 3800 60  0001 C CNN "Field5"
+F 9 "x,x" V 2130 3800 60  0001 C CNN "Field6"
+F 10 "TOPFET" V 2130 3800 60  0001 C CNN "Field7"
+F 11 "other,more,stuff" V 2130 3800 60  0001 C CNN "Field8"
 	1    4000 2050
 	1    0    0    -1
@@
 U 1 1 48AE08BB
 P 3400 2300
-F 0 "R42" V 3480 2300 50  0000 C C
-F 1 "10k" V 3400 2300 50  0000 C C
-F 2 "R4-SM0805" V 3580 2400 60  0001 C C
-F 4 "newark,38K0328" V 1230 2850 60  0001 C C
-F 5 "vendor1, smd w hem" V 1230 2850 60  0001 C C
-F 6 "vendor2, thru w hem" V 1230 2850 60  0001 C C
-F 7 "vendor2, smd w hem" V 1230 2850 60  0001 C C
-F 8 "250,mW" V 1230 2850 60  0001 C C
-F 9 "5,%" V 1230 2850 60  0001 C C
-F 10 "carbon film" V 1230 2850 60  0001 C C
-F 11 "other,more,stuff" V 1230 2850 60  0001 C C
+F 0 "R42" V 3480 2300 50  0000 C CNN
+F 1 "10k" V 3400 2300 50  0000 C CNN
+F 2 "R4-SM0805" V 3580 2400 60  0001 C CNN
+F 4 "newark,38K0328" V 1230 2850 60  0001 C CNN "Field1"
+F 5 "vendor1, smd w hem" V 1230 2850 60  0001 C CNN "Field2"
+F 6 "vendor2, thru w hem" V 1230 2850 60  0001 C CNN "Field3"
+F 7 "vendor2, smd w hem" V 1230 2850 60  0001 C CNN "Field4"
+F 8 "250,mW" V 1230 2850 60  0001 C CNN "Field5"
+F 9 "5,%" V 1230 2850 60  0001 C CNN "Field6"
+F 10 "carbon film" V 1230 2850 60  0001 C CNN "Field7"
+F 11 "other,more,stuff" V 1230 2850 60  0001 C CNN "Field8"
 	1    3400 2300
 	-1   0    0    1
@@
 U 1 1 48AE0832
 P 2450 1450
-F 0 "SW5" H 2250 1600 50  0000 C C
-F 1 "SWITCH_INV" H 2300 1300 50  0000 C C
-F 2 "SIL-3" H 2350 1700 60  0001 C C
+F 0 "SW5" H 2250 1600 50  0000 C CNN
+F 1 "SWITCH_INV" H 2300 1300 50  0000 C CNN
+F 2 "SIL-3" H 2350 1700 60  0001 C CNN
 	1    2450 1450
 	-1   0    0    -1
@@
 U 1 1 48AA2529
 P 3850 1650
-F 0 "D29" H 3850 1750 50  0000 C C
-F 1 "LED" H 3850 1550 50  0000 C C
-F 2 "LEDV" V 1680 5050 60  0001 C C
-F 4 "newark,58k2469" V 430 2100 60  0001 C C
-F 5 "vendor1, smd w hem" V 430 2100 60  0001 C C
-F 6 "vendor2, thru w hem" V 430 2100 60  0001 C C
-F 7 "vendor2, smd w hem" V 430 2100 60  0001 C C
-F 8 "x,x" V 430 2100 60  0001 C C
-F 9 "x,x" V 430 2100 60  0001 C C
-F 10 "green" V 430 2100 60  0001 C C
-F 11 "other,more,stuff" V 430 2100 60  0001 C C
+F 0 "D29" H 3850 1750 50  0000 C CNN
+F 1 "LED" H 3850 1550 50  0000 C CNN
+F 2 "LEDV" V 1680 5050 60  0001 C CNN
+F 4 "newark,58k2469" V 430 2100 60  0001 C CNN "Field1"
+F 5 "vendor1, smd w hem" V 430 2100 60  0001 C CNN "Field2"
+F 6 "vendor2, thru w hem" V 430 2100 60  0001 C CNN "Field3"
+F 7 "vendor2, smd w hem" V 430 2100 60  0001 C CNN "Field4"
+F 8 "x,x" V 430 2100 60  0001 C CNN "Field5"
+F 9 "x,x" V 430 2100 60  0001 C CNN "Field6"
+F 10 "green" V 430 2100 60  0001 C CNN "Field7"
+F 11 "other,more,stuff" V 430 2100 60  0001 C CNN "Field8"
 	1    3850 1650
 	1    0    0    -1
@@
 U 1 1 48AA2523
 P 3300 1650
-F 0 "R41" V 3380 1650 50  0000 C C
-F 1 "3k" V 3300 1650 50  0000 C C
-F 2 "R4-SM0805" V 1980 1650 60  0001 C C
-F 4 "newark,38k0340" V -120 2400 60  0001 C C
-F 5 "vendor1, smd w hem" V -120 2400 60  0001 C C
-F 6 "vendor2, thru w hem" V -120 2400 60  0001 C C
-F 7 "vendor2, smd w hem" V -120 2400 60  0001 C C
-F 8 "1/4,W" V -120 2400 60  0001 C C
-F 9 "5,%" V -120 2400 60  0001 C C
-F 10 "carbon film" V -120 2400 60  0001 C C
-F 11 "other,more,stuff" V -120 2400 60  0001 C C
+F 0 "R41" V 3380 1650 50  0000 C CNN
+F 1 "3k" V 3300 1650 50  0000 C CNN
+F 2 "R4-SM0805" V 1980 1650 60  0001 C CNN
+F 4 "newark,38k0340" V -120 2400 60  0001 C CNN "Field1"
+F 5 "vendor1, smd w hem" V -120 2400 60  0001 C CNN "Field2"
+F 6 "vendor2, thru w hem" V -120 2400 60  0001 C CNN "Field3"
+F 7 "vendor2, smd w hem" V -120 2400 60  0001 C CNN "Field4"
+F 8 "1/4,W" V -120 2400 60  0001 C CNN "Field5"
+F 9 "5,%" V -120 2400 60  0001 C CNN "Field6"
+F 10 "carbon film" V -120 2400 60  0001 C CNN "Field7"
+F 11 "other,more,stuff" V -120 2400 60  0001 C CNN "Field8"
 	1    3300 1650
 	0    1    1    0
@@
 U 1 1 48AA1A4E
 P 5450 2650
-F 0 "P15" H 5530 2650 40  0000 L C
-F 1 "CONN_1" H 5450 2705 30  0001 C C
-F 2 "1PIN" V 1880 2850 60  0001 C C
+F 0 "P15" H 5530 2650 40  0000 L CNN
+F 1 "CONN_1" H 5450 2705 30  0001 C CNN
+F 2 "1PIN" V 1880 2850 60  0001 C CNN
 	1    5450 2650
 	1    0    0    -1
@@
 U 1 1 48AA1A4A
 P 5450 2200
-F 0 "P14" H 5530 2200 40  0000 L C
-F 1 "CONN_1" H 5450 2255 30  0001 C C
-F 2 "1PIN" V 1880 2600 60  0001 C C
+F 0 "P14" H 5530 2200 40  0000 L CNN
+F 1 "CONN_1" H 5450 2255 30  0001 C CNN
+F 2 "1PIN" V 1880 2600 60  0001 C CNN
 	1    5450 2200
 	1    0    0    -1
 $EndComp
-Text GLabel 1750 1550 0    60   Input
+Text HLabel 1750 1550 0    60   Input ~ 0
 5V_reg
 $Comp
@@
 U 1 1 489395E6
 P 3100 2050
-F 0 "R39" V 3180 2050 50  0000 C C
-F 1 "1k" V 3100 2050 50  0000 C C
-F 2 "R4-SM0805" V 3280 2150 60  0001 C C
-F 4 "newark,38k0327" V 930 2600 60  0001 C C
-F 5 "vendor1, smd w hem" V 930 2600 60  0001 C C
-F 6 "vendor2, thru w hem" V 930 2600 60  0001 C C
-F 7 "vendor2, smd w hem" V 930 2600 60  0001 C C
-F 8 "250,mW" V 930 2600 60  0001 C C
-F 9 "5,%" V 930 2600 60  0001 C C
-F 10 "carbon film" V 930 2600 60  0001 C C
-F 11 "other,more,stuff" V 930 2600 60  0001 C C
+F 0 "R39" V 3180 2050 50  0000 C CNN
+F 1 "1k" V 3100 2050 50  0000 C CNN
+F 2 "R4-SM0805" V 3280 2150 60  0001 C CNN
+F 4 "newark,38k0327" V 930 2600 60  0001 C CNN "Field1"
+F 5 "vendor1, smd w hem" V 930 2600 60  0001 C CNN "Field2"
+F 6 "vendor2, thru w hem" V 930 2600 60  0001 C CNN "Field3"
+F 7 "vendor2, smd w hem" V 930 2600 60  0001 C CNN "Field4"
+F 8 "250,mW" V 930 2600 60  0001 C CNN "Field5"
+F 9 "5,%" V 930 2600 60  0001 C CNN "Field6"
+F 10 "carbon film" V 930 2600 60  0001 C CNN "Field7"
+F 11 "other,more,stuff" V 930 2600 60  0001 C CNN "Field8"
 	1    3100 2050
 	0    1    1    0
@@
 U 1 1 489395D4
 P 3300 1450
-F 0 "R40" V 3380 1450 50  0000 C C
-F 1 "1k" V 3300 1450 50  0000 C C
-F 2 "R4-SM0805" V 3480 1550 60  0001 C C
-F 4 "newark,38k0327" V 1130 2350 60  0001 C C
-F 5 "vendor1, smd w hem" V 1130 2350 60  0001 C C
-F 6 "vendor2, thru w hem" V 1130 2350 60  0001 C C
-F 7 "vendor2, smd w hem" V 1130 2350 60  0001 C C
-F 8 "250,mW" V 1130 2350 60  0001 C C
-F 9 "5,%" V 1130 2350 60  0001 C C
-F 10 "carbon film" V 1130 2350 60  0001 C C
-F 11 "other,more,stuff" V 1130 2350 60  0001 C C
+F 0 "R40" V 3380 1450 50  0000 C CNN
+F 1 "1k" V 3300 1450 50  0000 C CNN
+F 2 "R4-SM0805" V 3480 1550 60  0001 C CNN
+F 4 "newark,38k0327" V 1130 2350 60  0001 C CNN "Field1"
+F 5 "vendor1, smd w hem" V 1130 2350 60  0001 C CNN "Field2"
+F 6 "vendor2, thru w hem" V 1130 2350 60  0001 C CNN "Field3"
+F 7 "vendor2, smd w hem" V 1130 2350 60  0001 C CNN "Field4"
+F 8 "250,mW" V 1130 2350 60  0001 C CNN "Field5"
+F 9 "5,%" V 1130 2350 60  0001 C CNN "Field6"
+F 10 "carbon film" V 1130 2350 60  0001 C CNN "Field7"
+F 11 "other,more,stuff" V 1130 2350 60  0001 C CNN "Field8"
 	1    3300 1450
 	0    1    1    0
 $EndComp
-Text GLabel 1750 1350 0    60   Input
+Text HLabel 1750 1350 0    60   Input ~ 0
 12V_bat
-Text GLabel 2750 2650 0    60   BiDi
+Text HLabel 2750 2650 0    60   BiDi ~ 0
 low_power_inductive_gnd
-Text GLabel 2800 2050 0    60   Input
+Text HLabel 2800 2050 0    60   Input ~ 0
 low_power_inductive_drive
 $EndSCHEMATC

Commit message: Implemented P&H, removed current sense circuitry, removed all unnecessary files from the repo
Parts:
- renumbered D29 to D?, P14 to P?, P15 to P?, Q5 to Q?, R40 to R?, R39 to R?, R41 to R?, R42 to R?, SW5 to SW?
Changed lines of the file:
@@
-EESchema Schematic File Version 2  date Fri 02 Jul 2010 05:44:26 PM ART
+EESchema Schematic File Version 2  date Sat 03 Jul 2010 10:49:02 AM ART
 LIBS:power
 LIBS:freeEMS_lib
@@
 EELAYER END
 $Descr A4 11700 8267
-Sheet 14 41
+Sheet 1 41
 Title "freeEMS 1.0"
-Date "2 jul 2010"
-Rev "A.20"
+Date "3 jul 2010"
+Rev "A.07"
 Comp "diyefi.org"
 Comment1 "ignition.sch"
@@
 Connection ~ 3400 2050
 $Comp
-L PIP-3104 Q5
+L PIP-3104 Q?
 U 1 1 48B16ED5
 P 4000 2050
-F 0 "Q5" H 4010 2220 60  0000 R CNN
+F 0 "Q?" H 4010 2220 60  0000 R CNN
 F 1 "MOSFET_N" H 4010 1900 60  0000 R CNN
 F 2 "TO220_sm" V 3930 2800 60  0001 C CNN
@@
 $EndComp
 $Comp
-L R R42
+L R R?
 U 1 1 48AE08BB
 P 3400 2300
-F 0 "R42" V 3480 2300 50  0000 C CNN
+F 0 "R?" V 3480 2300 50  0000 C CNN
 F 1 "10k" V 3400 2300 50  0000 C CNN
 F 2 "R4-SM0805" V 3580 2400 60  0001 C CNN
@@
 $EndComp
 $Comp
-L SWITCH_INV SW5
+L SWITCH_INV SW?
 U 1 1 48AE0832
 P 2450 1450
-F 0 "SW5" H 2250 1600 50  0000 C CNN
+F 0 "SW?" H 2250 1600 50  0000 C CNN
 F 1 "SWITCH_INV" H 2300 1300 50  0000 C CNN
 F 2 "SIL-3" H 2350 1700 60  0001 C CNN
@@
 $EndComp
 $Comp
-L LED D29
+L LED D?
 U 1 1 48AA2529
 P 3850 1650
-F 0 "D29" H 3850 1750 50  0000 C CNN
+F 0 "D?" H 3850 1750 50  0000 C CNN
 F 1 "LED" H 3850 1550 50  0000 C CNN
 F 2 "LEDV" V 1680 5050 60  0001 C CNN
@@
 $EndComp
 $Comp
-L R R41
+L R R?
 U 1 1 48AA2523
 P 3300 1650
-F 0 "R41" V 3380 1650 50  0000 C CNN
+F 0 "R?" V 3380 1650 50  0000 C CNN
 F 1 "3k" V 3300 1650 50  0000 C CNN
 F 2 "R4-SM0805" V 1980 1650 60  0001 C CNN
@@
 $EndComp
 $Comp
-L CONN_1 P15
+L CONN_1 P?
 U 1 1 48AA1A4E
 P 5450 2650
-F 0 "P15" H 5530 2650 40  0000 L CNN
+F 0 "P?" H 5530 2650 40  0000 L CNN
 F 1 "CONN_1" H 5450 2705 30  0001 C CNN
 F 2 "1PIN" V 1880 2850 60  0001 C CNN
@@
 $EndComp
 $Comp
-L CONN_1 P14
+L CONN_1 P?
 U 1 1 48AA1A4A
 P 5450 2200
-F 0 "P14" H 5530 2200 40  0000 L CNN
+F 0 "P?" H 5530 2200 40  0000 L CNN
 F 1 "CONN_1" H 5450 2255 30  0001 C CNN
 F 2 "1PIN" V 1880 2600 60  0001 C CNN
@@
 5V_reg
 $Comp
-L R R39
+L R R?
 U 1 1 489395E6
 P 3100 2050
-F 0 "R39" V 3180 2050 50  0000 C CNN
+F 0 "R?" V 3180 2050 50  0000 C CNN
 F 1 "1k" V 3100 2050 50  0000 C CNN
 F 2 "R4-SM0805" V 3280 2150 60  0001 C CNN
@@
 $EndComp
 $Comp
-L R R40
+L R R?
 U 1 1 489395D4
 P 3300 1450
-F 0 "R40" V 3380 1450 50  0000 C CNN
+F 0 "R?" V 3380 1450 50  0000 C CNN
 F 1 "1k" V 3300 1450 50  0000 C CNN
 F 2 "R4-SM0805" V 3480 1550 60  0001 C CNN

Commit message: Corrected ERC errors by fixing the custom FreeEMS components pinouts
Parts:
- removed D?: LED, LEDV, symbol LED
- removed P?: CONN_1, 1PIN, symbol CONN_1
- removed Q?: MOSFET_N, TO220_sm, symbol PIP-3104
- removed R? (x2): 1k, R4-SM0805, symbol R
- removed R?: 3k, R4-SM0805, symbol R
- removed R?: 10k, R4-SM0805, symbol R
- removed SW?: SWITCH_INV, SIL-3, symbol SWITCH_INV
- added D21: LED, LEDV, symbol LED
- added P14: CONN_1, 1PIN, symbol CONN_1
- added Q5: MOSFET_N, TO220_sm, symbol PIP-3104
- added R31, R32: 1k, R4-SM0805, symbol R
- added R33: 3k, R4-SM0805, symbol R
- added R34: 10k, R4-SM0805, symbol R
- added SW5: SWITCH_INV, SIL-3, symbol SWITCH_INV
- gave numbers to parts that had none: 1
Connections:
- net 12V_bat: now also SW5.1
- net 5V_reg: now also SW5.3
- net low_power_inductive_drive: now also R31.2
- net low_power_inductive_gnd: now also Q5.3 (S), R34.1
- new net: D21.2 (K), P14.1, Q5.2 (D), R32.1
- new net: R32.2, R33.2, SW5.2
- new net: Q5.1 (I), R31.1, R34.2
- new net: D21.1 (A), R33.1
Changed lines of the file:
@@
-EESchema Schematic File Version 2  date Sat 03 Jul 2010 10:49:02 AM ART
+EESchema Schematic File Version 2  date Sat 03 Jul 2010 12:32:24 PM ART
 LIBS:power
 LIBS:freeEMS_lib
@@
 Connection ~ 3400 2050
 $Comp
-L PIP-3104 Q?
-U 1 1 48B16ED5
+L PIP-3104 Q5
+U 1 1 4C2F5332
 P 4000 2050
-F 0 "Q?" H 4010 2220 60  0000 R CNN
+F 0 "Q5" H 4010 2220 60  0000 R CNN
 F 1 "MOSFET_N" H 4010 1900 60  0000 R CNN
 F 2 "TO220_sm" V 3930 2800 60  0001 C CNN
@@
 $EndComp
 $Comp
-L R R?
-U 1 1 48AE08BB
+L R R34
+U 1 1 4C2F532D
 P 3400 2300
-F 0 "R?" V 3480 2300 50  0000 C CNN
+F 0 "R34" V 3480 2300 50  0000 C CNN
 F 1 "10k" V 3400 2300 50  0000 C CNN
 F 2 "R4-SM0805" V 3580 2400 60  0001 C CNN
@@
 $EndComp
 $Comp
-L SWITCH_INV SW?
-U 1 1 48AE0832
+L SWITCH_INV SW5
+U 1 1 4C2F5328
 P 2450 1450
-F 0 "SW?" H 2250 1600 50  0000 C CNN
+F 0 "SW5" H 2250 1600 50  0000 C CNN
 F 1 "SWITCH_INV" H 2300 1300 50  0000 C CNN
 F 2 "SIL-3" H 2350 1700 60  0001 C CNN
@@
 $EndComp
 $Comp
-L LED D?
-U 1 1 48AA2529
+L LED D21
+U 1 1 4C2F5322
 P 3850 1650
-F 0 "D?" H 3850 1750 50  0000 C CNN
+F 0 "D21" H 3850 1750 50  0000 C CNN
 F 1 "LED" H 3850 1550 50  0000 C CNN
 F 2 "LEDV" V 1680 5050 60  0001 C CNN
@@
 $EndComp
 $Comp
-L R R?
-U 1 1 48AA2523
+L R R33
+U 1 1 4C2F531E
 P 3300 1650
-F 0 "R?" V 3380 1650 50  0000 C CNN
+F 0 "R33" V 3380 1650 50  0000 C CNN
 F 1 "3k" V 3300 1650 50  0000 C CNN
 F 2 "R4-SM0805" V 1980 1650 60  0001 C CNN
@@
 $EndComp
 $Comp
-L CONN_1 P?
+L CONN_1 P15
 U 1 1 48AA1A4E
 P 5450 2650
-F 0 "P?" H 5530 2650 40  0000 L CNN
+F 0 "P15" H 5530 2650 40  0000 L CNN
 F 1 "CONN_1" H 5450 2705 30  0001 C CNN
 F 2 "1PIN" V 1880 2850 60  0001 C CNN
@@
 $EndComp
 $Comp
-L CONN_1 P?
-U 1 1 48AA1A4A
+L CONN_1 P14
+U 1 1 4C2F5312
 P 5450 2200
-F 0 "P?" H 5530 2200 40  0000 L CNN
+F 0 "P14" H 5530 2200 40  0000 L CNN
 F 1 "CONN_1" H 5450 2255 30  0001 C CNN
 F 2 "1PIN" V 1880 2600 60  0001 C CNN
@@
 5V_reg
 $Comp
-L R R?
-U 1 1 489395E6
+L R R31
+U 1 1 4C2F52E8
 P 3100 2050
-F 0 "R?" V 3180 2050 50  0000 C CNN
+F 0 "R31" V 3180 2050 50  0000 C CNN
 F 1 "1k" V 3100 2050 50  0000 C CNN
 F 2 "R4-SM0805" V 3280 2150 60  0001 C CNN
@@
 $EndComp
 $Comp
-L R R?
-U 1 1 489395D4
+L R R32
+U 1 1 4C2F52E1
 P 3300 1450
-F 0 "R?" V 3380 1450 50  0000 C CNN
+F 0 "R32" V 3380 1450 50  0000 C CNN
 F 1 "1k" V 3300 1450 50  0000 C CNN
 F 2 "R4-SM0805" V 3480 1550 60  0001 C CNN
