File: power_reg1.sch (KiCad schematic (older format))
At the start: 10 parts, among them U4 7805-DIYEFI

Commit message: Removed LM1815 options. Now adaptive mode and square waves are the default,
Parts:
- C10: Field1 (none) -> newark,69K8230; Field2 (none) -> vendor1, smd w hem; Field3 (none) -> vendor2, thru w hem; Field4 (none) -> vendor2, smd w hem; Field5 (none) -> 50,V; Field6 (none) -> x,x; Field7 (none) -> Aluminum Electrolytic; Field8 (none) -> other,more,stuff
- C11, C8: Field1 (none) -> newark,97M4217; Field2 (none) -> vendor1, smd w hem; Field3 (none) -> vendor2, thru w hem; Field4 (none) -> vendor2, smd w hem; Field5 (none) -> 35,V; Field6 (none) -> 10,%; Field7 (none) -> Tantalum; Field8 (none) -> other,more,stuff
- C12, C9: Field1 (none) -> newark,97M4164; Field2 (none) -> vendor1, smd w hem; Field3 (none) -> vendor2, thru w hem; Field4 (none) -> vendor2, smd w hem; Field5 (none) -> 50,V; Field6 (none) -> 20,%; Field7 (none) -> multilayer ceramic; Field8 (none) -> other,more,stuff
- C7: Field1 (none) -> newark,69K8230; Field2 (none) -> vendor1, smd w hem; Field3 (none) -> vendor2, thru w hem; Field4 (none) -> vendor2, smd w hem; Field5 (none) -> 50,V; Field6 (none) -> X,%; Field7 (none) -> Aluminum Electrolytic; Field8 (none) -> other,more,stuff
- D11, D12: Field1 (none) -> newark,18C8923; Field2 (none) -> DIGI,S1MBDIDKR-ND; Field3 (none) -> DIGI,1N4007RLOSCT-ND; Field4 (none) -> vendor2, smd w hem; Field5 (none) -> max,V; Field6 (none) -> x,x; Field7 (none) -> construct; Field8 (none) -> other,more,stuff
- R10: Field1 (none) -> newark, 65K3871; Field2 (none) -> farnell,1155286; Field3 (none) -> vendor2, thru w hem; Field4 (none) -> vendor2, smd w hem; Field5 (none) -> power,W; Field6 (none) -> tol,%; Field7 (none) -> construct; Field8 (none) -> other,more,stuff
- U4: Field1 (none) -> newark,45J1442; Field2 (none) -> vendor1, smd w hem; Field3 (none) -> vendor2, thru w hem; Field4 (none) -> vendor2, smd w hem; Field5 (none) -> x,x; Field6 (none) -> x,x; Field7 (none) -> linear; Field8 (none) -> other,more,stuff

Commit message: Implemented P&H, removed current sense circuitry, removed all unnecessary files from the repo
Parts:
- C?: renamed from C9; Field1 newark,97M4164 -> newark,56K3664
- C?: renamed from C12; Field1 newark,97M4164 -> newark,56K3664
- D?: renamed from D12; Field1 newark,18C8923 -> DIGI,1N4007RLOSCT-ND; Field3 DIGI,1N4007RLOSCT-ND -> newark,18C8923
- renumbered C11 to C?, C8 to C?, C10 to C?, C7 to C?, D11 to D?, R10 to R?, U4 to U?
Changed lines of the file:
@@
-EESchema Schematic File Version 2  date Fri 02 Jul 2010 05:44:26 PM ART
+EESchema Schematic File Version 2  date Sat 03 Jul 2010 10:49:02 AM ART
 LIBS:power
 LIBS:freeEMS_lib
@@
 EELAYER END
 $Descr A 11000 8500
-Sheet 3 41
+Sheet 1 41
 Title "freeEMS 1.0"
-Date "2 jul 2010"
-Rev "A.20"
+Date "3 jul 2010"
+Rev "A.07"
 Comp "diyefi.org"
 Comment1 "power_reg.sch"
@@
 $EndDescr
 $Comp
-L 7805-DIYEFI U4
+L 7805-DIYEFI U?
 U 1 1 48B14C8F
 P 5800 3350
-F 0 "U4" H 5950 3154 60  0000 C CNN
+F 0 "U?" H 5950 3154 60  0000 C CNN
 F 1 "7805-DIYEFI" H 5800 3550 60  0000 C CNN
 F 2 "TO220_sm" V 2630 2600 60  0001 C CNN
@@
 Connection ~ 5350 3300
 Wire Wire Line
-	5350 3300 5350 2900
-Wire Wire Line
-	5350 2900 5600 2900
+	5350 2900 5350 3300
+Wire Wire Line
+	5600 2900 5350 2900
 Connection ~ 6550 3700
 Connection ~ 6550 3300
@@
 Connection ~ 6250 3300
 $Comp
-L C C7
+L C C?
 U 1 1 4895133C
 P 4400 3500
-F 0 "C7" H 4450 3600 50  0000 L CNN
+F 0 "C?" H 4450 3600 50  0000 L CNN
 F 1 "2200uF" H 4450 3400 50  0000 L CNN
 F 2 "C1V7" V -170 2600 60  0001 C CNN
@@
 $EndComp
 $Comp
-L C C10
+L C C?
 U 1 1 489512E0
 P 6550 3500
-F 0 "C10" H 6600 3600 50  0000 L CNN
+F 0 "C?" H 6600 3600 50  0000 L CNN
 F 1 "2200uF" H 6600 3400 50  0000 L CNN
 F 2 "C1V7" V 4130 2600 60  0001 C CNN
@@
 gnd
 $Comp
-L C C12
+L C C?
 U 1 1 486ED024
 P 7450 3500
-F 0 "C12" H 7500 3600 50  0000 L CNN
+F 0 "C?" H 7500 3600 50  0000 L CNN
 F 1 ".1uF" H 7500 3400 50  0000 L CNN
 F 2 "C1V7" V 5930 2600 60  0001 C CNN
-F 4 "newark,97M4164" V 5930 2600 60  0001 C CNN "Field1"
+F 4 "newark,56K3664" V 5930 2600 60  0001 C CNN "Field1"
 F 5 "vendor1, smd w hem" V 5930 2600 60  0001 C CNN "Field2"
 F 6 "vendor2, thru w hem" V 5930 2600 60  0001 C CNN "Field3"
@@
 $EndComp
 $Comp
-L DIODE D11
+L DIODE D?
 U 1 1 486ECB4E
 P 2850 3300
-F 0 "D11" H 2850 3400 40  0000 C CNN
+F 0 "D?" H 2850 3400 40  0000 C CNN
 F 1 "1N4007" H 2850 3200 40  0000 C CNN
 F 2 "D4-SMB" H 2950 3500 60  0001 C CNN
@@
 $EndComp
 $Comp
-L DIODE D12
+L DIODE D?
 U 1 1 486ECB44
 P 5800 2900
-F 0 "D12" H 5800 3000 40  0000 C CNN
+F 0 "D?" H 5800 3000 40  0000 C CNN
 F 1 "1N4007" H 5800 2800 40  0000 C CNN
 F 2 "D4-SMB" H 8850 3500 60  0001 C CNN
-F 4 "newark,18C8923" H 8850 3500 60  0001 C CNN "Field1"
+F 4 "DIGI,1N4007RLOSCT-ND" H 8850 3500 60  0001 C CNN "Field1"
 F 5 "DIGI,S1MBDIDKR-ND" H 8850 3500 60  0001 C CNN "Field2"
-F 6 "DIGI,1N4007RLOSCT-ND" H 2630 2600 60  0001 C CNN "Field3"
+F 6 "newark,18C8923" H 2630 2600 60  0001 C CNN "Field3"
 F 7 "vendor2, smd w hem" H 2630 2600 60  0001 C CNN "Field4"
 F 8 "max,V" H 2630 2600 60  0001 C CNN "Field5"
@@
 $EndComp
 $Comp
-L VSS #PWR023
+L VSS #PWR?
 U 1 1 486CA95E
 P 7850 3750
-F 0 "#PWR023" H 7850 3750 30  0001 C CNN
+F 0 "#PWR?" H 7850 3750 30  0001 C CNN
 F 1 "VSS" H 7850 3680 30  0000 C CNN
 	1    7850 3750
@@
 $EndComp
 $Comp
-L R R10
+L R R?
 U 1 1 486CA8FD
 P 3350 3300
-F 0 "R10" V 3430 3300 50  0000 C CNN
+F 0 "R?" V 3430 3300 50  0000 C CNN
 F 1 "1R" V 3350 3300 50  0000 C CNN
 F 2 "R7" V 3530 3400 60  0001 C CNN
@@
 $EndComp
 $Comp
-L CAPAPOL C8
+L CAPAPOL C?
 U 1 1 486CA8EA
 P 4850 3500
-F 0 "C8" H 4900 3600 50  0000 L CNN
+F 0 "C?" H 4900 3600 50  0000 L CNN
 F 1 "10uF" H 4900 3400 50  0000 L CNN
 F 2 "C1V7" V 730 2600 60  0001 C CNN
@@
 $EndComp
 $Comp
-L CAPAPOL C11
+L CAPAPOL C?
 U 1 1 486CA8E4
 P 7000 3500
-F 0 "C11" H 7050 3600 50  0000 L CNN
+F 0 "C?" H 7050 3600 50  0000 L CNN
 F 1 "10uF" H 7050 3400 50  0000 L CNN
 F 2 "C1V7" V 5030 2600 60  0001 C CNN
@@
 $EndComp
 $Comp
-L C C9
+L C C?
 U 1 1 486CA8CD
 P 5250 3500
-F 0 "C9" H 5300 3600 50  0000 L CNN
+F 0 "C?" H 5300 3600 50  0000 L CNN
 F 1 ".1uF" H 5300 3400 50  0000 L CNN
 F 2 "C1V7" V 1530 2600 60  0001 C CNN
-F 4 "newark,97M4164" V 1530 2600 60  0001 C CNN "Field1"
+F 4 "newark,56K3664" V 1530 2600 60  0001 C CNN "Field1"
 F 5 "vendor1, smd w hem" V 1530 2600 60  0001 C CNN "Field2"
 F 6 "vendor2, thru w hem" V 1530 2600 60  0001 C CNN "Field3"
@@
 $EndComp
 $Comp
-L GND #PWR024
+L GND #PWR?
 U 1 1 486CA86E
 P 2600 3750
-F 0 "#PWR024" H 2600 3750 30  0001 C CNN
+F 0 "#PWR?" H 2600 3750 30  0001 C CNN
 F 1 "GND" H 2600 3680 30  0001 C CNN
 	1    2600 3750

Commit message: Corrected ERC errors by fixing the custom FreeEMS components pinouts
Parts:
- removed C?: .1uF, C1V7, symbol C
- removed C? (x2): 2200uF, C1V7, symbol C
- removed D? (x2): 1N4007, D4-SMB, symbol DIODE
- added C10, C7: 2200uF, C1V7, symbol C
- added C12: .1uF, C1V7, symbol C
- added D3, D4: 1N4007, D4-SMB, symbol DIODE
- gave numbers to parts that had none: 5
Changed lines of the file:
@@
-EESchema Schematic File Version 2  date Sat 03 Jul 2010 10:49:02 AM ART
+EESchema Schematic File Version 2  date Sat 03 Jul 2010 12:32:24 PM ART
 LIBS:power
 LIBS:freeEMS_lib
@@
 EELAYER END
 $Descr A 11000 8500
-Sheet 1 41
+Sheet 9 41
 Title "freeEMS 1.0"
 Date "3 jul 2010"
@@
 Comment4 ""
 $EndDescr
-$Comp
-L 7805-DIYEFI U?
+Connection ~ 3500 3700
+Connection ~ 6250 3300
+Wire Wire Line
+	6250 3300 6250 2900
+Wire Wire Line
+	6250 2900 6000 2900
+Wire Wire Line
+	2500 3300 2650 3300
+Connection ~ 5800 3700
+Connection ~ 4850 3700
+Connection ~ 4850 3300
+Wire Wire Line
+	3050 3300 3100 3300
+Wire Wire Line
+	2600 3750 2600 3700
+Connection ~ 7000 3700
+Wire Wire Line
+	5800 3700 5800 3600
+Wire Wire Line
+	7850 3750 7850 3700
+Connection ~ 7000 3300
+Connection ~ 7450 3300
+Wire Wire Line
+	7850 3300 6200 3300
+Connection ~ 7450 3700
+Connection ~ 4400 3300
+Connection ~ 5250 3700
+Connection ~ 4400 3700
+Connection ~ 5250 3300
+Wire Wire Line
+	7850 3700 2600 3700
+Wire Wire Line
+	5400 3300 3600 3300
+Connection ~ 6550 3300
+Connection ~ 6550 3700
+Wire Wire Line
+	5600 2900 5350 2900
+Wire Wire Line
+	5350 2900 5350 3300
+Connection ~ 5350 3300
+$Comp
+L PWR_FLAG #FLG042
+U 1 1 4C2F56F1
+P 3500 3700
+F 0 "#FLG042" H 3500 3970 30  0001 C CNN
+F 1 "PWR_FLAG" H 3500 3930 30  0000 C CNN
+	1    3500 3700
+	1    0    0    -1
+$EndComp
+$Comp
+L PWR_FLAG #FLG043
+U 1 1 4C2F5631
+P 4850 3300
+F 0 "#FLG043" H 4850 3570 30  0001 C CNN
+F 1 "PWR_FLAG" H 4850 3530 30  0000 C CNN
+	1    4850 3300
+	1    0    0    -1
+$EndComp
+$Comp
+L 7805-DIYEFI U4
 U 1 1 48B14C8F
 P 5800 3350
-F 0 "U?" H 5950 3154 60  0000 C CNN
+F 0 "U4" H 5950 3154 60  0000 C CNN
 F 1 "7805-DIYEFI" H 5800 3550 60  0000 C CNN
 F 2 "TO220_sm" V 2630 2600 60  0001 C CNN
@@
 	1    0    0    -1
 $EndComp
-Connection ~ 5350 3300
-Wire Wire Line
-	5350 2900 5350 3300
-Wire Wire Line
-	5600 2900 5350 2900
-Connection ~ 6550 3700
-Connection ~ 6550 3300
-Wire Wire Line
-	5400 3300 3600 3300
-Wire Wire Line
-	7850 3700 2600 3700
-Connection ~ 5250 3300
-Connection ~ 4400 3700
-Connection ~ 5250 3700
-Connection ~ 4400 3300
-Connection ~ 7450 3700
-Wire Wire Line
-	7850 3300 6200 3300
-Connection ~ 7450 3300
-Connection ~ 7000 3300
-Wire Wire Line
-	7850 3700 7850 3750
-Wire Wire Line
-	5800 3700 5800 3600
-Connection ~ 7000 3700
-Wire Wire Line
-	2600 3700 2600 3750
-Wire Wire Line
-	3050 3300 3100 3300
-Connection ~ 4850 3300
-Connection ~ 4850 3700
-Connection ~ 5800 3700
-Wire Wire Line
-	2500 3300 2650 3300
-Wire Wire Line
-	6000 2900 6250 2900
-Wire Wire Line
-	6250 2900 6250 3300
-Connection ~ 6250 3300
-$Comp
-L C C?
-U 1 1 4895133C
+$Comp
+L C C7
+U 1 1 4C2F52EB
 P 4400 3500
-F 0 "C?" H 4450 3600 50  0000 L CNN
+F 0 "C7" H 4450 3600 50  0000 L CNN
 F 1 "2200uF" H 4450 3400 50  0000 L CNN
 F 2 "C1V7" V -170 2600 60  0001 C CNN
@@
 $EndComp
 $Comp
-L C C?
-U 1 1 489512E0
+L C C10
+U 1 1 4C2F52EA
 P 6550 3500
-F 0 "C?" H 6600 3600 50  0000 L CNN
+F 0 "C10" H 6600 3600 50  0000 L CNN
 F 1 "2200uF" H 6600 3400 50  0000 L CNN
 F 2 "C1V7" V 4130 2600 60  0001 C CNN
@@
 gnd
 $Comp
-L C C?
-U 1 1 486ED024
+L C C12
+U 1 1 4C2F52A3
 P 7450 3500
-F 0 "C?" H 7500 3600 50  0000 L CNN
+F 0 "C12" H 7500 3600 50  0000 L CNN
 F 1 ".1uF" H 7500 3400 50  0000 L CNN
 F 2 "C1V7" V 5930 2600 60  0001 C CNN
@@
 $EndComp
 $Comp
-L DIODE D?
-U 1 1 486ECB4E
+L DIODE D3
+U 1 1 4C2F52A2
 P 2850 3300
-F 0 "D?" H 2850 3400 40  0000 C CNN
+F 0 "D3" H 2850 3400 40  0000 C CNN
 F 1 "1N4007" H 2850 3200 40  0000 C CNN
 F 2 "D4-SMB" H 2950 3500 60  0001 C CNN
@@
 $EndComp
 $Comp
-L DIODE D?
-U 1 1 486ECB44
+L DIODE D4
+U 1 1 4C2F52A1
 P 5800 2900
-F 0 "D?" H 5800 3000 40  0000 C CNN
+F 0 "D4" H 5800 3000 40  0000 C CNN
 F 1 "1N4007" H 5800 2800 40  0000 C CNN
 F 2 "D4-SMB" H 8850 3500 60  0001 C CNN
@@
 $EndComp
 $Comp
-L VSS #PWR?
+L VSS #PWR044
 U 1 1 486CA95E
 P 7850 3750
-F 0 "#PWR?" H 7850 3750 30  0001 C CNN
+F 0 "#PWR044" H 7850 3750 30  0001 C CNN
 F 1 "VSS" H 7850 3680 30  0000 C CNN
 	1    7850 3750
@@
 $EndComp
 $Comp
-L R R?
+L R R2
 U 1 1 486CA8FD
 P 3350 3300
-F 0 "R?" V 3430 3300 50  0000 C CNN
+F 0 "R2" V 3430 3300 50  0000 C CNN
 F 1 "1R" V 3350 3300 50  0000 C CNN
 F 2 "R7" V 3530 3400 60  0001 C CNN
@@
 $EndComp
 $Comp
-L CAPAPOL C?
+L CAPAPOL C8
 U 1 1 486CA8EA
 P 4850 3500
-F 0 "C?" H 4900 3600 50  0000 L CNN
+F 0 "C8" H 4900 3600 50  0000 L CNN
 F 1 "10uF" H 4900 3400 50  0000 L CNN
 F 2 "C1V7" V 730 2600 60  0001 C CNN
@@
 $EndComp
 $Comp
-L CAPAPOL C?
+L CAPAPOL C11
 U 1 1 486CA8E4
 P 7000 3500
-F 0 "C?" H 7050 3600 50  0000 L CNN
+F 0 "C11" H 7050 3600 50  0000 L CNN
 F 1 "10uF" H 7050 3400 50  0000 L CNN
 F 2 "C1V7" V 5030 2600 60  0001 C CNN
@@
 $EndComp
 $Comp
-L C C?
+L C C9
 U 1 1 486CA8CD
 P 5250 3500
-F 0 "C?" H 5300 3600 50  0000 L CNN
+F 0 "C9" H 5300 3600 50  0000 L CNN
 F 1 ".1uF" H 5300 3400 50  0000 L CNN
 F 2 "C1V7" V 1530 2600 60  0001 C CNN
@@
 $EndComp
 $Comp
-L GND #PWR?
-U 1 1 486CA86E
+L GND #PWR045
+U 1 1 4C2F529B
 P 2600 3750
-F 0 "#PWR?" H 2600 3750 30  0001 C CNN
+F 0 "#PWR045" H 2600 3750 30  0001 C CNN
 F 1 "GND" H 2600 3680 30  0001 C CNN
 	1    2600 3750
