File: design/power_reg1.sch (KiCad schematic (older format))
At the start: 10 parts, among them U4 LM2940

Commit message: Im  decided about the components, no further changes will be made in that subject. Power regulators were moved, one supplies the cpu, the other everything else. MAX9926 is from now on the magnetic reluctor driver
Parts:
- U4: value LM2940 -> LM2937
Changed lines of the file:
@@
-EESchema Schematic File Version 2  date Sat 04 Sep 2010 04:23:02 PM ART
+EESchema Schematic File Version 2  date Tue 05 Oct 2010 05:44:15 PM ART
 LIBS:power
 LIBS:freeEMS_lib
@@
 EELAYER END
 $Descr A 11000 8500
-Sheet 17 46
+Sheet 20 46
 Title "freeEMS 1.0"
-Date "4 sep 2010"
+Date "5 oct 2010"
 Rev "A.07"
 Comp "diyefi.org"
@@
 P 5800 3350
 F 0 "U4" H 5950 3154 60  0000 C CNN
-F 1 "LM2940" H 5800 3550 60  0000 C CNN
+F 1 "LM2937" H 5800 3550 60  0000 C CNN
 F 2 "TO220_sm" V 2630 2600 60  0001 C CNN
 F 4 "newark,45J1442" V 2630 2600 60  0001 C CNN "Field1"

Commit message: Updated specs notes
Parts:
- removed C7: 2200uF, C1V7, symbol C
- C10: value 2200uF -> 22uF
- C11: value 10uF -> 2200uF
Other:
- note added: "*C10: aluminum\n*C11: tantalum, close to the regulator"
Changed lines of the file:
@@
-EESchema Schematic File Version 2  date Tue 05 Oct 2010 05:44:15 PM ART
+EESchema Schematic File Version 2  date Fri 15 Oct 2010 07:57:43 PM ART
 LIBS:power
 LIBS:freeEMS_lib
@@
 EELAYER END
 $Descr A 11000 8500
-Sheet 20 46
+Sheet 22 44
 Title "freeEMS 1.0"
-Date "5 oct 2010"
+Date "15 oct 2010"
 Rev "A.07"
 Comp "diyefi.org"
@@
 Comment4 ""
 $EndDescr
+Text Notes 6350 4050 0    60   ~ 0
+*C10: aluminum\n*C11: tantalum, close to the regulator
+$Comp
+L C C12
+U 1 1 4C2F52A3
+P 7450 3500
+F 0 "C12" H 7500 3600 50  0000 L CNN
+F 1 ".1uF" H 7500 3400 50  0000 L CNN
+F 2 "C1V7" V 5930 2600 60  0001 C CNN
+F 4 "newark,56K3664" V 5930 2600 60  0001 C CNN "Field1"
+F 5 "vendor1, smd w hem" V 5930 2600 60  0001 C CNN "Field2"
+F 6 "vendor2, thru w hem" V 5930 2600 60  0001 C CNN "Field3"
+F 7 "vendor2, smd w hem" V 5930 2600 60  0001 C CNN "Field4"
+F 8 "50,V" V 5930 2600 60  0001 C CNN "Field5"
+F 9 "20,%" V 5930 2600 60  0001 C CNN "Field6"
+F 10 "multilayer ceramic" V 5930 2600 60  0001 C CNN "Field7"
+F 11 "other,more,stuff" V 5930 2600 60  0001 C CNN "Field8"
+	1    7450 3500
+	-1   0    0    -1
+$EndComp
+Connection ~ 7450 3700
+Connection ~ 7450 3300
+Wire Wire Line
+	3600 3300 5400 3300
 Connection ~ 3350 3700
 Connection ~ 5350 3300
@@
 Connection ~ 6550 3300
 Wire Wire Line
-	5400 3300 3600 3300
-Wire Wire Line
 	7850 3700 2600 3700
 Connection ~ 5250 3300
-Connection ~ 4400 3700
 Connection ~ 5250 3700
-Connection ~ 4400 3300
-Connection ~ 7450 3700
 Wire Wire Line
 	7850 3300 6200 3300
-Connection ~ 7450 3300
 Connection ~ 7000 3300
 Wire Wire Line
@@
 Connection ~ 6250 3300
 $Comp
-L PWR_FLAG #FLG050
+L PWR_FLAG #FLG056
 U 1 1 4C66D6BC
 P 3350 3700
-F 0 "#FLG050" H 3350 3970 30  0001 C CNN
+F 0 "#FLG056" H 3350 3970 30  0001 C CNN
 F 1 "PWR_FLAG" H 3350 3930 30  0000 C CNN
 	1    3350 3700
@@
 $EndComp
 $Comp
-L PWR_FLAG #FLG051
+L PWR_FLAG #FLG057
 U 1 1 4C2F5631
 P 4850 3300
-F 0 "#FLG051" H 4850 3570 30  0001 C CNN
+F 0 "#FLG057" H 4850 3570 30  0001 C CNN
 F 1 "PWR_FLAG" H 4850 3530 30  0000 C CNN
 	1    4850 3300
@@
 $EndComp
 $Comp
-L C C7
-U 1 1 4C2F52EB
-P 4400 3500
-F 0 "C7" H 4450 3600 50  0000 L CNN
-F 1 "2200uF" H 4450 3400 50  0000 L CNN
-F 2 "C1V7" V -170 2600 60  0001 C CNN
-F 4 "newark,69K8230" V -170 2600 60  0001 C CNN "Field1"
-F 5 "vendor1, smd w hem" V -170 2600 60  0001 C CNN "Field2"
-F 6 "vendor2, thru w hem" V -170 2600 60  0001 C CNN "Field3"
-F 7 "vendor2, smd w hem" V -170 2600 60  0001 C CNN "Field4"
-F 8 "50,V" V -170 2600 60  0001 C CNN "Field5"
-F 9 "X,%" V -170 2600 60  0001 C CNN "Field6"
-F 10 "Aluminum Electrolytic" V -170 2600 60  0001 C CNN "Field7"
-F 11 "other,more,stuff" V -170 2600 60  0001 C CNN "Field8"
-	1    4400 3500
-	-1   0    0    -1
-$EndComp
-$Comp
 L C C10
 U 1 1 4C2F52EA
 P 6550 3500
 F 0 "C10" H 6600 3600 50  0000 L CNN
-F 1 "2200uF" H 6600 3400 50  0000 L CNN
+F 1 "22uF" H 6600 3400 50  0000 L CNN
 F 2 "C1V7" V 4130 2600 60  0001 C CNN
 F 4 "newark,69K8230" V 4130 2600 60  0001 C CNN "Field1"
@@
 gnd
 $Comp
-L C C12
-U 1 1 4C2F52A3
-P 7450 3500
-F 0 "C12" H 7500 3600 50  0000 L CNN
-F 1 ".1uF" H 7500 3400 50  0000 L CNN
-F 2 "C1V7" V 5930 2600 60  0001 C CNN
-F 4 "newark,56K3664" V 5930 2600 60  0001 C CNN "Field1"
-F 5 "vendor1, smd w hem" V 5930 2600 60  0001 C CNN "Field2"
-F 6 "vendor2, thru w hem" V 5930 2600 60  0001 C CNN "Field3"
-F 7 "vendor2, smd w hem" V 5930 2600 60  0001 C CNN "Field4"
-F 8 "50,V" V 5930 2600 60  0001 C CNN "Field5"
-F 9 "20,%" V 5930 2600 60  0001 C CNN "Field6"
-F 10 "multilayer ceramic" V 5930 2600 60  0001 C CNN "Field7"
-F 11 "other,more,stuff" V 5930 2600 60  0001 C CNN "Field8"
-	1    7450 3500
-	-1   0    0    -1
-$EndComp
-$Comp
 L DIODE D3
 U 1 1 4C2F52A2
@@
 $EndComp
 $Comp
-L VSS #PWR052
+L VSS #PWR058
 U 1 1 486CA95E
 P 7850 3750
-F 0 "#PWR052" H 7850 3750 30  0001 C CNN
+F 0 "#PWR058" H 7850 3750 30  0001 C CNN
 F 1 "VSS" H 7850 3680 30  0000 C CNN
 	1    7850 3750
@@
 P 7000 3500
 F 0 "C11" H 7050 3600 50  0000 L CNN
-F 1 "10uF" H 7050 3400 50  0000 L CNN
+F 1 "2200uF" H 7050 3400 50  0000 L CNN
 F 2 "C1V7" V 5030 2600 60  0001 C CNN
 F 4 "newark,97M4217" V 5030 2600 60  0001 C CNN "Field1"
@@
 $EndComp
 $Comp
-L GND #PWR053
+L GND #PWR059
 U 1 1 4C2F529B
 P 2600 3750
-F 0 "#PWR053" H 2600 3750 30  0001 C CNN
+F 0 "#PWR059" H 2600 3750 30  0001 C CNN
 F 1 "GND" H 2600 3680 30  0001 C CNN
 	1    2600 3750

Commit message: Added signal connector in a proper way, modified analog ground plane, still not convinced about it. board almost routed
Parts:
- added Q18: NPN, symbol NPN
- added Q19: PNP, symbol PNP
- added R226: 22k, symbol R
- added R227: 10k, symbol R
Connections:
- net labels added: ENABLE
- wire segments 12 -> 18
Changed lines of the file:
@@
-EESchema Schematic File Version 2  date Sun 24 Oct 2010 05:17:02 PM ART
+EESchema Schematic File Version 2  date Fri 29 Oct 2010 12:01:49 PM ART
 LIBS:power
 LIBS:freeEMS_lib
@@
 Sheet 22 44
 Title "freeEMS 1.0"
-Date "24 oct 2010"
+Date "29 oct 2010"
 Rev "A.07"
 Comp "diyefi.org"
@@
 Comment4 ""
 $EndDescr
+Wire Wire Line
+	2950 4600 2500 4600
+Wire Wire Line
+	4200 3800 4200 3600
+Wire Wire Line
+	4000 3300 3600 3300
+Connection ~ 7450 3700
+Connection ~ 7450 3300
+Connection ~ 3350 3700
+Connection ~ 5350 3300
+Wire Wire Line
+	5350 3300 5350 2900
+Wire Wire Line
+	5350 2900 5600 2900
+Connection ~ 6550 3700
+Connection ~ 6550 3300
+Wire Wire Line
+	7850 3700 2600 3700
+Connection ~ 5250 3300
+Connection ~ 5250 3700
+Wire Wire Line
+	7850 3300 6200 3300
+Connection ~ 7000 3300
+Wire Wire Line
+	7850 3700 7850 3750
+Wire Wire Line
+	5800 3700 5800 3600
+Connection ~ 7000 3700
+Wire Wire Line
+	2600 3700 2600 3750
+Wire Wire Line
+	3050 3300 3100 3300
+Connection ~ 4850 3700
+Connection ~ 5800 3700
+Wire Wire Line
+	2500 3300 2650 3300
+Wire Wire Line
+	6000 2900 6250 2900
+Wire Wire Line
+	6250 2900 6250 3300
+Connection ~ 6250 3300
+Wire Wire Line
+	5400 3300 4400 3300
+Connection ~ 4850 3300
+Wire Wire Line
+	4200 4950 4200 4800
+Wire Wire Line
+	4200 4300 4200 4400
+Wire Wire Line
+	3450 4600 3900 4600
+$Comp
+L R R226
+U 1 1 4CC4C2A7
+P 3200 4600
+F 0 "R226" V 3280 4600 50  0000 C CNN
+F 1 "22k" V 3200 4600 50  0000 C CNN
+	1    3200 4600
+	0    1    1    0
+$EndComp
+Text HLabel 2500 4600 0    60   Input ~ 0
+ENABLE
+$Comp
+L R R227
+U 1 1 4CC4C257
+P 4200 4050
+F 0 "R227" V 4280 4050 50  0000 C CNN
+F 1 "10k" V 4200 4050 50  0000 C CNN
+	1    4200 4050
+	1    0    0    -1
+$EndComp
+$Comp
+L GND #PWR057
+U 1 1 4CC4C238
+P 4200 4950
+F 0 "#PWR057" H 4200 4950 30  0001 C CNN
+F 1 "GND" H 4200 4880 30  0001 C CNN
+	1    4200 4950
+	1    0    0    -1
+$EndComp
+$Comp
+L NPN Q18
+U 1 1 4CC4C212
+P 4100 4600
+F 0 "Q18" H 4100 4450 50  0000 R CNN
+F 1 "NPN" H 4100 4750 50  0000 R CNN
+	1    4100 4600
+	1    0    0    -1
+$EndComp
+$Comp
+L PNP Q19
+U 1 1 4CC4C0CD
+P 4200 3400
+F 0 "Q19" H 4200 3250 60  0000 R CNN
+F 1 "PNP" H 4200 3550 60  0000 R CNN
+	1    4200 3400
+	0    1    -1   0
+$EndComp
 Text Notes 6350 4050 0    60   ~ 0
 *C10: aluminum\n*C11: tantalum, close to the regulator
@@
 	-1   0    0    -1
 $EndComp
-Connection ~ 7450 3700
-Connection ~ 7450 3300
-Wire Wire Line
-	3600 3300 5400 3300
-Connection ~ 3350 3700
-Connection ~ 5350 3300
-Wire Wire Line
-	5350 3300 5350 2900
-Wire Wire Line
-	5350 2900 5600 2900
-Connection ~ 6550 3700
-Connection ~ 6550 3300
-Wire Wire Line
-	7850 3700 2600 3700
-Connection ~ 5250 3300
-Connection ~ 5250 3700
-Wire Wire Line
-	7850 3300 6200 3300
-Connection ~ 7000 3300
-Wire Wire Line
-	7850 3700 7850 3750
-Wire Wire Line
-	5800 3700 5800 3600
-Connection ~ 7000 3700
-Wire Wire Line
-	2600 3700 2600 3750
-Wire Wire Line
-	3050 3300 3100 3300
-Connection ~ 4850 3300
-Connection ~ 4850 3700
-Connection ~ 5800 3700
-Wire Wire Line
-	2500 3300 2650 3300
-Wire Wire Line
-	6000 2900 6250 2900
-Wire Wire Line
-	6250 2900 6250 3300
-Connection ~ 6250 3300
-$Comp
-L PWR_FLAG #FLG056
+$Comp
+L PWR_FLAG #FLG058
 U 1 1 4C66D6BC
 P 3350 3700
-F 0 "#FLG056" H 3350 3970 30  0001 C CNN
+F 0 "#FLG058" H 3350 3970 30  0001 C CNN
 F 1 "PWR_FLAG" H 3350 3930 30  0000 C CNN
 	1    3350 3700
@@
 $EndComp
 $Comp
-L PWR_FLAG #FLG057
+L PWR_FLAG #FLG059
 U 1 1 4C2F5631
 P 4850 3300
-F 0 "#FLG057" H 4850 3570 30  0001 C CNN
+F 0 "#FLG059" H 4850 3570 30  0001 C CNN
 F 1 "PWR_FLAG" H 4850 3530 30  0000 C CNN
 	1    4850 3300
@@
 $EndComp
 $Comp
-L VSS #PWR058
+L VSS #PWR060
 U 1 1 486CA95E
 P 7850 3750
-F 0 "#PWR058" H 7850 3750 30  0001 C CNN
+F 0 "#PWR060" H 7850 3750 30  0001 C CNN
 F 1 "VSS" H 7850 3680 30  0000 C CNN
 	1    7850 3750
@@
 $EndComp
 $Comp
-L GND #PWR059
+L GND #PWR061
 U 1 1 4C2F529B
 P 2600 3750
-F 0 "#PWR059" H 2600 3750 30  0001 C CNN
+F 0 "#PWR061" H 2600 3750 30  0001 C CNN
 F 1 "GND" H 2600 3680 30  0001 C CNN
 	1    2600 3750

Commit message: Routing complete
Changed lines of the file:
@@
-EESchema Schematic File Version 2  date Sat 30 Oct 2010 04:18:53 PM ART
+EESchema Schematic File Version 2  date Sun 07 Nov 2010 11:30:10 PM ART
 LIBS:power
 LIBS:freeEMS_lib
@@
 EELAYER END
 $Descr A 11000 8500
-Sheet 22 44
+Sheet 22 50
 Title "freeEMS 1.0"
-Date "30 oct 2010"
+Date "8 nov 2010"
 Rev "A.07"
 Comp "diyefi.org"
@@
 Comment4 ""
 $EndDescr
+Connection ~ 6250 3300
+Wire Wire Line
+	6200 3300 7850 3300
+Wire Wire Line
+	3450 4600 3900 4600
+Wire Wire Line
+	4200 4300 4200 4400
+Wire Wire Line
+	4200 4950 4200 4800
+Connection ~ 4850 3300
+Wire Wire Line
+	5400 3300 4400 3300
+Wire Wire Line
+	6250 3300 6250 2900
+Wire Wire Line
+	6250 2900 6000 2900
+Wire Wire Line
+	2500 3300 2650 3300
+Connection ~ 5800 3700
+Connection ~ 4850 3700
+Wire Wire Line
+	3050 3300 3100 3300
+Wire Wire Line
+	2600 3750 2600 3700
+Connection ~ 7000 3700
+Wire Wire Line
+	5800 3700 5800 3600
+Wire Wire Line
+	7850 3750 7850 3700
+Connection ~ 7000 3300
+Connection ~ 5250 3700
+Connection ~ 5250 3300
+Wire Wire Line
+	7850 3700 2600 3700
+Connection ~ 6550 3300
+Connection ~ 6550 3700
+Wire Wire Line
+	5600 2900 5350 2900
+Wire Wire Line
+	5350 2900 5350 3300
+Connection ~ 5350 3300
+Connection ~ 7450 3300
+Connection ~ 7450 3700
+Wire Wire Line
+	4000 3300 3600 3300
+Wire Wire Line
+	4200 3800 4200 3600
 Wire Wire Line
 	2950 4600 2500 4600
-Wire Wire Line
-	4200 3800 4200 3600
-Wire Wire Line
-	4000 3300 3600 3300
-Connection ~ 7450 3700
-Connection ~ 7450 3300
-Connection ~ 3350 3700
-Connection ~ 5350 3300
-Wire Wire Line
-	5350 3300 5350 2900
-Wire Wire Line
-	5350 2900 5600 2900
-Connection ~ 6550 3700
-Connection ~ 6550 3300
-Wire Wire Line
-	7850 3700 2600 3700
-Connection ~ 5250 3300
-Connection ~ 5250 3700
-Wire Wire Line
-	7850 3300 6200 3300
-Connection ~ 7000 3300
-Wire Wire Line
-	7850 3700 7850 3750
-Wire Wire Line
-	5800 3700 5800 3600
-Connection ~ 7000 3700
-Wire Wire Line
-	2600 3700 2600 3750
-Wire Wire Line
-	3050 3300 3100 3300
-Connection ~ 4850 3700
-Connection ~ 5800 3700
-Wire Wire Line
-	2500 3300 2650 3300
-Wire Wire Line
-	6000 2900 6250 2900
-Wire Wire Line
-	6250 2900 6250 3300
-Connection ~ 6250 3300
-Wire Wire Line
-	5400 3300 4400 3300
-Connection ~ 4850 3300
-Wire Wire Line
-	4200 4950 4200 4800
-Wire Wire Line
-	4200 4300 4200 4400
-Wire Wire Line
-	3450 4600 3900 4600
 $Comp
 L R R226
@@
 $EndComp
 $Comp
-L GND #PWR057
+L GND #PWR13
 U 1 1 4CC4C238
 P 4200 4950
-F 0 "#PWR057" H 4200 4950 30  0001 C CNN
+F 0 "#PWR13" H 4200 4950 30  0001 C CNN
 F 1 "GND" H 4200 4880 30  0001 C CNN
 	1    4200 4950
@@
 	1    7450 3500
 	-1   0    0    -1
-$EndComp
-$Comp
-L PWR_FLAG #FLG058
-U 1 1 4C66D6BC
-P 3350 3700
-F 0 "#FLG058" H 3350 3970 30  0001 C CNN
-F 1 "PWR_FLAG" H 3350 3930 30  0000 C CNN
-	1    3350 3700
-	1    0    0    -1
-$EndComp
-$Comp
-L PWR_FLAG #FLG059
-U 1 1 4C2F5631
-P 4850 3300
-F 0 "#FLG059" H 4850 3570 30  0001 C CNN
-F 1 "PWR_FLAG" H 4850 3530 30  0000 C CNN
-	1    4850 3300
-	1    0    0    -1
 $EndComp
 $Comp
@@
 $EndComp
 $Comp
-L VSS #PWR060
+L VSS #PWR14
 U 1 1 486CA95E
 P 7850 3750
-F 0 "#PWR060" H 7850 3750 30  0001 C CNN
+F 0 "#PWR14" H 7850 3750 30  0001 C CNN
 F 1 "VSS" H 7850 3680 30  0000 C CNN
 	1    7850 3750
@@
 $EndComp
 $Comp
-L GND #PWR061
+L GND #PWR12
 U 1 1 4C2F529B
 P 2600 3750
-F 0 "#PWR061" H 2600 3750 30  0001 C CNN
+F 0 "#PWR12" H 2600 3750 30  0001 C CNN
 F 1 "GND" H 2600 3680 30  0001 C CNN
 	1    2600 3750
