File: design/digi_protect_I2.sch (KiCad schematic (older format))
At the start: 4 parts

Commit message: Everything routed except the undefined output pins.
Connections:
- net GND renamed digi_gnd
Changed lines of the file:
@@
-EESchema Schematic File Version 2  date Sun 29 Aug 2010 06:27:37 AM ART
+EESchema Schematic File Version 2  date Sun 29 Aug 2010 11:22:28 PM ART
 LIBS:power
 LIBS:freeEMS_lib
@@
 EELAYER END
 $Descr A4 11700 8267
-Sheet 11 50
+Sheet 21 50
 Title "freeEMS 1.0"
-Date "29 aug 2010"
+Date "30 aug 2010"
 Rev "A.08"
 Comp "diyefi.org"
@@
 Wire Wire Line
 	3850 1750 2650 1750
-Wire Wire Line
-	2800 2250 2800 2150
 Wire Wire Line
 	4350 1750 4550 1750
@@
 	1    0    0    -1
 $EndComp
-$Comp
-L GND #PWR053
-U 1 1 4C2F52AE
-P 2800 2250
-F 0 "#PWR053" H 2800 2250 30  0001 C CNN
-F 1 "GND" H 2800 2180 30  0001 C CNN
-	1    2800 2250
-	1    0    0    -1
-$EndComp
