File: design/digi_protect_fuel.sch (KiCad schematic (older format))
At the start: 4 parts

Commit message: Updated specs notes
Parts:
- removed C27: 100nF, C1V7, symbol C
- R43, R44: value 10k -> 1k
Changed lines of the file:
@@
-EESchema Schematic File Version 2  date Tue 05 Oct 2010 05:44:15 PM ART
+EESchema Schematic File Version 2  date Tue 12 Oct 2010 12:24:50 AM ART
 LIBS:power
 LIBS:freeEMS_lib
@@
 EELAYER END
 $Descr A4 11700 8267
-Sheet 36 46
+Sheet 35 47
 Title "freeEMS 1.0"
-Date "5 oct 2010"
+Date "12 oct 2010"
 Rev "A.08"
 Comp "diyefi.org"
@@
 $EndDescr
 Connection ~ 2800 1750
-Connection ~ 2800 2150
 Wire Wire Line
-	3250 2150 1950 2150
+	2800 2150 1950 2150
 Wire Wire Line
 	2150 1750 1950 1750
-Connection ~ 3250 1750
 Wire Wire Line
 	3850 1750 2650 1750
@@
 P 4100 1750
 F 0 "R44" V 4180 1750 50  0000 C CNN
-F 1 "10k" V 4100 1750 50  0000 C CNN
+F 1 "1k" V 4100 1750 50  0000 C CNN
 F 2 "R4-SM0805" V 4280 1850 60  0001 C CNN
 F 4 "newark,38K0328" V 1130 2600 60  0001 C CNN "Field1"
@@
 P 2400 1750
 F 0 "R43" V 2480 1750 50  0000 C CNN
-F 1 "10k" V 2400 1750 50  0000 C CNN
+F 1 "1k" V 2400 1750 50  0000 C CNN
 F 2 "R4-SM0805" V 2580 1850 60  0001 C CNN
 F 4 "newark,38K0328" V 1130 2600 60  0001 C CNN "Field1"
@@
 	0    1    1    0
 $EndComp
-$Comp
-L C C27
-U 1 1 4C2F52B7
-P 3250 1950
-F 0 "C27" H 3300 2050 50  0000 L CNN
-F 1 "100nF" H 3300 1850 50  0000 L CNN
-F 2 "C1V7" V 1130 2600 60  0001 C CNN
-F 4 "newark,39K8137" V 1130 2600 60  0001 C CNN "Field1"
-F 5 "vendor1, smd w hem" V 1130 2600 60  0001 C CNN "Field2"
-F 6 "vendor2, thru w hem" V 1130 2600 60  0001 C CNN "Field3"
-F 7 "vendor2, smd w hem" V 1130 2600 60  0001 C CNN "Field4"
-F 8 "50,V" V 1130 2600 60  0001 C CNN "Field5"
-F 9 "10,%" V 1130 2600 60  0001 C CNN "Field6"
-F 10 "Multilayer Ceramic" V 1130 2600 60  0001 C CNN "Field7"
-F 11 "other,more,stuff" V 1130 2600 60  0001 C CNN "Field8"
-	1    3250 1950
-	1    0    0    -1
-$EndComp
 Text HLabel 1950 2150 0    60   BiDi ~ 0

Commit message: Includes a script to update all components information, and a more verbose BOM
Parts:
- D28: Field1 newark,18M3285 -> (none); Field2 vendor1, smd w hem -> (none); Field3 vendor2, thru w hem -> (none); Field4 vendor2, smd w hem -> (none); Field5 500,mW -> (none); Field6 20,mA -> (none); Field7 X -> (none); Field8 other,more,stuff -> (none); construct (none) -> zener; current (none) -> .01; mfg (none) -> Diodes Inc; mfg# (none) -> BZT52C5V1-7-F; misc (none) -> other,more,stuff; vend1 (none) -> digikey; vend1# (none) -> BZT52C5V1-FDICT-ND; voltage (none) -> 5.1v
- R43, R44: Field1 newark,38K0328 -> (none); Field2 vendor1, smd w hem -> (none); Field3 vendor2, thru w hem -> (none); Field4 vendor2, smd w hem -> (none); Field5 250,mW -> (none); Field6 5,% -> (none); Field7 Carbon Film -> (none); Field8 other,more,stuff -> (none); Power (none) -> .125w; construct (none) -> Thick Film; mfg (none) -> Stackpole; mfg# (none) -> RMCF0805JT1K00; misc (none) -> other,more,stuff; tolerance (none) -> 5%; vend1 (none) -> digikey; vend1# (none) -> RMCF0805JT1K00TR-ND
Changed lines of the file:
@@
 F 1 "1k" V 4100 1750 50  0000 C CNN
 F 2 "R4-SM0805" V 4280 1850 60  0001 C CNN
-F 4 "newark,38K0328" V 1130 2600 60  0001 C CNN "Field1"
-F 5 "vendor1, smd w hem" V 1130 2600 60  0001 C CNN "Field2"
-F 6 "vendor2, thru w hem" V 1130 2600 60  0001 C CNN "Field3"
-F 7 "vendor2, smd w hem" V 1130 2600 60  0001 C CNN "Field4"
-F 8 "250,mW" V 1130 2600 60  0001 C CNN "Field5"
-F 9 "5,%" V 1130 2600 60  0001 C CNN "Field6"
-F 10 "Carbon Film" V 1130 2600 60  0001 C CNN "Field7"
-F 11 "other,more,stuff" V 1130 2600 60  0001 C CNN "Field8"
+F 4 "Stackpole" V 1130 2600 60  0001 C CNN "mfg"
+F 5 "RMCF0805JT1K00" V 1130 2600 60  0001 C CNN "mfg#"
+F 6 "digikey" V 1130 2600 60  0001 C CNN "vend1"
+F 7 "RMCF0805JT1K00TR-ND" V 1130 2600 60  0001 C CNN "vend1#"
+F 8 ".125w" V 1130 2600 60  0001 C CNN "Power"
+F 9 "5%" V 1130 2600 60  0001 C CNN "tolerance"
+F 10 "Thick Film" V 1130 2600 60  0001 C CNN "construct"
+F 11 "other,more,stuff" V 1130 2600 60  0001 C CNN "misc"
 	1    4100 1750
 	0    1    1    0
@@
 F 1 "5V1" H 2800 1850 40  0000 C CNN
 F 2 "D4-SMB" V 1130 2600 60  0001 C CNN
-F 4 "newark,18M3285" V 1130 2600 60  0001 C CNN "Field1"
-F 5 "vendor1, smd w hem" V 1130 2600 60  0001 C CNN "Field2"
-F 6 "vendor2, thru w hem" V 1130 2600 60  0001 C CNN "Field3"
-F 7 "vendor2, smd w hem" V 1130 2600 60  0001 C CNN "Field4"
-F 8 "500,mW" V 1130 2600 60  0001 C CNN "Field5"
-F 9 "20,mA" V 1130 2600 60  0001 C CNN "Field6"
-F 10 "X" V 1130 2600 60  0001 C CNN "Field7"
-F 11 "other,more,stuff" V 1130 2600 60  0001 C CNN "Field8"
+F 4 "Diodes Inc" V 1130 2600 60  0001 C CNN "mfg"
+F 5 "BZT52C5V1-7-F" V 1130 2600 60  0001 C CNN "mfg#"
+F 6 "digikey" V 1130 2600 60  0001 C CNN "vend1"
+F 7 "BZT52C5V1-FDICT-ND" V 1130 2600 60  0001 C CNN "vend1#"
+F 8 ".01" V 1130 2600 60  0001 C CNN "current"
+F 9 "5.1v" V 1130 2600 60  0001 C CNN "voltage"
+F 10 "zener" V 1130 2600 60  0001 C CNN "construct"
+F 11 "other,more,stuff" V 1130 2600 60  0001 C CNN "misc"
 	1    2800 1950
 	0    -1   -1   0
@@
 F 1 "1k" V 2400 1750 50  0000 C CNN
 F 2 "R4-SM0805" V 2580 1850 60  0001 C CNN
-F 4 "newark,38K0328" V 1130 2600 60  0001 C CNN "Field1"
-F 5 "vendor1, smd w hem" V 1130 2600 60  0001 C CNN "Field2"
-F 6 "vendor2, thru w hem" V 1130 2600 60  0001 C CNN "Field3"
-F 7 "vendor2, smd w hem" V 1130 2600 60  0001 C CNN "Field4"
-F 8 "250,mW" V 1130 2600 60  0001 C CNN "Field5"
-F 9 "5,%" V 1130 2600 60  0001 C CNN "Field6"
-F 10 "Carbon Film" V 1130 2600 60  0001 C CNN "Field7"
-F 11 "other,more,stuff" V 1130 2600 60  0001 C CNN "Field8"
+F 4 "Stackpole" V 1130 2600 60  0001 C CNN "mfg"
+F 5 "RMCF0805JT1K00" V 1130 2600 60  0001 C CNN "mfg#"
+F 6 "digikey" V 1130 2600 60  0001 C CNN "vend1"
+F 7 "RMCF0805JT1K00TR-ND" V 1130 2600 60  0001 C CNN "vend1#"
+F 8 ".125w" V 1130 2600 60  0001 C CNN "Power"
+F 9 "5%" V 1130 2600 60  0001 C CNN "tolerance"
+F 10 "Thick Film" V 1130 2600 60  0001 C CNN "construct"
+F 11 "other,more,stuff" V 1130 2600 60  0001 C CNN "misc"
 	1    2400 1750
 	0    1    1    0

Commit message: Schematic BOM is now fully populated with only 3 exceptions, .cmp file is obsolete at this point, so it has been removed.
Signed-off-by: Jared Harvey <TortiseGIT@jaredharvey.com>
Parts:
- R43, R44: footprint R4-SM0805 -> SM0805
Changed lines of the file:
@@
 F 0 "R44" V 4180 1750 50  0000 C CNN
 F 1 "1k" V 4100 1750 50  0000 C CNN
-F 2 "R4-SM0805" V 4280 1850 60  0001 C CNN
+F 2 "SM0805" V 1130 2600 60  0001 C CNN
 F 4 "Stackpole" V 1130 2600 60  0001 C CNN "mfg"
 F 5 "RMCF0805JT1K00" V 1130 2600 60  0001 C CNN "mfg#"
@@
 F 0 "R43" V 2480 1750 50  0000 C CNN
 F 1 "1k" V 2400 1750 50  0000 C CNN
-F 2 "R4-SM0805" V 2580 1850 60  0001 C CNN
+F 2 "SM0805" V 1130 2600 60  0001 C CNN
 F 4 "Stackpole" V 1130 2600 60  0001 C CNN "mfg"
 F 5 "RMCF0805JT1K00" V 1130 2600 60  0001 C CNN "mfg#"
