File: design/digi_protect_stepper4.sch (KiCad schematic (older format))
At the start: 3 parts

Commit message: Updated specs notes
Parts:
- removed D12: 5V1, D4-SMB, symbol ZENER
- removed R10, R9: 10k, R4-SM0805, symbol R
- added D96: 5V1, D4-SMB, symbol ZENER
- added R228, R229: 10k, R4-SM0805, symbol R
Connections:
- net digi_CPU: now also R228.2
- net digi_device: now also R229.1
- net digi_gnd: now also D96.1 (A)
- new net: D96.2 (K), R228.1, R229.2
Changed lines of the file:
@@
-EESchema Schematic File Version 2  date Fri 15 Oct 2010 07:57:43 PM ART
+EESchema Schematic File Version 2  date Mon 11 Oct 2010 11:06:53 PM ART
 LIBS:power
 LIBS:freeEMS_lib
@@
 EELAYER END
 $Descr A4 11700 8267
-Sheet 28 44
+Sheet 5 51
 Title "freeEMS 1.0"
-Date "15 oct 2010"
+Date "11 oct 2010"
 Rev "A.08"
 Comp "diyefi.org"
@@
 	4350 1750 4550 1750
 $Comp
-L R R10
-U 1 1 4C2F5304
+L R R229
+U 1 1 4C2F5303
 P 4100 1750
-F 0 "R10" V 4180 1750 50  0000 C CNN
+F 0 "R229" V 4180 1750 50  0000 C CNN
 F 1 "10k" V 4100 1750 50  0000 C CNN
 F 2 "R4-SM0805" V 4280 1850 60  0001 C CNN
@@
 $EndComp
 $Comp
-L ZENER D12
-U 1 1 4C2F52CE
+L ZENER D96
+U 1 1 4C2F52D0
 P 2800 1950
-F 0 "D12" H 2800 2050 50  0000 C CNN
+F 0 "D96" H 2800 2050 50  0000 C CNN
 F 1 "5V1" H 2800 1850 40  0000 C CNN
 F 2 "D4-SMB" V 1130 2600 60  0001 C CNN
@@
 $EndComp
 $Comp
-L R R9
-U 1 1 4C2F52C1
+L R R228
+U 1 1 4CB382B5
 P 2400 1750
-F 0 "R9" V 2480 1750 50  0000 C CNN
+F 0 "R228" V 2480 1750 50  0000 C CNN
 F 1 "10k" V 2400 1750 50  0000 C CNN
 F 2 "R4-SM0805" V 2580 1850 60  0001 C CNN

Commit message: Includes a script to update all components information, and a more verbose BOM
Parts:
- D96: Field1 newark,18M3285 -> (none); Field2 vendor1, smd w hem -> (none); Field3 vendor2, thru w hem -> (none); Field4 vendor2, smd w hem -> (none); Field5 500,mW -> (none); Field6 20,mA -> (none); Field7 X -> (none); Field8 other,more,stuff -> (none); construct (none) -> zener; current (none) -> .01; mfg (none) -> Diodes Inc; mfg# (none) -> BZT52C5V1-7-F; misc (none) -> other,more,stuff; vend1 (none) -> digikey; vend1# (none) -> BZT52C5V1-FDICT-ND; voltage (none) -> 5.1v
- R228, R229: Field1 newark,38K0328 -> (none); Field2 vendor1, smd w hem -> (none); Field3 vendor2, thru w hem -> (none); Field4 vendor2, smd w hem -> (none); Field5 250,mW -> (none); Field6 5,% -> (none); Field7 Carbon Film -> (none); Field8 other,more,stuff -> (none); construct (none) -> thick film; mfg (none) -> Stackpole; mfg# (none) -> RMCF0805JT10K0CT; misc (none) -> other,more,stuff; power (none) -> .125w; tol (none) -> 5%; vend1 (none) -> digikey; vend1# (none) -> RMCF0805JT10K0CT-ND
Changed lines of the file:
@@
 F 1 "10k" V 4100 1750 50  0000 C CNN
 F 2 "R4-SM0805" V 4280 1850 60  0001 C CNN
-F 4 "newark,38K0328" V 1130 2600 60  0001 C CNN "Field1"
-F 5 "vendor1, smd w hem" V 1130 2600 60  0001 C CNN "Field2"
-F 6 "vendor2, thru w hem" V 1130 2600 60  0001 C CNN "Field3"
-F 7 "vendor2, smd w hem" V 1130 2600 60  0001 C CNN "Field4"
-F 8 "250,mW" V 1130 2600 60  0001 C CNN "Field5"
-F 9 "5,%" V 1130 2600 60  0001 C CNN "Field6"
-F 10 "Carbon Film" V 1130 2600 60  0001 C CNN "Field7"
-F 11 "other,more,stuff" V 1130 2600 60  0001 C CNN "Field8"
+F 4 "Stackpole" V 1130 2600 60  0001 C CNN "mfg"
+F 5 "RMCF0805JT10K0CT" V 1130 2600 60  0001 C CNN "mfg#"
+F 6 "digikey" V 1130 2600 60  0001 C CNN "vend1"
+F 7 "RMCF0805JT10K0CT-ND" V 1130 2600 60  0001 C CNN "vend1#"
+F 8 ".125w" V 1130 2600 60  0001 C CNN "power"
+F 9 "5%" V 1130 2600 60  0001 C CNN "tol"
+F 10 "thick film" V 1130 2600 60  0001 C CNN "construct"
+F 11 "other,more,stuff" V 1130 2600 60  0001 C CNN "misc"
 	1    4100 1750
 	0    1    1    0
@@
 F 1 "5V1" H 2800 1850 40  0000 C CNN
 F 2 "D4-SMB" V 1130 2600 60  0001 C CNN
-F 4 "newark,18M3285" V 1130 2600 60  0001 C CNN "Field1"
-F 5 "vendor1, smd w hem" V 1130 2600 60  0001 C CNN "Field2"
-F 6 "vendor2, thru w hem" V 1130 2600 60  0001 C CNN "Field3"
-F 7 "vendor2, smd w hem" V 1130 2600 60  0001 C CNN "Field4"
-F 8 "500,mW" V 1130 2600 60  0001 C CNN "Field5"
-F 9 "20,mA" V 1130 2600 60  0001 C CNN "Field6"
-F 10 "X" V 1130 2600 60  0001 C CNN "Field7"
-F 11 "other,more,stuff" V 1130 2600 60  0001 C CNN "Field8"
+F 4 "Diodes Inc" V 1130 2600 60  0001 C CNN "mfg"
+F 5 "BZT52C5V1-7-F" V 1130 2600 60  0001 C CNN "mfg#"
+F 6 "digikey" V 1130 2600 60  0001 C CNN "vend1"
+F 7 "BZT52C5V1-FDICT-ND" V 1130 2600 60  0001 C CNN "vend1#"
+F 8 ".01" V 1130 2600 60  0001 C CNN "current"
+F 9 "5.1v" V 1130 2600 60  0001 C CNN "voltage"
+F 10 "zener" V 1130 2600 60  0001 C CNN "construct"
+F 11 "other,more,stuff" V 1130 2600 60  0001 C CNN "misc"
 	1    2800 1950
 	0    -1   -1   0
@@
 F 1 "10k" V 2400 1750 50  0000 C CNN
 F 2 "R4-SM0805" V 2580 1850 60  0001 C CNN
-F 4 "newark,38K0328" V 1130 2600 60  0001 C CNN "Field1"
-F 5 "vendor1, smd w hem" V 1130 2600 60  0001 C CNN "Field2"
-F 6 "vendor2, thru w hem" V 1130 2600 60  0001 C CNN "Field3"
-F 7 "vendor2, smd w hem" V 1130 2600 60  0001 C CNN "Field4"
-F 8 "250,mW" V 1130 2600 60  0001 C CNN "Field5"
-F 9 "5,%" V 1130 2600 60  0001 C CNN "Field6"
-F 10 "Carbon Film" V 1130 2600 60  0001 C CNN "Field7"
-F 11 "other,more,stuff" V 1130 2600 60  0001 C CNN "Field8"
+F 4 "Stackpole" V 1130 2600 60  0001 C CNN "mfg"
+F 5 "RMCF0805JT10K0CT" V 1130 2600 60  0001 C CNN "mfg#"
+F 6 "digikey" V 1130 2600 60  0001 C CNN "vend1"
+F 7 "RMCF0805JT10K0CT-ND" V 1130 2600 60  0001 C CNN "vend1#"
+F 8 ".125w" V 1130 2600 60  0001 C CNN "power"
+F 9 "5%" V 1130 2600 60  0001 C CNN "tol"
+F 10 "thick film" V 1130 2600 60  0001 C CNN "construct"
+F 11 "other,more,stuff" V 1130 2600 60  0001 C CNN "misc"
 	1    2400 1750
 	0    1    1    0

Commit message: Schematic BOM is now fully populated with only 3 exceptions, .cmp file is obsolete at this point, so it has been removed.
Signed-off-by: Jared Harvey <TortiseGIT@jaredharvey.com>
Parts:
- R228, R229: footprint R4-SM0805 -> SM0805
Changed lines of the file:
@@
 F 0 "R229" V 4180 1750 50  0000 C CNN
 F 1 "10k" V 4100 1750 50  0000 C CNN
-F 2 "R4-SM0805" V 4280 1850 60  0001 C CNN
+F 2 "SM0805" V 1130 2600 60  0001 C CNN
 F 4 "Stackpole" V 1130 2600 60  0001 C CNN "mfg"
 F 5 "RMCF0805JT10K0CT" V 1130 2600 60  0001 C CNN "mfg#"
@@
 F 0 "R228" V 2480 1750 50  0000 C CNN
 F 1 "10k" V 2400 1750 50  0000 C CNN
-F 2 "R4-SM0805" V 2580 1850 60  0001 C CNN
+F 2 "SM0805" V 1130 2600 60  0001 C CNN
 F 4 "Stackpole" V 1130 2600 60  0001 C CNN "mfg"
 F 5 "RMCF0805JT10K0CT" V 1130 2600 60  0001 C CNN "mfg#"
