File: design/digi_protect_rpm1.sch (KiCad schematic (older format))
At the start: 3 parts

Commit message: updating bom, lets commit this before I run a script to update the footprints for the resistors
Signed-off-by: Jared Harvey <TortiseGIT@jaredharvey.com>
Parts:
- D24: footprint D4-SMB -> SOD-123
Changed lines of the file:
@@
-EESchema Schematic File Version 2  date 2/14/2011 7:45:19 AM
+EESchema Schematic File Version 2  date 2/16/2011 5:39:17 AM
 LIBS:power
 LIBS:freeEMS_lib
@@
 EELAYER END
 $Descr A4 11700 8267
-Sheet 45 55
+Sheet 45 56
 Title "Puma board"
-Date "14 feb 2011"
+Date "16 feb 2011"
 Rev "v0.02"
 Comp "diyefi.org"
@@
 F 0 "D24" H 2800 2050 50  0000 C CNN
 F 1 "5V1" H 2800 1850 40  0000 C CNN
-F 2 "D4-SMB" V 1130 2600 60  0001 C CNN
+F 2 "SOD-123" V 1130 2600 60  0001 C CNN
 F 4 "Diodes Inc" V 1130 2600 60  0001 C CNN "mfg"
 F 5 "BZT52C5V1-7-F" V 1130 2600 60  0001 C CNN "mfg#"

Commit message: Schematic BOM is now fully populated with only 3 exceptions, .cmp file is obsolete at this point, so it has been removed.
Signed-off-by: Jared Harvey <TortiseGIT@jaredharvey.com>
Parts:
- R39, R40: footprint R4-SM0805 -> SM0805
Changed lines of the file:
@@
-EESchema Schematic File Version 2  date 2/16/2011 5:39:17 AM
+EESchema Schematic File Version 2  date 2/16/2011 8:44:20 AM
 LIBS:power
 LIBS:freeEMS_lib
@@
 F 0 "R40" V 4180 1750 50  0000 C CNN
 F 1 "1k" V 4100 1750 50  0000 C CNN
-F 2 "R4-SM0805" V 4280 1850 60  0001 C CNN
+F 2 "SM0805" V 1130 2600 60  0001 C CNN
 F 4 "Stackpole" V 1130 2600 60  0001 C CNN "mfg"
 F 5 "RMCF0805JT1K00" V 1130 2600 60  0001 C CNN "mfg#"
@@
 F 0 "R39" V 2480 1750 50  0000 C CNN
 F 1 "1k" V 2400 1750 50  0000 C CNN
-F 2 "R4-SM0805" V 2580 1850 60  0001 C CNN
+F 2 "SM0805" V 1130 2600 60  0001 C CNN
 F 4 "Stackpole" V 1130 2600 60  0001 C CNN "mfg"
 F 5 "RMCF0805JT1K00" V 1130 2600 60  0001 C CNN "mfg#"
