File: design/puma.sch (KiCad schematic (older format))
At the start: 35 parts, among them P100 CONN_1, P103 CONN_1, P104 CONN_1, P105 CONN_1, P2 CONN_1, P3 CONN_1, P4 CONN_1, P5 CONN_1, P75 CONN_1, P76 CONN_1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

Commit message: puma.sch is back to what it was with the linear regulators. We'll make the smaller changes and deal with the regulator upgrade later.
Signed-off-by: Jared Harvey <TortiseGIT@jaredharvey.com>
Connections:
- net voltage regulator (switched)/12v batt sw is gone; now on net 12V bat: F3.2
- net voltage regulator (switched)/12v batt renamed voltage regulator (cpu)/12v batt
Other:
- moved on the sheet: F1, F3, P100, P2, P3, P4, P5

Commit message: updating bom, lets commit this before I run a script to update the footprints for the resistors
Signed-off-by: Jared Harvey <TortiseGIT@jaredharvey.com>
Parts:
- F1: Field1 newark,63K6823 -> (none); Field2 WK6242-ND -> (none); Field3 vendor2, thru w hem -> (none); Field4 vendor2, smd w hem -> (none); Field5 x,x -> (none); Field6 10,A -> (none); Field7 construct -> 2,A; Field8 other,more,stuff -> -; mfg (none) -> little fuse; mfg# (none) -> 52000001009; vend1 (none) -> digikey; vend1# (none) -> WK6242-ND; vend2 (none) -> newark; vend2# (none) -> 63K6823
- F3: Field1 newark,63K6823 -> (none); Field2 WK6242-ND -> (none); Field3 vendor2, thru w hem -> (none); Field4 vendor2, smd w hem -> (none); Field5 x,x -> (none); Field6 10,A -> (none); Field7 construct -> 10,A; Field8 other,more,stuff -> -; mfg (none) -> little fuse; mfg# (none) -> 52000001009; vend1 (none) -> digikey; vend1# (none) -> WK6242-ND; vend2 (none) -> newark; vend2# (none) -> 63K6823
- P100, P75, P76, P77, P78, P79, P80, P81, P82, P83, P84, P85, P86, P87, P88, P89, P90: footprint (none) -> PINTST
- P2, P3, P4, P5: footprint 1PIN -> PINTST
- P99: footprint (none) -> PIN_ARRAY_20X2
Changed lines of the file:
@@
-EESchema Schematic File Version 2  date 1/19/2011 5:46:05 PM
+EESchema Schematic File Version 2  date 2/16/2011 5:39:13 AM
 LIBS:power
 LIBS:freeEMS_lib
@@
 Sheet 1 56
 Title "Puma board"
-Date "19 jan 2011"
+Date "16 feb 2011"
 Rev "v0.01"
 Comp "diyefi.org"
@@
 Comment4 ""
 $EndDescr
+Wire Wire Line
+	3700 1400 4600 1400
 Connection ~ 19000 5300
 Wire Wire Line
-	18000 5300 19000 5300
+	19000 5300 18000 5300
 Connection ~ 19000 4300
 Wire Wire Line
-	18000 4300 19000 4300
+	19000 4300 18000 4300
 Connection ~ 19000 3350
 Wire Wire Line
-	18000 3350 19000 3350
+	19000 3350 18000 3350
 Connection ~ 19000 2350
 Wire Wire Line
-	18000 2350 19000 2350
+	19000 2350 18000 2350
 Connection ~ 19000 1750
 Connection ~ 19000 1750
@@
 	6500 6950 6200 6950
 Wire Bus Line
-	12100 9650 12100 13200
+	12100 13200 12100 9650
 Wire Wire Line
 	6750 4650 7150 4650
@@
 Connection ~ 18850 11600
 Wire Wire Line
-	18000 11600 18850 11600
+	18850 11600 18000 11600
 Wire Wire Line
 	7300 8350 7400 8350
@@
 	10700 12500 10700 9850
 Connection ~ 8650 1400
-Connection ~ 4100 1400
 Connection ~ 10700 11050
 Wire Wire Line
@@
 	9150 3650 10100 3650
 Wire Bus Line
-	14250 1750 14250 10700
+	14250 10700 14250 1750
 Wire Wire Line
 	15050 2150 14350 2150
@@
 	14350 3150 15050 3150
 Wire Wire Line
-	18850 6050 18000 6050
+	18000 6050 18850 6050
 Connection ~ 18850 6500
 Wire Wire Line
@@
 	9150 3750 10100 3750
 Wire Wire Line
-	3700 1400 4150 1400
-Wire Wire Line
 	18150 1650 18150 5400
 Wire Wire Line
@@
 Connection ~ 14850 1750
 Wire Wire Line
-	7800 2850 5300 2850
+	5300 2850 7800 2850
 Connection ~ 7200 2850
 Wire Wire Line
@@
 	18000 4800 19000 4800
 Connection ~ 19000 4800
-Text Label 4250 1200 0    60   ~ 0
+$Comp
+L FUSE F3
+U 1 1 4D5B9F59
+P 6000 1200
+F 0 "F3" H 6100 1250 40  0000 C CNN
+F 1 "10A" H 5900 1150 40  0000 C CNN
+F 2 "FUSE5-20-DEFAULT-10A" V 5830 6000 60  0001 C CNN
+F 4 "little fuse" V 4580 3050 60  0001 C CNN "mfg"
+F 5 "52000001009" V 4580 3050 60  0001 C CNN "mfg#"
+F 6 "digikey" V 4580 3050 60  0001 C CNN "vend1"
+F 7 "WK6242-ND" V 4580 3050 60  0001 C CNN "vend1#"
+F 8 "newark" V 4580 3050 60  0001 C CNN "vend2"
+F 9 "63K6823" V 4580 3050 60  0001 C CNN "vend2#"
+F 10 "10,A" V 4580 3050 60  0001 C CNN "Field7"
+F 11 "-" V 4580 3050 60  0001 C CNN "Field8"
+	1    6000 1200
+	1    0    0    -1
+$EndComp
+Text Label 3750 1200 0    60   ~ 0
 bat_pwr
-Text Label 4250 1300 0    60   ~ 0
+Text Label 3750 1300 0    60   ~ 0
 bat_mcu
 $Comp
@@
 F 0 "P90" H 18680 1750 40  0000 L CNN
 F 1 "CONN_1" H 18600 1805 30  0001 C CNN
+F 2 "PINTST" H 18600 1750 60  0001 C CNN
 	1    18600 1750
 	1    0    0    -1
@@
 F 0 "P89" H 19230 1750 40  0000 L CNN
 F 1 "CONN_1" H 19150 1805 30  0001 C CNN
+F 2 "PINTST" H 19150 1750 60  0001 C CNN
 	1    19150 1750
 	1    0    0    -1
@@
 F 0 "P87" H 19230 2250 40  0000 L CNN
 F 1 "CONN_1" H 19150 2305 30  0001 C CNN
+F 2 "PINTST" H 19150 2250 60  0001 C CNN
 	1    19150 2250
 	1    0    0    -1
@@
 F 0 "P88" H 18680 2250 40  0000 L CNN
 F 1 "CONN_1" H 18600 2305 30  0001 C CNN
+F 2 "PINTST" H 18600 2250 60  0001 C CNN
 	1    18600 2250
 	1    0    0    -1
@@
 F 0 "P76" H 18680 2750 40  0000 L CNN
 F 1 "CONN_1" H 18600 2805 30  0001 C CNN
+F 2 "PINTST" H 18600 2750 60  0001 C CNN
 	1    18600 2750
 	1    0    0    -1
@@
 F 0 "P75" H 19230 2750 40  0000 L CNN
 F 1 "CONN_1" H 19150 2805 30  0001 C CNN
+F 2 "PINTST" H 19150 2750 60  0001 C CNN
 	1    19150 2750
 	1    0    0    -1
@@
 F 0 "P77" H 19230 3250 40  0000 L CNN
 F 1 "CONN_1" H 19150 3305 30  0001 C CNN
+F 2 "PINTST" H 19150 3250 60  0001 C CNN
 	1    19150 3250
 	1    0    0    -1
@@
 F 0 "P78" H 18680 3250 40  0000 L CNN
 F 1 "CONN_1" H 18600 3305 30  0001 C CNN
+F 2 "PINTST" H 18600 3250 60  0001 C CNN
 	1    18600 3250
 	1    0    0    -1
@@
 F 0 "P80" H 18680 3750 40  0000 L CNN
 F 1 "CONN_1" H 18600 3805 30  0001 C CNN
+F 2 "PINTST" H 18600 3750 60  0001 C CNN
 	1    18600 3750
 	1    0    0    -1
@@
 F 0 "P79" H 19230 3750 40  0000 L CNN
 F 1 "CONN_1" H 19150 3805 30  0001 C CNN
+F 2 "PINTST" H 19150 3750 60  0001 C CNN
 	1    19150 3750
 	1    0    0    -1
@@
 F 0 "P81" H 19230 4200 40  0000 L CNN
 F 1 "CONN_1" H 19150 4255 30  0001 C CNN
+F 2 "PINTST" H 19150 4200 60  0001 C CNN
 	1    19150 4200
 	1    0    0    -1
@@
 F 0 "P82" H 18680 4200 40  0000 L CNN
 F 1 "CONN_1" H 18600 4255 30  0001 C CNN
+F 2 "PINTST" H 18600 4200 60  0001 C CNN
 	1    18600 4200
 	1    0    0    -1
@@
 F 0 "P84" H 18680 4700 40  0000 L CNN
 F 1 "CONN_1" H 18600 4755 30  0001 C CNN
+F 2 "PINTST" H 18600 4700 60  0001 C CNN
 	1    18600 4700
 	1    0    0    -1
@@
 F 0 "P83" H 19230 4700 40  0000 L CNN
 F 1 "CONN_1" H 19150 4755 30  0001 C CNN
+F 2 "PINTST" H 19150 4700 60  0001 C CNN
 	1    19150 4700
 	1    0    0    -1
@@
 F 0 "P85" H 19230 5200 40  0000 L CNN
 F 1 "CONN_1" H 19150 5255 30  0001 C CNN
+F 2 "PINTST" H 19150 5200 60  0001 C CNN
 	1    19150 5200
 	1    0    0    -1
@@
 F 0 "P86" H 18680 5200 40  0000 L CNN
 F 1 "CONN_1" H 18600 5255 30  0001 C CNN
+F 2 "PINTST" H 18600 5200 60  0001 C CNN
 	1    18600 5200
 	1    0    0    -1
@@
 F 0 "P100" H 3630 1600 40  0000 L CNN
 F 1 "CONN_1" H 3550 1655 30  0001 C CNN
+F 2 "PINTST" H 3550 1600 60  0001 C CNN
 	1    3550 1600
 	-1   0    0    1
@@
 F 0 "P99" H 20950 8050 60  0000 C CNN
 F 1 "CONN_20X2" V 20950 7000 50  0000 C CNN
+F 2 "PIN_ARRAY_20X2" H 20950 7000 60  0001 C CNN
 	1    20950 7000
 	1    0    0    -1
@@
 L PWR_FLAG #FLG04
 U 1 1 4C8266A6
-P 4100 1400
-F 0 "#FLG04" H 4100 1670 30  0001 C CNN
-F 1 "PWR_FLAG" H 4100 1630 30  0000 C CNN
-	1    4100 1400
-	1    0    0    -1
+P 4600 1400
+F 0 "#FLG04" H 4600 1670 30  0001 C CNN
+F 1 "PWR_FLAG" H 4600 1630 30  0000 C CNN
+	1    4600 1400
+	0    1    1    0
 $EndComp
 $Comp
@@
 Text Label 18150 5400 0    60   ~ 0
 power_gnd
-Text Label 4150 1400 0    60   ~ 0
+Text Label 3750 1400 0    60   ~ 0
 power_gnd
 Text Label 9250 3650 0    60   ~ 0
@@
 F 0 "P5" H 3630 1500 40  0000 L CNN
 F 1 "CONN_1" H 3550 1555 30  0001 C CNN
-F 2 "1PIN" V 3730 3150 60  0001 C CNN
+F 2 "PINTST" V 3730 3150 60  0001 C CNN
 	1    3550 1500
 	-1   0    0    1
@@
 F 0 "P4" H 3630 1400 40  0000 L CNN
 F 1 "CONN_1" H 3550 1455 30  0001 C CNN
-F 2 "1PIN" V 3730 3150 60  0001 C CNN
+F 2 "PINTST" V 3730 3150 60  0001 C CNN
 	1    3550 1400
 	-1   0    0    1
@@
 F 0 "P3" H 3630 1300 40  0000 L CNN
 F 1 "CONN_1" H 3550 1355 30  0001 C CNN
-F 2 "1PIN" V 3730 3150 60  0001 C CNN
+F 2 "PINTST" V 3730 3150 60  0001 C CNN
 	1    3550 1300
 	-1   0    0    1
@@
 F 0 "P2" H 3630 1200 40  0000 L CNN
 F 1 "CONN_1" H 3550 1255 30  0001 C CNN
-F 2 "1PIN" V 3730 3150 60  0001 C CNN
+F 2 "PINTST" V 3730 3150 60  0001 C CNN
 	1    3550 1200
 	-1   0    0    1
-$EndComp
-$Comp
-L FUSE F3
-U 1 1 48A559CE
-P 6000 1200
-F 0 "F3" H 6100 1250 40  0000 C CNN
-F 1 "10A" H 5900 1150 40  0000 C CNN
-F 2 "FUSE5-20-DEFAULT-10A" V 4980 6100 60  0001 C CNN
-F 4 "newark,63K6823" V 3730 3150 60  0001 C CNN "Field1"
-F 5 "WK6242-ND" V 3730 3150 60  0001 C CNN "Field2"
-F 6 "vendor2, thru w hem" V 3730 3150 60  0001 C CNN "Field3"
-F 7 "vendor2, smd w hem" V 3730 3150 60  0001 C CNN "Field4"
-F 8 "x,x" V 3730 3150 60  0001 C CNN "Field5"
-F 9 "10,A" V 3730 3150 60  0001 C CNN "Field6"
-F 10 "construct" V 3730 3150 60  0001 C CNN "Field7"
-F 11 "other,more,stuff" V 3730 3150 60  0001 C CNN "Field8"
-	1    6000 1200
-	1    0    0    -1
 $EndComp
 $Comp
@@
 F 1 "2A" H 5050 1250 40  0000 C CNN
 F 2 "FUSE5-20-DEFAULT-2A" V 4980 6100 60  0001 C CNN
-F 4 "newark,63K6823" V 3730 3150 60  0001 C CNN "Field1"
-F 5 "WK6242-ND" V 3730 3150 60  0001 C CNN "Field2"
-F 6 "vendor2, thru w hem" V 3730 3150 60  0001 C CNN "Field3"
-F 7 "vendor2, smd w hem" V 3730 3150 60  0001 C CNN "Field4"
-F 8 "x,x" V 3730 3150 60  0001 C CNN "Field5"
-F 9 "10,A" V 3730 3150 60  0001 C CNN "Field6"
-F 10 "construct" V 3730 3150 60  0001 C CNN "Field7"
-F 11 "other,more,stuff" V 3730 3150 60  0001 C CNN "Field8"
+F 4 "little fuse" V 3730 3150 60  0001 C CNN "mfg"
+F 5 "52000001009" V 3730 3150 60  0001 C CNN "mfg#"
+F 6 "digikey" V 3730 3150 60  0001 C CNN "vend1"
+F 7 "WK6242-ND" V 3730 3150 60  0001 C CNN "vend1#"
+F 8 "newark" V 3730 3150 60  0001 C CNN "vend2"
+F 9 "63K6823" V 3730 3150 60  0001 C CNN "vend2#"
+F 10 "2,A" V 3730 3150 60  0001 C CNN "Field7"
+F 11 "-" V 3730 3150 60  0001 C CNN "Field8"
 	1    5150 1300
 	1    0    0    -1

Commit message: Schematic BOM is now fully populated with only 3 exceptions, .cmp file is obsolete at this point, so it has been removed.
Signed-off-by: Jared Harvey <TortiseGIT@jaredharvey.com>
Parts:
- R228, R229, R230, R231, R232, R233: footprint (none) -> SM0805
- U33: footprint (none) -> SO14E; Field2 74HC86DR2GOSCT-ND -> (none); mfg (none) -> on semi; mfg# (none) -> 74HC86DR2G; vend1 (none) -> digikey; vend1# (none) -> 74HC86DR2GOSCT-ND
- U33: footprint (none) -> SO14E
- U33: footprint (none) -> SO14E; mfg (none) -> on semi; mfg# (none) -> 74HC86DR2G; vend1 (none) -> digikey; vend1# (none) -> 74HC86DR2GOSCT-ND
Changed lines of the file:
@@
-EESchema Schematic File Version 2  date 2/16/2011 5:39:13 AM
+EESchema Schematic File Version 2  date 2/16/2011 8:44:18 AM
 LIBS:power
 LIBS:freeEMS_lib
@@
 F 0 "R232" V 7130 8350 50  0000 C CNN
 F 1 "1.6k" V 7050 8350 50  0000 C CNN
+F 2 "SM0805" V 1130 2600 60  0001 C CNN
 F 4 "Stackpole Electronics Inc" V 1130 2600 60  0001 C CNN "mfg"
 F 5 "RMCF0805JT1K00CT" V 1130 2600 60  0001 C CNN "mfg#"
@@
 F 0 "R233" V 7130 8800 50  0000 C CNN
 F 1 "1.6k" V 7050 8800 50  0000 C CNN
+F 2 "SM0805" V 1130 2600 60  0001 C CNN
 F 4 "Stackpole Electronics Inc" V 1130 2600 60  0001 C CNN "mfg"
 F 5 "RMCF0805JT1K00CT" V 1130 2600 60  0001 C CNN "mfg#"
@@
 F 0 "R231" V 7130 7900 50  0000 C CNN
 F 1 "1.6k" V 7050 7900 50  0000 C CNN
+F 2 "SM0805" V 1130 2600 60  0001 C CNN
 F 4 "Stackpole Electronics Inc" V 1130 2600 60  0001 C CNN "mfg"
 F 5 "RMCF0805JT1K00CT" V 1130 2600 60  0001 C CNN "mfg#"
@@
 F 0 "R230" V 7130 7450 50  0000 C CNN
 F 1 "1.6k" V 7050 7450 50  0000 C CNN
+F 2 "SM0805" V 1130 2600 60  0001 C CNN
 F 4 "Stackpole Electronics Inc" V 1130 2600 60  0001 C CNN "mfg"
 F 5 "RMCF0805JT1K00CT" V 1130 2600 60  0001 C CNN "mfg#"
@@
 F 0 "R229" V 6830 9300 50  0000 C CNN
 F 1 "10k" V 6750 9300 50  0000 C CNN
+F 2 "SM0805" V 1130 2600 60  0001 C CNN
 F 4 "Stackpole" V 1130 2600 60  0001 C CNN "mfg"
 F 5 "RMCF0805JT10K0CT" V 1130 2600 60  0001 C CNN "mfg#"
@@
 F 0 "R228" V 6630 9300 50  0000 C CNN
 F 1 "10k" V 6550 9300 50  0000 C CNN
+F 2 "SM0805" V 1130 2600 60  0001 C CNN
 F 4 "Stackpole" V 1130 2600 60  0001 C CNN "mfg"
 F 5 "RMCF0805JT10K0CT" V 1130 2600 60  0001 C CNN "mfg#"
@@
 F 0 "U33" H 5500 8950 50  0000 C CNN
 F 1 "74LS86" H 5500 8850 40  0000 C CNN
+F 2 "SO14E" H 5450 8900 60  0001 C CNN
+F 4 "on semi" H 5450 8900 60  0001 C CNN "mfg"
+F 5 "74HC86DR2G" H 5450 8900 60  0001 C CNN "mfg#"
+F 6 "digikey" H 5450 8900 60  0001 C CNN "vend1"
+F 7 "74HC86DR2GOSCT-ND" H 5450 8900 60  0001 C CNN "vend1#"
 	4    5450 8900
 	-1   0    0    -1
@@
 F 0 "U33" H 5500 8500 50  0000 C CNN
 F 1 "74LS86" H 5500 8400 40  0000 C CNN
+F 2 "SO14E" H 5450 8450 60  0001 C CNN
 	3    5450 8450
 	-1   0    0    -1
@@
 F 0 "U33" H 5500 8050 50  0000 C CNN
 F 1 "74LS86" H 5500 7950 40  0000 C CNN
+F 2 "SO14E" H 5450 8000 60  0001 C CNN
 	2    5450 8000
 	-1   0    0    -1
@@
 F 0 "U33" H 5500 7600 50  0000 C CNN
 F 1 "74LS86" H 5500 7500 40  0000 C CNN
-F 5 "74HC86DR2GOSCT-ND" H 5450 7550 60  0001 C CNN "Field2"
+F 2 "SO14E" H 5450 7550 60  0001 C CNN
+F 4 "on semi" H 5450 7550 60  0001 C CNN "mfg"
+F 5 "74HC86DR2G" H 5450 7550 60  0001 C CNN "mfg#"
+F 6 "digikey" H 5450 7550 60  0001 C CNN "vend1"
+F 7 "74HC86DR2GOSCT-ND" H 5450 7550 60  0001 C CNN "vend1#"
 	1    5450 7550
 	-1   0    0    -1

Commit message: Silkscreen rearrange, fat 12v track ready to be removed, VR resistors changed to 1210, intra-protection circuits removed, changed XOR resistor to 330ohm, new config for FT232, fixed osc schematic, fixed MAP diagnosis pullup
Parts:
- removed P75, P77, P79, P81, P83, P85, P87, P89: CONN_1, PINTST, symbol CONN_1
Changed lines of the file:
@@
-EESchema Schematic File Version 2  date 2/20/2011 12:36:46 PM
+EESchema Schematic File Version 2  date Wed 23 Feb 2011 05:11:09 AM ART
 LIBS:power
 LIBS:freeEMS_lib
@@
 EELAYER END
 $Descr A2 23400 16535
-Sheet 1 56
+Sheet 1 54
 Title "Puma board"
-Date "20 feb 2011"
+Date "23 feb 2011"
 Rev "v0.01"
 Comp "diyefi.org"
@@
 $EndDescr
 Wire Wire Line
+	19000 14200 19000 1200
+Wire Wire Line
+	12200 11900 15000 11900
+Wire Wire Line
 	3700 1400 4600 1400
 Connection ~ 19000 5300
@@
 Wire Wire Line
 	19000 2350 18000 2350
-Connection ~ 19000 1750
-Connection ~ 19000 1750
-Connection ~ 19000 1750
-Connection ~ 19000 1750
 Wire Wire Line
 	18000 1750 18450 1750
-Connection ~ 19000 1750
-Connection ~ 19000 1750
-Connection ~ 19000 1750
-Connection ~ 19000 2250
-Connection ~ 19000 2250
-Connection ~ 19000 2250
 Wire Wire Line
 	18000 2250 18450 2250
-Connection ~ 19000 2250
-Connection ~ 19000 2250
-Connection ~ 19000 2250
-Connection ~ 19000 2750
-Connection ~ 19000 2750
-Connection ~ 19000 2750
 Wire Wire Line
 	18000 2750 18450 2750
-Connection ~ 19000 2750
-Connection ~ 19000 2750
-Connection ~ 19000 3250
-Connection ~ 19000 3250
 Wire Wire Line
 	18000 3250 18450 3250
-Connection ~ 19000 3250
-Connection ~ 19000 3250
-Connection ~ 19000 3750
-Connection ~ 19000 3750
 Wire Wire Line
 	18000 3750 18450 3750
-Connection ~ 19000 3750
-Connection ~ 19000 4200
 Wire Wire Line
 	18000 4200 18450 4200
-Connection ~ 19000 4200
-Connection ~ 19000 4700
 Wire Wire Line
 	18000 4700 18450 4700
@@
 	6500 6950 6200 6950
 Wire Bus Line
-	12100 13200 12100 9650
+	12100 9650 12100 13200
 Wire Wire Line
 	6750 4650 7150 4650
@@
 Wire Wire Line
 	12200 12850 15000 12850
-Connection ~ 14850 12000
-Wire Wire Line
-	14850 12050 14850 11500
 Wire Wire Line
 	7000 12500 4350 12500
@@
 	9150 3650 10100 3650
 Wire Bus Line
-	14250 10700 14250 1750
+	14250 1750 14250 10700
 Wire Wire Line
 	15050 2150 14350 2150
@@
 Wire Wire Line
 	14850 3250 15050 3250
-Connection ~ 19000 2750
 Wire Wire Line
 	5350 3600 5300 3600
@@
 Connection ~ 6850 11150
 Wire Wire Line
-	6850 10350 6750 10350
-Wire Wire Line
-	6750 11150 6850 11150
+	6750 10350 6850 10350
+Wire Wire Line
+	6850 11150 6750 11150
 Wire Wire Line
 	6850 9950 6750 9950
@@
 Connection ~ 18200 12850
 Wire Wire Line
-	12900 11400 12200 11400
-Wire Wire Line
-	12900 11900 12200 11900
-Wire Wire Line
-	14550 12000 14850 12000
-Wire Wire Line
-	14550 11400 15000 11400
-Wire Wire Line
 	9150 5800 9600 5800
 Wire Wire Line
@@
 Wire Wire Line
 	18850 6500 18000 6500
-Connection ~ 19000 5200
-Connection ~ 19000 4200
-Connection ~ 19000 3250
 Wire Wire Line
 	19000 9100 18000 9100
@@
 Wire Wire Line
 	5300 2750 5450 2750
-Connection ~ 19000 3750
-Connection ~ 19000 4700
 Connection ~ 18850 6050
 Wire Wire Line
@@
 Wire Wire Line
 	9150 5700 9600 5700
-Wire Wire Line
-	14550 11900 15000 11900
-Wire Wire Line
-	14850 11500 14550 11500
 Wire Wire Line
 	14350 6400 15000 6400
@@
 Connection ~ 6850 10750
 Wire Wire Line
-	10850 14200 19000 14200
+	19000 14200 10850 14200
 Wire Wire Line
 	10850 14200 10850 9950
@@
 Wire Wire Line
 	14850 2250 15050 2250
-Connection ~ 19000 2250
 Connection ~ 18150 2650
 Wire Wire Line
 	18000 1650 18150 1650
 Wire Wire Line
-	6250 1200 19000 1200
-Wire Wire Line
-	19000 1200 19000 14200
-Connection ~ 19000 1750
+	19000 1200 6250 1200
 Wire Wire Line
 	15050 1650 14350 1650
@@
 	7200 1400 18850 1400
 Wire Wire Line
-	10550 12300 10850 12300
+	10850 12300 10550 12300
 Connection ~ 10850 12300
 Wire Wire Line
@@
 Connection ~ 14850 1750
 Wire Wire Line
-	5300 2850 7800 2850
+	7800 2850 5300 2850
 Connection ~ 7200 2850
 Wire Wire Line
@@
 	6550 9050 6750 9050
 Wire Wire Line
-	6050 8100 6550 8100
+	6550 8100 6050 8100
 Connection ~ 6550 8100
 Wire Wire Line
-	6550 9000 6050 9000
+	6050 9000 6550 9000
 Connection ~ 6550 9000
 Wire Wire Line
@@
 Connection ~ 19000 1850
 Wire Wire Line
-	18000 2850 19000 2850
+	19000 2850 18000 2850
 Connection ~ 19000 2850
 Wire Wire Line
-	18000 3850 19000 3850
+	19000 3850 18000 3850
 Connection ~ 19000 3850
 Wire Wire Line
-	18000 4800 19000 4800
+	19000 4800 18000 4800
 Connection ~ 19000 4800
+Wire Wire Line
+	15000 11400 12200 11400
 $Comp
 L FUSE F3
@@
 	1    0    0    -1
 $EndComp
-$Comp
-L CONN_1 P89
-U 1 1 4D187542
-P 19150 1750
-F 0 "P89" H 19230 1750 40  0000 L CNN
-F 1 "CONN_1" H 19150 1805 30  0001 C CNN
-F 2 "PINTST" H 19150 1750 60  0001 C CNN
-	1    19150 1750
-	1    0    0    -1
-$EndComp
 Text Label 18250 1750 0    60   ~ 0
 inj8
 Text Label 18250 2250 0    60   ~ 0
 inj7
-$Comp
-L CONN_1 P87
-U 1 1 4D18753E
-P 19150 2250
-F 0 "P87" H 19230 2250 40  0000 L CNN
-F 1 "CONN_1" H 19150 2305 30  0001 C CNN
-F 2 "PINTST" H 19150 2250 60  0001 C CNN
-	1    19150 2250
-	1    0    0    -1
-$EndComp
 $Comp
 L CONN_1 P88
@@
 	1    0    0    -1
 $EndComp
-$Comp
-L CONN_1 P75
-U 1 1 4D187534
-P 19150 2750
-F 0 "P75" H 19230 2750 40  0000 L CNN
-F 1 "CONN_1" H 19150 2805 30  0001 C CNN
-F 2 "PINTST" H 19150 2750 60  0001 C CNN
-	1    19150 2750
-	1    0    0    -1
-$EndComp
 Text Label 18250 2750 0    60   ~ 0
 inj6
 Text Label 18250 3250 0    60   ~ 0
 inj5
-$Comp
-L CONN_1 P77
-U 1 1 4D187531
-P 19150 3250
-F 0 "P77" H 19230 3250 40  0000 L CNN
-F 1 "CONN_1" H 19150 3305 30  0001 C CNN
-F 2 "PINTST" H 19150 3250 60  0001 C CNN
-	1    19150 3250
-	1    0    0    -1
-$EndComp
 $Comp
 L CONN_1 P78
@@
 	1    0    0    -1
 $EndComp
-$Comp
-L CONN_1 P79
-U 1 1 4D18752C
-P 19150 3750
-F 0 "P79" H 19230 3750 40  0000 L CNN
-F 1 "CONN_1" H 19150 3805 30  0001 C CNN
-F 2 "PINTST" H 19150 3750 60  0001 C CNN
-	1    19150 3750
-	1    0    0    -1
-$EndComp
 Text Label 18250 3750 0    60   ~ 0
 inj4
 Text Label 18250 4200 0    60   ~ 0
 inj3
-$Comp
-L CONN_1 P81
-U 1 1 4D187529
-P 19150 4200
-F 0 "P81" H 19230 4200 40  0000 L CNN
-F 1 "CONN_1" H 19150 4255 30  0001 C CNN
-F 2 "PINTST" H 19150 4200 60  0001 C CNN
-	1    19150 4200
-	1    0    0    -1
-$EndComp
 $Comp
 L CONN_1 P82
@@
 	1    0    0    -1
 $EndComp
-$Comp
-L CONN_1 P83
-U 1 1 4D187522
-P 19150 4700
-F 0 "P83" H 19230 4700 40  0000 L CNN
-F 1 "CONN_1" H 19150 4755 30  0001 C CNN
-F 2 "PINTST" H 19150 4700 60  0001 C CNN
-	1    19150 4700
-	1    0    0    -1
-$EndComp
 Text Label 18250 4700 0    60   ~ 0
 inj2
 Text Label 18250 5200 0    60   ~ 0
 inj1
-$Comp
-L CONN_1 P85
-U 1 1 4D1873A5
-P 19150 5200
-F 0 "P85" H 19230 5200 40  0000 L CNN
-F 1 "CONN_1" H 19150 5255 30  0001 C CNN
-F 2 "PINTST" H 19150 5200 60  0001 C CNN
-	1    19150 5200
-	1    0    0    -1
-$EndComp
 $Comp
 L CONN_1 P86
@@
 F83 "5v_microcontroller" I L 7800 2950 60
 $EndSheet
-$Comp
-L GND #PWR03
-U 1 1 4CB3CDC4
-P 14850 12050
-F 0 "#PWR03" H 14850 12050 30  0001 C CNN
-F 1 "GND" H 14850 11980 30  0001 C CNN
-	1    14850 12050
-	1    0    0    -1
-$EndComp
 NoConn ~ 7800 4550
 NoConn ~ 7800 4650
@@
 $EndSheet
 $Comp
-L PWR_FLAG #FLG04
+L PWR_FLAG #FLG03
 U 1 1 4C8266A6
 P 4600 1400
-F 0 "#FLG04" H 4600 1670 30  0001 C CNN
+F 0 "#FLG03" H 4600 1670 30  0001 C CNN
 F 1 "PWR_FLAG" H 4600 1630 30  0000 C CNN
 	1    4600 1400
@@
 $EndComp
 $Comp
-L GND #PWR05
+L GND #PWR04
 U 1 1 4C826576
 P 5850 9550
-F 0 "#PWR05" H 5850 9550 30  0001 C CNN
+F 0 "#PWR04" H 5850 9550 30  0001 C CNN
 F 1 "GND" H 5850 9480 30  0001 C CNN
 	1    5850 9550
@@
 	4250 9750 4350 9850
 $Comp
-L GND #PWR06
+L GND #PWR05
 U 1 1 489663FC
 P 12650 4900
-F 0 "#PWR06" H 12650 4900 30  0001 C CNN
+F 0 "#PWR05" H 12650 4900 30  0001 C CNN
 F 1 "GND" H 12650 4830 30  0001 C CNN
 	1    12650 4900
@@
 $EndComp
 $Comp
-L GND #PWR07
+L GND #PWR06
 U 1 1 489663D4
 P 4550 5400
-F 0 "#PWR07" H 4550 5400 30  0001 C CNN
+F 0 "#PWR06" H 4550 5400 30  0001 C CNN
 F 1 "GND" H 4550 5330 30  0001 C CNN
 	1    4550 5400
@@
 NoConn ~ 9150 4450
 $Comp
-L GND #PWR08
+L GND #PWR07
 U 1 1 489662CC
 P 18200 11000
-F 0 "#PWR08" H 18200 11000 30  0001 C CNN
+F 0 "#PWR07" H 18200 11000 30  0001 C CNN
 F 1 "GND" H 18200 10930 30  0001 C CNN
 	1    18200 11000
@@
 F3 "analog_sensor_MAP" O L 15000 7750 60
 F4 "5v reg" I R 18000 7850 60
-$EndSheet
-$Sheet
-S 12900 11350 1650 200
-U 4C2E1E73
-F0 "digi_protect_rpm1" 60
-F1 "digi_protect_rpm1.sch" 60
-F2 "digi_CPU" B L 12900 11400 60
-F3 "digi_device" B R 14550 11400 60
-F4 "digi_gnd" B R 14550 11500 60
-$EndSheet
-$Sheet
-S 12900 11850 1650 200
-U 4C2E1E75
-F0 "digi_protect_rpm2" 60
-F1 "digi_protect_rpm2.sch" 60
-F2 "digi_CPU" B L 12900 11900 60
-F3 "digi_device" B R 14550 11900 60
-F4 "digi_gnd" B R 14550 12000 60
 $EndSheet
 Text Label 12750 5700 0    60   ~ 0
@@
 	14250 2750 14350 2650
 $Comp
-L GND #PWR09
+L GND #PWR08
 U 1 1 486F7889
 P 18200 11950
-F 0 "#PWR09" H 18200 11950 30  0001 C CNN
+F 0 "#PWR08" H 18200 11950 30  0001 C CNN
 F 1 "GND" H 18200 11880 30  0001 C CNN
 	1    18200 11950
@@
 $EndComp
 $Comp
-L GND #PWR010
+L GND #PWR09
 U 1 1 486F7315
 P 5350 3750
-F 0 "#PWR010" H 5350 3750 30  0001 C CNN
+F 0 "#PWR09" H 5350 3750 30  0001 C CNN
 F 1 "GND" H 5350 3680 30  0001 C CNN
 	1    5350 3750
