File: design/an_protect2.sch (KiCad schematic (older format))
At the start: 20 parts

Commit message: updating bom, lets commit this before I run a script to update the footprints for the resistors
Signed-off-by: Jared Harvey <TortiseGIT@jaredharvey.com>
Parts:
- D31, D33, D35, D74: footprint D4-SMB -> SOD-123
Changed lines of the file:
@@
-EESchema Schematic File Version 2  date 2/14/2011 7:45:19 AM
+EESchema Schematic File Version 2  date 2/16/2011 5:39:17 AM
 LIBS:power
 LIBS:freeEMS_lib
@@
 EELAYER END
 $Descr A 11000 8500
-Sheet 47 55
+Sheet 47 56
 Title "Puma board"
-Date "14 feb 2011"
+Date "16 feb 2011"
 Rev "v0.02"
 Comp "diyefi.org"
@@
 F 0 "D74" H 2650 5150 40  0000 C CNN
 F 1 "1N4148" H 2650 4950 40  0000 C CNN
-F 2 "D4-SMB" V 1130 4000 60  0001 C CNN
+F 2 "SOD-123" V 1130 4000 60  0001 C CNN
 F 4 "Micro Commercial Co" V 1130 2600 60  0001 C CNN "mfg"
 F 5 "1N4148W-TP" V 1130 2600 60  0001 C CNN "mfg#"
@@
 F 0 "D31" H 2650 3750 40  0000 C CNN
 F 1 "1N4148" H 2650 3550 40  0000 C CNN
-F 2 "D4-SMB" V 1130 2600 60  0001 C CNN
+F 2 "SOD-123" V 1130 2600 60  0001 C CNN
 F 4 "Micro Commercial Co" V 1130 2600 60  0001 C CNN "mfg"
 F 5 "1N4148W-TP" V 1130 2600 60  0001 C CNN "mfg#"
@@
 F 0 "D33" H 2700 2450 40  0000 C CNN
 F 1 "1N4148" H 2700 2250 40  0000 C CNN
-F 2 "D4-SMB" V 1130 2600 60  0001 C CNN
+F 2 "SOD-123" V 1130 2600 60  0001 C CNN
 F 4 "Micro Commercial Co" V 1130 2600 60  0001 C CNN "mfg"
 F 5 "1N4148W-TP" V 1130 2600 60  0001 C CNN "mfg#"
@@
 F 0 "D35" H 2750 1100 40  0000 C CNN
 F 1 "1N4148" H 2750 900 40  0000 C CNN
-F 2 "D4-SMB" V 1130 2600 60  0001 C CNN
+F 2 "SOD-123" V 1130 2600 60  0001 C CNN
 F 4 "Micro Commercial Co" V 1130 2600 60  0001 C CNN "mfg"
 F 5 "1N4148W-TP" V 1130 2600 60  0001 C CNN "mfg#"

Commit message: Schematic BOM is now fully populated with only 3 exceptions, .cmp file is obsolete at this point, so it has been removed.
Signed-off-by: Jared Harvey <TortiseGIT@jaredharvey.com>
Parts:
- R186, R187, R47, R48, R49, R50, R51, R52: footprint R4-SM0805 -> SM0805
Changed lines of the file:
@@
-EESchema Schematic File Version 2  date 2/16/2011 5:39:17 AM
+EESchema Schematic File Version 2  date 2/16/2011 8:44:21 AM
 LIBS:power
 LIBS:freeEMS_lib
@@
 F 0 "R186" V 2330 5450 50  0000 C CNN
 F 1 "1k" V 2250 5450 50  0000 C CNN
-F 2 "R4-SM0805" V 2430 5550 60  0001 C CNN
+F 2 "SM0805" V 1130 2600 60  0001 C CNN
 F 4 "Stackpole" V 1130 2600 60  0001 C CNN "mfg"
 F 5 "RMCF0805JT1K00" V 1130 2600 60  0001 C CNN "mfg#"
@@
 $EndComp
 $Comp
-L GND #PWR075
+L GND #PWR073
 U 1 1 4C5989C2
 P 2000 5900
-F 0 "#PWR075" H 2000 5900 30  0001 C CNN
+F 0 "#PWR073" H 2000 5900 30  0001 C CNN
 F 1 "GND" H 2000 5830 30  0001 C CNN
 	1    2000 5900
@@
 F 0 "R187" V 4030 5450 50  0000 C CNN
 F 1 "1k" V 3950 5450 50  0000 C CNN
-F 2 "R4-SM0805" V 4130 5550 60  0001 C CNN
+F 2 "SM0805" V 1130 2600 60  0001 C CNN
 F 4 "Stackpole" V 1130 2600 60  0001 C CNN "mfg"
 F 5 "RMCF0805JT1K00" V 1130 2600 60  0001 C CNN "mfg#"
@@
 F 0 "R50" V 4030 4050 50  0000 C CNN
 F 1 "1k" V 3950 4050 50  0000 C CNN
-F 2 "R4-SM0805" V 4130 4150 60  0001 C CNN
+F 2 "SM0805" V 1130 2600 60  0001 C CNN
 F 4 "Stackpole" V 1130 2600 60  0001 C CNN "mfg"
 F 5 "RMCF0805JT1K00" V 1130 2600 60  0001 C CNN "mfg#"
@@
 P 2000 4500
 AR Path="/4C4C6618/4C2F52F6" Ref="#PWR056"  Part="1"
-AR Path="/4C2E1E7B/4C2F52F6" Ref="#PWR076"  Part="1"
-F 0 "#PWR076" H 2000 4500 30  0001 C CNN
+AR Path="/4C2E1E7B/4C2F52F6" Ref="#PWR074"  Part="1"
+F 0 "#PWR074" H 2000 4500 30  0001 C CNN
 F 1 "GND" H 2000 4430 30  0001 C CNN
 	1    2000 4500
@@
 F 0 "R47" V 2330 4050 50  0000 C CNN
 F 1 "1k" V 2250 4050 50  0000 C CNN
-F 2 "R4-SM0805" V 2430 4150 60  0001 C CNN
+F 2 "SM0805" V 1130 2600 60  0001 C CNN
 F 4 "Stackpole" V 1130 2600 60  0001 C CNN "mfg"
 F 5 "RMCF0805JT1K00" V 1130 2600 60  0001 C CNN "mfg#"
@@
 F 0 "R51" V 4080 2750 50  0000 C CNN
 F 1 "1k" V 4000 2750 50  0000 C CNN
-F 2 "R4-SM0805" V 4180 2850 60  0001 C CNN
+F 2 "SM0805" V 1130 2600 60  0001 C CNN
 F 4 "Stackpole" V 1130 2600 60  0001 C CNN "mfg"
 F 5 "RMCF0805JT1K00" V 1130 2600 60  0001 C CNN "mfg#"
@@
 P 2050 3200
 AR Path="/4C4C6618/489597B8" Ref="#PWR057"  Part="1"
-AR Path="/4C2E1E7B/489597B8" Ref="#PWR077"  Part="1"
-F 0 "#PWR077" H 2050 3200 30  0001 C CNN
+AR Path="/4C2E1E7B/489597B8" Ref="#PWR075"  Part="1"
+F 0 "#PWR075" H 2050 3200 30  0001 C CNN
 F 1 "GND" H 2050 3130 30  0001 C CNN
 	1    2050 3200
@@
 F 0 "R48" V 2380 2750 50  0000 C CNN
 F 1 "1k" V 2300 2750 50  0000 C CNN
-F 2 "R4-SM0805" V 2480 2850 60  0001 C CNN
+F 2 "SM0805" V 1130 2600 60  0001 C CNN
 F 4 "Stackpole" V 1130 2600 60  0001 C CNN "mfg"
 F 5 "RMCF0805JT1K00" V 1130 2600 60  0001 C CNN "mfg#"
@@
 F 0 "R52" V 4130 1400 50  0000 C CNN
 F 1 "1k" V 4050 1400 50  0000 C CNN
-F 2 "R4-SM0805" V 4230 1500 60  0001 C CNN
+F 2 "SM0805" V 1130 2600 60  0001 C CNN
 F 4 "Stackpole" V 1130 2600 60  0001 C CNN "mfg"
 F 5 "RMCF0805JT1K00" V 1130 2600 60  0001 C CNN "mfg#"
@@
 P 2100 1850
 AR Path="/4C4C6618/4C2F52A8" Ref="#PWR058"  Part="1"
-AR Path="/4C2E1E7B/4C2F52A8" Ref="#PWR078"  Part="1"
-F 0 "#PWR078" H 2100 1850 30  0001 C CNN
+AR Path="/4C2E1E7B/4C2F52A8" Ref="#PWR076"  Part="1"
+F 0 "#PWR076" H 2100 1850 30  0001 C CNN
 F 1 "GND" H 2100 1780 30  0001 C CNN
 	1    2100 1850
@@
 F 0 "R49" V 2430 1400 50  0000 C CNN
 F 1 "1k" V 2350 1400 50  0000 C CNN
-F 2 "R4-SM0805" V 2530 1500 60  0001 C CNN
-F 4 "Stackpole" V 1130 2600 60  0001 C CNN "mfg"
-F 5 "RMCF0805JT1K00" V 1130 2600 60  0001 C CNN "mfg#"
+F 2 "SM0805" V 1130 2600 60  0001 C CNN
+F 4 "Stackpole" V 1130 2600 60  0001 C CNN "mfg"
+F 5 "RMCF0805JT1K00" V 1130 2600 60  0001 C CNN "mfg#"
