File: design/an_protect4.sch (KiCad schematic (older format))
At the start: 20 parts

Commit message: updating bom, lets commit this before I run a script to update the footprints for the resistors
Signed-off-by: Jared Harvey <TortiseGIT@jaredharvey.com>
Parts:
- D66, D68, D70, D72: footprint D4-SMB -> SOD-123
Changed lines of the file:
@@
-EESchema Schematic File Version 2  date 2/14/2011 7:45:18 AM
+EESchema Schematic File Version 2  date 2/16/2011 5:39:15 AM
 LIBS:power
 LIBS:freeEMS_lib
@@
 EELAYER END
 $Descr A 11000 8500
-Sheet 24 55
+Sheet 24 56
 Title "Puma board"
-Date "14 feb 2011"
+Date "16 feb 2011"
 Rev "v0.02"
 Comp "diyefi.org"
@@
 AR Path="/4C4C6618/4C4973C4" Ref="D67"  Part="1"
 AR Path="/4C2E1E7D/4C4973C4" Ref="D59"  Part="1"
-F 0 "D59" H 2600 5750 40  0000 C CNN
+F 0 "D67" H 2600 5750 40  0000 C CNN
 F 1 "SCHOTTKY" H 2600 5550 40  0000 C CNN
 F 2 "SOD-123" H 2600 5650 60  0001 C CNN
@@
 AR Path="/4C4C6618/4C4973C0" Ref="D69"  Part="1"
 AR Path="/4C2E1E7D/4C4973C0" Ref="D61"  Part="1"
-F 0 "D61" H 2650 4350 40  0000 C CNN
+F 0 "D69" H 2650 4350 40  0000 C CNN
 F 1 "SCHOTTKY" H 2650 4150 40  0000 C CNN
 F 2 "SOD-123" H 2650 4250 60  0001 C CNN
@@
 AR Path="/4C4C6618/4C4973B6" Ref="D71"  Part="1"
 AR Path="/4C2E1E7D/4C4973B6" Ref="D63"  Part="1"
-F 0 "D63" H 2700 3050 40  0000 C CNN
+F 0 "D71" H 2700 3050 40  0000 C CNN
 F 1 "SCHOTTKY" H 2700 2850 40  0000 C CNN
 F 2 "SOD-123" H 2700 2950 60  0001 C CNN
@@
 AR Path="/4C4C6618/4C4973B0" Ref="D73"  Part="1"
 AR Path="/4C2E1E7D/4C4973B0" Ref="D65"  Part="1"
-F 0 "D65" H 2750 1700 40  0000 C CNN
+F 0 "D73" H 2750 1700 40  0000 C CNN
 F 1 "SCHOTTKY" H 2750 1500 40  0000 C CNN
 F 2 "SOD-123" H 2750 1600 60  0001 C CNN
@@
 AR Path="/4C4C6618/4C4C7B57" Ref="R171"  Part="1"
 AR Path="/4C2E1E7D/4C4C7B57" Ref="R163"  Part="1"
-F 0 "R163" V 3980 5450 50  0000 C CNN
+F 0 "R171" V 3980 5450 50  0000 C CNN
 F 1 "1k" V 3900 5450 50  0000 C CNN
 F 2 "R4-SM0805" V 4080 5550 60  0001 C CNN
@@
 AR Path="/4C4C6618/489597C4" Ref="#PWR053"  Part="1"
 AR Path="/4C2E1E7D/489597C4" Ref="#PWR079"  Part="1"
-F 0 "#PWR079" H 1950 5900 30  0001 C CNN
+F 0 "#PWR053" H 1950 5900 30  0001 C CNN
 F 1 "GND" H 1950 5830 30  0001 C CNN
 	1    1950 5900
@@
 AR Path="/4C4C6618/489597C2" Ref="C89"  Part="1"
 AR Path="/4C2E1E7D/489597C2" Ref="C85"  Part="1"
-F 0 "C85" H 3200 5750 50  0000 L CNN
+F 0 "C89" H 3200 5750 50  0000 L CNN
 F 1 "0.1uF" H 3200 5550 50  0000 L CNN
 F 2 "SM0805" V 1130 2600 60  0001 C CNN
@@
 AR Path="/4C4C6618/489597C1" Ref="R167"  Part="1"
 AR Path="/4C2E1E7D/489597C1" Ref="R159"  Part="1"
-F 0 "R159" V 2280 5450 50  0000 C CNN
+F 0 "R167" V 2280 5450 50  0000 C CNN
 F 1 "1k" V 2200 5450 50  0000 C CNN
 F 2 "R4-SM0805" V 2380 5550 60  0001 C CNN
@@
 AR Path="/4C4C6618/489597C0" Ref="D66"  Part="1"
 AR Path="/4C2E1E7D/489597C0" Ref="D58"  Part="1"
-F 0 "D58" H 2600 5150 40  0000 C CNN
+F 0 "D66" H 2600 5150 40  0000 C CNN
 F 1 "1N4148" H 2600 4950 40  0000 C CNN
-F 2 "D4-SMB" V 1130 2600 60  0001 C CNN
+F 2 "SOD-123" V 1130 2600 60  0001 C CNN
 F 4 "Micro Commercial Co" V 1130 2600 60  0001 C CNN "mfg"
 F 5 "1N4148W-TP" V 1130 2600 60  0001 C CNN "mfg#"
@@
 AR Path="/4C4C6618/4C4C7B52" Ref="R172"  Part="1"
 AR Path="/4C2E1E7D/4C4C7B52" Ref="R164"  Part="1"
-F 0 "R164" V 4030 4050 50  0000 C CNN
+F 0 "R172" V 4030 4050 50  0000 C CNN
 F 1 "1k" V 3950 4050 50  0000 C CNN
 F 2 "R4-SM0805" V 4130 4150 60  0001 C CNN
@@
 AR Path="/4C4C6618/4C4C7B51" Ref="#PWR054"  Part="1"
 AR Path="/4C2E1E7D/4C4C7B51" Ref="#PWR080"  Part="1"
-F 0 "#PWR080" H 2000 4500 30  0001 C CNN
+F 0 "#PWR054" H 2000 4500 30  0001 C CNN
 F 1 "GND" H 2000 4430 30  0001 C CNN
 	1    2000 4500
@@
 AR Path="/4C4C6618/4C2F52F4" Ref="C90"  Part="1"
 AR Path="/4C2E1E7D/4C2F52F4" Ref="C86"  Part="1"
-F 0 "C86" H 3250 4350 50  0000 L CNN
+F 0 "C90" H 3250 4350 50  0000 L CNN
 F 1 "0.1uF" H 3250 4150 50  0000 L CNN
 F 2 "SM0805" V 1130 2600 60  0001 C CNN
@@
 AR Path="/4C4C6618/4C2F52F3" Ref="R168"  Part="1"
 AR Path="/4C2E1E7D/4C2F52F3" Ref="R160"  Part="1"
-F 0 "R160" V 2330 4050 50  0000 C CNN
+F 0 "R168" V 2330 4050 50  0000 C CNN
 F 1 "1k" V 2250 4050 50  0000 C CNN
 F 2 "R4-SM0805" V 2430 4150 60  0001 C CNN
@@
 AR Path="/4C4C6618/4C4C7B50" Ref="D68"  Part="1"
 AR Path="/4C2E1E7D/4C4C7B50" Ref="D60"  Part="1"
-F 0 "D60" H 2650 3750 40  0000 C CNN
+F 0 "D68" H 2650 3750 40  0000 C CNN
 F 1 "1N4148" H 2650 3550 40  0000 C CNN
-F 2 "D4-SMB" V 1130 2600 60  0001 C CNN
+F 2 "SOD-123" V 1130 2600 60  0001 C CNN
 F 4 "Micro Commercial Co" V 1130 2600 60  0001 C CNN "mfg"
 F 5 "1N4148W-TP" V 1130 2600 60  0001 C CNN "mfg#"
@@
 AR Path="/4C4C6618/489597B9" Ref="R173"  Part="1"
 AR Path="/4C2E1E7D/489597B9" Ref="R165"  Part="1"
-F 0 "R165" V 4080 2750 50  0000 C CNN
+F 0 "R173" V 4080 2750 50  0000 C CNN
 F 1 "1k" V 4000 2750 50  0000 C CNN
 F 2 "R4-SM0805" V 4180 2850 60  0001 C CNN
@@
 AR Path="/4C4C6618/4C2F52F0" Ref="#PWR055"  Part="1"
 AR Path="/4C2E1E7D/4C2F52F0" Ref="#PWR081"  Part="1"
-F 0 "#PWR081" H 2050 3200 30  0001 C CNN
+F 0 "#PWR055" H 2050 3200 30  0001 C CNN
 F 1 "GND" H 2050 3130 30  0001 C CNN
 	1    2050 3200
@@
 AR Path="/4C4C6618/4C4C7B5C" Ref="C91"  Part="1"
 AR Path="/4C2E1E7D/4C4C7B5C" Ref="C87"  Part="1"
-F 0 "C87" H 3300 3050 50  0000 L CNN
+F 0 "C91" H 3300 3050 50  0000 L CNN
 F 1 "0.1uF" H 3300 2850 50  0000 L CNN
 F 2 "SM0805" V 1130 2600 60  0001 C CNN
@@
 AR Path="/4C4C6618/4C2F52ED" Ref="R169"  Part="1"
 AR Path="/4C2E1E7D/4C2F52ED" Ref="R161"  Part="1"
-F 0 "R161" V 2380 2750 50  0000 C CNN
+F 0 "R169" V 2380 2750 50  0000 C CNN
 F 1 "1k" V 2300 2750 50  0000 C CNN
 F 2 "R4-SM0805" V 2480 2850 60  0001 C CNN
@@
 AR Path="/4C4C6618/4C2F52EC" Ref="D70"  Part="1"
 AR Path="/4C2E1E7D/4C2F52EC" Ref="D62"  Part="1"
-F 0 "D62" H 2700 2450 40  0000 C CNN
+F 0 "D70" H 2700 2450 40  0000 C CNN
 F 1 "1N4148" H 2700 2250 40  0000 C CNN
-F 2 "D4-SMB" V 1130 2600 60  0001 C CNN
+F 2 "SOD-123" V 1130 2600 60  0001 C CNN
 F 4 "Micro Commercial Co" V 1130 2600 60  0001 C CNN "mfg"
 F 5 "1N4148W-TP" V 1130 2600 60  0001 C CNN "mfg#"
@@
 AR Path="/4C4C6618/4C2F52DC" Ref="R174"  Part="1"
 AR Path="/4C2E1E7D/4C2F52DC" Ref="R166"  Part="1"
-F 0 "R166" V 4130 1400 50  0000 C CNN
+F 0 "R174" V 4130 1400 50  0000 C CNN
 F 1 "1k" V 4050 1400 50  0000 C CNN
 F 2 "R4-SM0805" V 4230 1500 60  0001 C CNN
@@
 AR Path="/4C4C6618/4C4C7B4E" Ref="#PWR056"  Part="1"
 AR Path="/4C2E1E7D/4C4C7B4E" Ref="#PWR082"  Part="1"
-F 0 "#PWR082" H 2100 1850 30  0001 C CNN
+F 0 "#PWR056" H 2100 1850 30  0001 C CNN
 F 1 "GND" H 2100 1780 30  0001 C CNN
 	1    2100 1850
@@
 AR Path="/4C4C6618/4C4C7B4D" Ref="C92"  Part="1"
 AR Path="/4C2E1E7D/4C4C7B4D" Ref="C88"  Part="1"
-F 0 "C88" H 3350 1700 50  0000 L CNN
+F 0 "C92" H 3350 1700 50  0000 L CNN
 F 1 "0.1uF" H 3350 1500 50  0000 L CNN
 F 2 "SM0805" V 1130 2600 60  0001 C CNN
@@
 AR Path="/4C4C6618/4C4C7B4C" Ref="R170"  Part="1"
 AR Path="/4C2E1E7D/4C4C7B4C" Ref="R162"  Part="1"
-F 0 "R162" V 2430 1400 50  0000 C CNN
+F 0 "R170" V 2430 1400 50  0000 C CNN
 F 1 "1k" V 2350 1400 50  0000 C CNN
 F 2 "R4-SM0805" V 2530 1500 60  0001 C CNN
@@
 AR Path="/4C4C6618/4C2F52A4" Ref="D72"  Part="1"
 AR Path="/4C2E1E7D/4C2F52A4" Ref="D64"  Part="1"
-F 0 "D64" H 2750 1100 40  0000 C CNN
+F 0 "D72" H 2750 1100 40  0000 C CNN
 F 1 "1N4148" H 2750 900 40  0000 C CNN
-F 2 "D4-SMB" V 1130 2600 60  0001 C CNN
+F 2 "SOD-123" V 1130 2600 60  0001 C CNN
 F 4 "Micro Commercial Co" V 1130 2600 60  0001 C CNN "mfg"
 F 5 "1N4148W-TP" V 1130 2600 60  0001 C CNN "mfg#"

Commit message: Schematic BOM is now fully populated with only 3 exceptions, .cmp file is obsolete at this point, so it has been removed.
Signed-off-by: Jared Harvey <TortiseGIT@jaredharvey.com>
Parts:
- R167, R168, R169, R170, R171, R172, R173, R174: footprint R4-SM0805 -> SM0805
Changed lines of the file:
@@
-EESchema Schematic File Version 2  date 2/16/2011 5:39:15 AM
+EESchema Schematic File Version 2  date 2/16/2011 8:44:19 AM
 LIBS:power
 LIBS:freeEMS_lib
@@
 F 0 "R171" V 3980 5450 50  0000 C CNN
 F 1 "1k" V 3900 5450 50  0000 C CNN
-F 2 "R4-SM0805" V 4080 5550 60  0001 C CNN
+F 2 "SM0805" V 1130 2600 60  0001 C CNN
 F 4 "Stackpole" V 1130 2600 60  0001 C CNN "mfg"
 F 5 "RMCF0805JT1K00" V 1130 2600 60  0001 C CNN "mfg#"
@@
 $EndComp
 $Comp
-L GND #PWR053
+L GND #PWR051
 U 1 1 489597C4
 P 1950 5900
-AR Path="/4C4C6618/489597C4" Ref="#PWR053"  Part="1"
-AR Path="/4C2E1E7D/489597C4" Ref="#PWR079"  Part="1"
-F 0 "#PWR053" H 1950 5900 30  0001 C CNN
+AR Path="/4C4C6618/489597C4" Ref="#PWR051"  Part="1"
+AR Path="/4C2E1E7D/489597C4" Ref="#PWR077"  Part="1"
+F 0 "#PWR077" H 1950 5900 30  0001 C CNN
 F 1 "GND" H 1950 5830 30  0001 C CNN
 	1    1950 5900
@@
 F 0 "R167" V 2280 5450 50  0000 C CNN
 F 1 "1k" V 2200 5450 50  0000 C CNN
-F 2 "R4-SM0805" V 2380 5550 60  0001 C CNN
+F 2 "SM0805" V 1130 2600 60  0001 C CNN
 F 4 "Stackpole" V 1130 2600 60  0001 C CNN "mfg"
 F 5 "RMCF0805JT1K00" V 1130 2600 60  0001 C CNN "mfg#"
@@
 F 0 "R172" V 4030 4050 50  0000 C CNN
 F 1 "1k" V 3950 4050 50  0000 C CNN
-F 2 "R4-SM0805" V 4130 4150 60  0001 C CNN
+F 2 "SM0805" V 1130 2600 60  0001 C CNN
 F 4 "Stackpole" V 1130 2600 60  0001 C CNN "mfg"
 F 5 "RMCF0805JT1K00" V 1130 2600 60  0001 C CNN "mfg#"
@@
 $EndComp
 $Comp
-L GND #PWR054
+L GND #PWR052
 U 1 1 4C4C7B51
 P 2000 4500
-AR Path="/4C4C6618/4C4C7B51" Ref="#PWR054"  Part="1"
-AR Path="/4C2E1E7D/4C4C7B51" Ref="#PWR080"  Part="1"
-F 0 "#PWR054" H 2000 4500 30  0001 C CNN
+AR Path="/4C4C6618/4C4C7B51" Ref="#PWR052"  Part="1"
+AR Path="/4C2E1E7D/4C4C7B51" Ref="#PWR078"  Part="1"
+F 0 "#PWR078" H 2000 4500 30  0001 C CNN
 F 1 "GND" H 2000 4430 30  0001 C CNN
 	1    2000 4500
@@
 F 0 "R168" V 2330 4050 50  0000 C CNN
 F 1 "1k" V 2250 4050 50  0000 C CNN
-F 2 "R4-SM0805" V 2430 4150 60  0001 C CNN
+F 2 "SM0805" V 1130 2600 60  0001 C CNN
 F 4 "Stackpole" V 1130 2600 60  0001 C CNN "mfg"
 F 5 "RMCF0805JT1K00" V 1130 2600 60  0001 C CNN "mfg#"
@@
 F 0 "R173" V 4080 2750 50  0000 C CNN
 F 1 "1k" V 4000 2750 50  0000 C CNN
-F 2 "R4-SM0805" V 4180 2850 60  0001 C CNN
+F 2 "SM0805" V 1130 2600 60  0001 C CNN
 F 4 "Stackpole" V 1130 2600 60  0001 C CNN "mfg"
 F 5 "RMCF0805JT1K00" V 1130 2600 60  0001 C CNN "mfg#"
@@
 $EndComp
 $Comp
-L GND #PWR055
+L GND #PWR053
 U 1 1 4C2F52F0
 P 2050 3200
-AR Path="/4C4C6618/4C2F52F0" Ref="#PWR055"  Part="1"
-AR Path="/4C2E1E7D/4C2F52F0" Ref="#PWR081"  Part="1"
-F 0 "#PWR055" H 2050 3200 30  0001 C CNN
+AR Path="/4C4C6618/4C2F52F0" Ref="#PWR053"  Part="1"
+AR Path="/4C2E1E7D/4C2F52F0" Ref="#PWR079"  Part="1"
+F 0 "#PWR079" H 2050 3200 30  0001 C CNN
 F 1 "GND" H 2050 3130 30  0001 C CNN
 	1    2050 3200
@@
 F 0 "R169" V 2380 2750 50  0000 C CNN
 F 1 "1k" V 2300 2750 50  0000 C CNN
-F 2 "R4-SM0805" V 2480 2850 60  0001 C CNN
+F 2 "SM0805" V 1130 2600 60  0001 C CNN
 F 4 "Stackpole" V 1130 2600 60  0001 C CNN "mfg"
 F 5 "RMCF0805JT1K00" V 1130 2600 60  0001 C CNN "mfg#"
@@
 F 0 "R174" V 4130 1400 50  0000 C CNN
 F 1 "1k" V 4050 1400 50  0000 C CNN
-F 2 "R4-SM0805" V 4230 1500 60  0001 C CNN
+F 2 "SM0805" V 1130 2600 60  0001 C CNN
 F 4 "Stackpole" V 1130 2600 60  0001 C CNN "mfg"
 F 5 "RMCF0805JT1K00" V 1130 2600 60  0001 C CNN "mfg#"
@@
 $EndComp
 $Comp
-L GND #PWR056
+L GND #PWR054
 U 1 1 4C4C7B4E
 P 2100 1850
-AR Path="/4C4C6618/4C4C7B4E" Ref="#PWR056"  Part="1"
-AR Path="/4C2E1E7D/4C4C7B4E" Ref="#PWR082"  Part="1"
-F 0 "#PWR056" H 2100 1850 30  0001 C CNN
+AR Path="/4C4C6618/4C4C7B4E" Ref="#PWR054"  Part="1"
+AR Path="/4C2E1E7D/4C4C7B4E" Ref="#PWR080"  Part="1"
+F 0 "#PWR080" H 2100 1850 30  0001 C CNN
 F 1 "GND" H 2100 1780 30  0001 C CNN
 	1    2100 1850
@@
 F 0 "R170" V 2430 1400 50  0000 C CNN
 F 1 "1k" V 2350 1400 50  0000 C CNN
-F 2 "R4-SM0805" V 2530 1500 60  0001 C CNN
-F 4 "Stackpole" V 1130 2600 60  0001 C CNN "mfg"
-F 5 "RMCF0805JT1K00" V 1130 2600 60  0001 C CNN "mfg#"
+F 2 "SM0805" V 1130 2600 60  0001 C CNN
+F 4 "Stackpole" V 1130 2600 60  0001 C CNN "mfg"
+F 5 "RMCF0805JT1K00" V 1130 2600 60  0001 C CNN "mfg#"
