File: design/thermistor_resistor_input_1.sch (KiCad schematic (older format))
At the start: 6 parts

Commit message: Schematic BOM is now fully populated with only 3 exceptions, .cmp file is obsolete at this point, so it has been removed.
Signed-off-by: Jared Harvey <TortiseGIT@jaredharvey.com>
Parts:
- R156, R157, R158: footprint (none) -> SM0805
Changed lines of the file:
@@
-EESchema Schematic File Version 2  date 2/16/2011 5:39:18 AM
+EESchema Schematic File Version 2  date 2/16/2011 8:44:21 AM
 LIBS:power
 LIBS:freeEMS_lib
@@
 F 0 "R152" V 6230 1700 50  0000 C CNN
 F 1 "10k" V 6150 1700 50  0000 C CNN
+F 2 "SM0805" V 1130 2600 60  0001 C CNN
 F 4 "Stackpole" V 1130 2600 60  0001 C CNN "mfg"
 F 5 "RMCF0805JT10K0CT" V 1130 2600 60  0001 C CNN "mfg#"
@@
 F 0 "R151" V 5780 2100 50  0000 C CNN
 F 1 "39k" V 5700 2100 50  0000 C CNN
+F 2 "SM0805" V 1130 2600 60  0001 C CNN
 F 4 "Stackpole Electronics Inc" V 1130 2600 60  0001 C CNN "mfg"
 F 5 "RMCF0805JT39K0CT" V 1130 2600 60  0001 C CNN "mfg#"
@@
 F 0 "R150" V 5780 1300 50  0000 C CNN
 F 1 "2.2k" V 5700 1300 50  0000 C CNN
+F 2 "SM0805" V 1130 2600 60  0001 C CNN
 F 4 "Stackpole Electronics Inc" V 1130 2600 60  0001 C CNN "mfg"
 F 5 "RMCF0805JT2K20CT" V 1130 2600 60  0001 C CNN "mfg#"
