File: design/thermocuple_amplifier.sch (KiCad schematic (older format))
At the start: 2 parts, among them U18 AD597

Commit message: Schematic BOM is now fully populated with only 3 exceptions, .cmp file is obsolete at this point, so it has been removed.
Signed-off-by: Jared Harvey <TortiseGIT@jaredharvey.com>
Parts:
- U18: footprint (none) -> SO8E; Field2 AD8497ARMZ-ND -> (none); mfg (none) -> Analog Devices Inc; mfg# (none) -> AD8497ARMZ; vend1 (none) -> digikey; vend1# (none) -> AD8497ARMZ-ND
Changed lines of the file:
@@
-EESchema Schematic File Version 2  date 2/16/2011 5:39:15 AM
+EESchema Schematic File Version 2  date 2/16/2011 8:44:19 AM
 LIBS:power
 LIBS:freeEMS_lib
@@
 connector_19
 $Comp
-L GND #PWR051
+L GND #PWR049
 U 1 1 4C599401
 P 6400 4250
-F 0 "#PWR051" H 6400 4250 30  0001 C CNN
+F 0 "#PWR049" H 6400 4250 30  0001 C CNN
 F 1 "GND" H 6400 4180 30  0001 C CNN
 	1    6400 4250
@@
 5V_reg
 $Comp
-L GND #PWR052
+L GND #PWR050
 U 1 1 4C59878A
 P 5000 3950
-F 0 "#PWR052" H 5000 3950 30  0001 C CNN
+F 0 "#PWR050" H 5000 3950 30  0001 C CNN
 F 1 "GND" H 5000 3880 30  0001 C CNN
 	1    5000 3950
@@
 F 0 "U18" H 5700 3450 60  0000 C CNN
 F 1 "AD597" H 5700 3950 60  0000 C CNN
-F 5 "AD8497ARMZ-ND" H 5700 3700 60  0001 C CNN "Field2"
+F 2 "SO8E" H 5700 3700 60  0001 C CNN
+F 4 "Analog Devices Inc" H 5700 3700 60  0001 C CNN "mfg"
+F 5 "AD8497ARMZ" H 5700 3700 60  0001 C CNN "mfg#"
+F 6 "digikey" H 5700 3700 60  0001 C CNN "vend1"
+F 7 "AD8497ARMZ-ND" H 5700 3700 60  0001 C CNN "vend1#"
 	1    5700 3700
 	1    0    0    -1
