File: templates/injector_drive.sch (KiCad schematic (older format))
At the start: 17 parts

Commit message: Changed MOSFET injector driver in favor of P&H driver. Also, .gitignored .bak files. The netlist is screwed, so im going to reannotate the schematic, and associate components with SMD footprints
Parts:
- removed C?: 10pF, C1V7, symbol C
- removed D?: ZENER 4V7, D4-SMB, symbol ZENER
- removed D?: dsnub, D4-SMB, symbol DIODE
- removed D?: dsnub2, D4-SMB, symbol DIODE
- removed D?: LED, LEDV, symbol LED
- removed L?: INDUCTOR, SIL-2, symbol INDUCTOR
- removed Q?: HALL, SIL-3, symbol HALL
- removed Q?: PIP-3104, TO220_sm, symbol PIP-3104
- removed R? (x2): 2.2k, R4-SM0805, symbol R
- removed R?: 0R, R4-SM0805, symbol R
- removed R?: 680R, R4-SM0805, symbol R
- removed R?: 100k, R4-SM0805, symbol R
- removed R?: 3k, R4-SM0805, symbol R
- added C?: .01uF, symbol C
- added C?: 1uF, symbol C
- added D?: 33v 5w, symbol ZENER
- added Q?: 2N6044, symbol DARL_N
- added R?: 0.1, symbol R
- added R?: 3.9k, symbol R
- added U?: LM1949, DIP8, symbol LM1949
- R?: Field1 (none) -> newark,38k0327; Field2 (none) -> vendor1, smd w hem; Field3 (none) -> vendor2, thru w hem; Field4 (none) -> vendor2, smd w hem; Field5 (none) -> 250,mW; Field6 (none) -> 5,%; Field7 (none) -> carbon film; Field8 (none) -> other,more,stuff
Connections:
- net labels added: 5v_reg
- net labels removed: current_sense
- wire segments 48 -> 28
Other:
- note added: "3.9k x 1uF = 3.9msec"
- note added: "INJECTOR OUTPUT"
- note added: "PEAK & HOLD INJECTOR DRIVER"
- note added: "Rsense MUST BE KELVIN CONNECTED TO THE DEVICE PINS"
- note added: "TIMER CIRCUIT. 1 TAU IS THE MAX PEAK TIME."
- note removed: "CURRENT SENSE FEATURES"
- note removed: "CURRENT SENSING ALLOWS YOU TO MEASURE WHEN THE INJECTOR IS ON VS OFF"
- note removed: "IF YOU DON'T POPULATE THE SNUBBER FEATURE(S), THE MOSFET WILL DISAPATE ENERGY FROM THE INJECTOR"
- note removed: "NOTES:"
- note removed: "SNUBBER FEATURE"
- note removed: "SNUBBER FEATURE 2"
- note removed: "THE SNUBBER DIODE TO DECREASE INDUCTIVE CURRENT SPIKES"
- note removed: "YOU CAN POPULATE DIFFERENT FEATRUES WITH THIS CIRCUIT"
- moved on the sheet: P?, R?

Commit message: Implemented P&H, removed current sense circuitry, removed all unnecessary files from the repo
Parts:
- R?: value 0.1 -> 0.1 2W
Changed lines of the file:
@@
-EESchema Schematic File Version 2  date Sat 03 Jul 2010 03:41:11 AM ART
+EESchema Schematic File Version 2  date Sat 03 Jul 2010 10:29:54 AM ART
 LIBS:power
 LIBS:device
@@
 LIBS:freeEMS_lib
 LIBS:injector_drive-cache
-EELAYER 23  0
+EELAYER 24  0
 EELAYER END
 $Descr A4 11700 8267
@@
 P 5200 3450
 F 0 "R?" V 5280 3450 50  0000 C CNN
-F 1 "0.1" V 5200 3450 50  0000 C CNN
+F 1 "0.1 2W" V 5200 3450 50  0000 C CNN
 	1    5200 3450
 	0    1    1    0
